File: v2/amp_box/pot_board/pot_board.sch (KiCad schematic (older format))
At the start: 9 parts, among them P1 CONN_4, U1 ALPS_POT

Commit message: fixes
Parts:
- C1, C2: symbol C -> C-RESCUE-pot_board
Changed lines of the file:
@@
 EESchema Schematic File Version 2
+LIBS:pot_board-rescue
 LIBS:power
 LIBS:device
@@
 LIBS:valves
 LIBS:pot_board-cache
-EELAYER 27 0
+EELAYER 25 0
 EELAYER END
 $Descr A4 11693 8268
@@
 	7750 1900 7750 2150
 $Comp
-L GND #PWR2
+L GND-RESCUE-pot_board #PWR2
 U 1 1 55D48102
 P 7550 2000
@@
 	7650 1900 7550 1900
 $Comp
-L C C1
+L C-RESCUE-pot_board C1
 U 1 1 56177CF4
 P 7250 2050
@@
 $EndComp
 $Comp
-L C C2
+L C-RESCUE-pot_board C2
 U 1 1 56177D01
 P 7950 2050
@@
 	8150 2050 8150 2150
 $Comp
-L GND #PWR1
+L GND-RESCUE-pot_board #PWR1
 U 1 1 56177D58
 P 7050 2150
@@
 $EndComp
 $Comp
-L GND #PWR3
+L GND-RESCUE-pot_board #PWR3
 U 1 1 56177D5E
 P 8150 2150
