File: v2/selector_box/rid_relay_audio/selector_rid_ground.sch (KiCad schematic (older format))
At the start: 40 parts, among them K3 CONN_3, K6 CONN_3, K7 CONN_3, K8 CONN_3, K9 CONN_3, P1 DIP05-2A72-21L, P10 DIP05-2A72-21L, P11 DIP05-1A72-12L, P12 DIP05-2A72-21L, P13 CONN_4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

Commit message: fixes
Parts:
- removed C1, C10: 47uF, ~, symbol CP1
- removed D2, D3, D6, D9: DIODE, ~, symbol DIODE
- removed FB1, FB2: FILTER, ~, symbol FILTER
- removed K6, K7, K8, K9: CONN_3, ~, symbol CONN_3
- removed P10, P12, P5, P6: DIP05-2A72-21L, ~, symbol DIL14
- removed P11, P8, P9: DIP05-1A72-12L, ~, symbol DIL14
- removed P14, P15, P16: CONN_4, ~, symbol CONN_4
- removed P2, P3, P4: CONN_2, ~, symbol CONN_2
- removed Q2, Q3, Q4, Q5: BC547, TO92, symbol BC547
- removed R2, R3, R4, R5: 12K, ~, symbol R
- added P1: CONN_4, Pin_Headers:Pin_Header_Straight_1x04, symbol CONN_4
- D1: footprint ~ -> Diodes_ThroughHole:Diode_DO-35_SOD27_Horizontal_RM10
- K1: renamed from K3; footprint ~ -> Pin_Headers:Pin_Header_Straight_1x03
- P2: renamed from P13; footprint ~ -> Pin_Headers:Pin_Header_Straight_1x04
- P3: renamed from P1; footprint ~ -> Housings_DIP:DIP-14_W7.62mm_LongPads
- P4: renamed from P7; footprint ~ -> Housings_DIP:DIP-14_W7.62mm_LongPads
- Q1: footprint TO92 -> TO_SOT_Packages_THT:TO-92_Inline_Narrow_Oval
- R1: footprint ~ -> Discret:R4; symbol R -> R-RESCUE-selector_rid_ground
Connections:
- net labels removed: EN2, EN3, EN4, EN_MUTE, G_IN2, G_IN3, G_IN4, L_IN2, L_IN3, L_IN4, R_IN2, R_IN3, R_IN4
- wire segments 143 -> 34
- no-connect marks 80 -> 18
Other:
- moved on the sheet: P2
