File: v2/power_box/bridge_fuse/bridge_fuse.sch (KiCad schematic (older format))
At the start: 9 parts, among them K1 CONN_3

Commit message: update
Parts:
- C1, C2, C3, C4, C5, C6: symbol C -> C-RESCUE-bridge_fuse
Changed lines of the file:
@@
 EESchema Schematic File Version 2
+LIBS:bridge_fuse-rescue
 LIBS:power
 LIBS:device
@@
 LIBS:valves
 LIBS:bridge_fuse-cache
-EELAYER 27 0
+EELAYER 25 0
 EELAYER END
 $Descr A4 11693 8268
@@
 $EndComp
 $Comp
-L C C1
+L C-RESCUE-bridge_fuse C1
 U 1 1 52497C07
 P 8800 3350
@@
 $EndComp
 $Comp
-L C C2
+L C-RESCUE-bridge_fuse C2
 U 1 1 52497C14
 P 8800 3850
@@
 $EndComp
 $Comp
-L C C3
+L C-RESCUE-bridge_fuse C3
 U 1 1 52497C74
 P 6300 3250
@@
 $EndComp
 $Comp
-L C C4
+L C-RESCUE-bridge_fuse C4
 U 1 1 52497C7E
 P 6300 4200
@@
 $EndComp
 $Comp
-L C C5
+L C-RESCUE-bridge_fuse C5
 U 1 1 52497C84
 P 4600 4200
@@
 $EndComp
 $Comp
-L C C6
+L C-RESCUE-bridge_fuse C6
 U 1 1 52497C8D
 P 4600 3250
