File: v2/power_box/soft_start/soft_start.sch (KiCad schematic (older format))
At the start: 26 parts, among them K1 CONN_3, P1 CONN_2, P2 CONN_2, P3 CONN_2, P4 CONN_2, P5 CONN_2, P6 CONN_2, P7 CONN_2, P8 CONN_2, Q1 BC547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

Commit message: update
Parts:
- R1, R2, R3, R4, R5, R6: symbol R -> R-RESCUE-soft_start
Changed lines of the file:
@@
 EESchema Schematic File Version 2
+LIBS:soft_start-rescue
 LIBS:power
 LIBS:device
@@
 LIBS:w_relay
 LIBS:soft_start-cache
-EELAYER 27 0
+EELAYER 25 0
 EELAYER END
 $Descr A4 11693 8268
@@
 $EndComp
 $Comp
-L GND #PWR2
+L GND-RESCUE-soft_start #PWR2
 U 1 1 53943F3B
 P 3150 2650
@@
 $EndComp
 $Comp
-L GND #PWR3
+L GND-RESCUE-soft_start #PWR3
 U 1 1 53943F48
 P 3150 4100
@@
 EN_2
 $Comp
-L R R1
+L R-RESCUE-soft_start R1
 U 1 1 53944164
 P 3850 2350
@@
 $EndComp
 $Comp
-L R R2
+L R-RESCUE-soft_start R2
 U 1 1 53944171
 P 3850 3800
@@
 5V
 $Comp
-L GND #PWR5
+L GND-RESCUE-soft_start #PWR5
 U 1 1 5394462F
 P 4950 4950
@@
 $EndComp
 $Comp
-L GND #PWR1
+L GND-RESCUE-soft_start #PWR1
 U 1 1 53FC7314
 P 2650 5950
@@
 EN_3
 $Comp
-L R R3
+L R-RESCUE-soft_start R3
 U 1 1 53FC7320
 P 3350 5650
@@
 5V
 $Comp
-L GND #PWR6
+L GND-RESCUE-soft_start #PWR6
 U 1 1 53FC8FA5
 P 5800 2900
@@
 5V
 $Comp
-L GND #PWR4
+L GND-RESCUE-soft_start #PWR4
 U 1 1 53FC8FC7
 P 4800 2900
@@
 	2800 2650 2750 2650
 $Comp
-L R R4
+L R-RESCUE-soft_start R4
 U 1 1 53FC9A1C
 P 8550 2250
@@
 $EndComp
 $Comp
-L R R5
+L R-RESCUE-soft_start R5
 U 1 1 53FC9A29
 P 8550 2500
@@
 $EndComp
 $Comp
-L R R6
+L R-RESCUE-soft_start R6
 U 1 1 53FC9A2F
 P 8550 2750
