File: v2/selector_box/selector_ctrl_v2/selector_ctrl.sch (KiCad schematic (older format))
At the start: 59 parts, among them J1 ATMEGA328P, P1 CONN_4, P10 DIP05-1A72-12L, P11 Msgeq7_1, P12 Msgeq7_1, P16 DIP05-2A72-21L, P17 DIP05-2A72-21L, P18 DIP05-1A72-12L, P19 DIP05-1A72-12L, P2 CONN_4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

Commit message: update
Parts:
- C1, C3: symbol CP1 -> CP1-RESCUE-selector_ctrl
- C10, C11, C12, C2, C4, C5, C6, C7, C8, C9: symbol C -> C-RESCUE-selector_ctrl
- R1, R2, R3, R4, R5, R6, R7, R8: symbol R -> R-RESCUE-selector_ctrl
Connections:
- wire segments 234 -> 233
Changed lines of the file:
@@
 EESchema Schematic File Version 2
+LIBS:selector_ctrl-rescue
 LIBS:power
 LIBS:device
@@
 LIBS:valves
 LIBS:selector_ctrl-cache
-EELAYER 27 0
+EELAYER 25 0
 EELAYER END
 $Descr A4 11693 8268
@@
 $EndComp
 $Comp
-L CP1 C1
+L CP1-RESCUE-selector_ctrl C1
 U 1 1 564ED6D5
 P 2100 -14500
@@
 $EndComp
 $Comp
-L C C2
+L C-RESCUE-selector_ctrl C2
 U 1 1 564ED6D6
 P 4200 -11550
@@
 $EndComp
 $Comp
-L CP1 C3
+L CP1-RESCUE-selector_ctrl C3
 U 1 1 564ED6DA
 P 5350 -14800
@@
 	5650 -15150 5650 -14450
 $Comp
-L R R3
+L R-RESCUE-selector_ctrl R3
 U 1 1 564ED6DB
 P 5550 -15250
@@
 	4800 -11050 5000 -11050
 $Comp
-L C C12
+L C-RESCUE-selector_ctrl C12
 U 1 1 564ED6E0
 P 7500 -11800
@@
 $EndComp
 $Comp
-L C C5
+L C-RESCUE-selector_ctrl C5
 U 1 1 564ED6EE
 P 5700 -8250
@@
 $EndComp
 $Comp
-L C C9
+L C-RESCUE-selector_ctrl C9
 U 1 1 564ED6EF
 P 7200 -7750
@@
 $EndComp
 $Comp
-L C C11
+L C-RESCUE-selector_ctrl C11
 U 1 1 564ED6F0
 P 7400 -8150
@@
 $EndComp
 $Comp
-L C C7
+L C-RESCUE-selector_ctrl C7
 U 1 1 564ED6F1
 P 6850 -7450
@@
 Connection ~ 5700 -8050
 $Comp
-L R R5
+L R-RESCUE-selector_ctrl R5
 U 1 1 564ED6F2
 P 6550 -8400
@@
 $EndComp
 $Comp
-L C C4
+L C-RESCUE-selector_ctrl C4
 U 1 1 564ED6F7
 P 5550 -5850
@@
 $EndComp
 $Comp
-L C C8
+L C-RESCUE-selector_ctrl C8
 U 1 1 564ED6F8
 P 7050 -5350
@@
 $EndComp
 $Comp
-L C C10
+L C-RESCUE-selector_ctrl C10
 U 1 1 564ED6F9
 P 7250 -5750
@@
 $EndComp
 $Comp
-L C C6
+L C-RESCUE-selector_ctrl C6
 U 1 1 564ED6FA
 P 6700 -5050
@@
 Connection ~ 5550 -5650
 $Comp
-L R R4
+L R-RESCUE-selector_ctrl R4
 U 1 1 564ED6FB
 P 6400 -6000
@@
 $EndComp
 $Comp
-L R R1
+L R-RESCUE-selector_ctrl R1
 U 1 1 564ED704
 P 2100 2650
@@
 $EndComp
 $Comp
-L R R6
+L R-RESCUE-selector_ctrl R6
 U 1 1 564ED70A
 P 7000 6050
@@
 Wire Wire Line
 	4000 3000 3750 3000
-Wire Wire Line
-	3650 3000 3650 2850
 Wire Wire Line
 	2800 2850 2800 3000
@@
 Wire Wire Line
 	7900 6900 7900 5800
-Text Label 3650 2850 0    60   ~ 0
-G_OUT
 Text Label 5650 2650 3    60   ~ 0
 G_OUT
@@
 $EndComp
 $Comp
-L R R2
+L R-RESCUE-selector_ctrl R2
 U 1 1 564ED714
 P 2200 6100
@@
 $EndComp
 $Comp
-L R R7
+L R-RESCUE-selector_ctrl R7
 U 1 1 564ED719
 P 6800 2800
@@
 $EndComp
 $Comp
-L R R8
+L R-RESCUE-selector_ctrl R8
 U 1 1 564ED722
 P 13650 2300
