File: siprog/ponyser1.sch (KiCad schematic (older format))
At the start: 26 parts, among them J1 DB9 FEMALE, J2 RJ45, K1 CONN_3, K2 CONN_3, K3 CONN_3, P1 CONN_2, P2 CONN_2, P3 CONN_4, P4 CONN_2, P5 CONN_2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

Commit message: updates
Parts:
- C12: symbol C -> C-RESCUE-ponyser1
- C3, C4: symbol CP1 -> CP1-RESCUE-ponyser1
- R1, R3, R4, R5, R6: symbol R -> R-RESCUE-ponyser1
- Z1, Z2, Z3: symbol ZENER -> ZENER-RESCUE-ponyser1
Changed lines of the file:
@@
 EESchema Schematic File Version 2
+LIBS:ponyser1-rescue
 LIBS:power
 LIBS:device
@@
 LIBS:db9_fm
 LIBS:ponyser1-cache
-EELAYER 27 0
+EELAYER 25 0
 EELAYER END
 $Descr A4 11693 8268
@@
 $EndDescr
 $Comp
-L R R4
+L R-RESCUE-ponyser1 R4
 U 1 1 523C4D70
 P 6050 2800
@@
 $EndComp
 $Comp
-L R R5
+L R-RESCUE-ponyser1 R5
 U 1 1 523C4D8E
 P 6050 3050
@@
 $EndComp
 $Comp
-L R R6
+L R-RESCUE-ponyser1 R6
 U 1 1 523C4D94
 P 6050 3300
@@
 $EndComp
 $Comp
-L R R3
+L R-RESCUE-ponyser1 R3
 U 1 1 523C4D9A
 P 6800 2650
@@
 $EndComp
 $Comp
-L R R1
+L R-RESCUE-ponyser1 R1
 U 1 1 523C4DA0
 P 8000 3150
@@
 $EndComp
 $Comp
-L ZENER Z1
+L ZENER-RESCUE-ponyser1 Z1
 U 1 1 523C4DAD
 P 6500 3700
@@
 $EndComp
 $Comp
-L ZENER Z2
+L ZENER-RESCUE-ponyser1 Z2
 U 1 1 523C4DBA
 P 6800 3700
@@
 $EndComp
 $Comp
-L ZENER Z3
+L ZENER-RESCUE-ponyser1 Z3
 U 1 1 523C4DC0
 P 7100 3700
@@
 $EndComp
 $Comp
-L CP1 C3
+L CP1-RESCUE-ponyser1 C3
 U 1 1 523C4E2F
 P 6850 1950
@@
 $EndComp
 $Comp
-L C C12
+L C-RESCUE-ponyser1 C12
 U 1 1 523C4E3E
 P 7350 1950
@@
 $EndComp
 $Comp
-L CP1 C4
+L CP1-RESCUE-ponyser1 C4
 U 1 1 523C51C1
 P 8800 1900
@@
 $EndComp
 $Comp
-L GND #PWR01
+L GND-RESCUE-ponyser1 #PWR01
 U 1 1 523C528C
 P 6850 2300
@@
 $EndComp
 $Comp
-L GND #PWR02
+L GND-RESCUE-ponyser1 #PWR02
 U 1 1 523C52DE
 P 7350 2300
@@
 $EndComp
 $Comp
-L GND #PWR03
+L GND-RESCUE-ponyser1 #PWR03
 U 1 1 523C5307
 P 8100 2300
@@
 $EndComp
 $Comp
-L GND #PWR04
+L GND-RESCUE-ponyser1 #PWR04
 U 1 1 523C5331
 P 8800 2300
@@
 $EndComp
 $Comp
-L GND #PWR05
+L GND-RESCUE-ponyser1 #PWR05
 U 1 1 523C5383
 P 6500 4050
@@
 $EndComp
 $Comp
-L GND #PWR06
+L GND-RESCUE-ponyser1 #PWR06
 U 1 1 523C5389
 P 6800 4050
@@
 $EndComp
 $Comp
-L GND #PWR07
+L GND-RESCUE-ponyser1 #PWR07
 U 1 1 523C538F
 P 7100 4050
@@
 $EndComp
 $Comp
-L GND #PWR08
+L GND-RESCUE-ponyser1 #PWR08
 U 1 1 523C5410
 P 8250 3250
@@
 $EndComp
 $Comp
-L GND #PWR09
+L GND-RESCUE-ponyser1 #PWR09
 U 1 1 523C54B3
 P 9450 1800
@@
 $EndComp
 $Comp
-L GND #PWR010
+L GND-RESCUE-ponyser1 #PWR010
 U 1 1 523C597B
 P 4250 3850
@@
 	3050 6750 3050 6800
 $Comp
-L GND #PWR012
+L GND-RESCUE-ponyser1 #PWR012
 U 1 1 53B04D17
 P 3050 7250
@@
 	3050 5600 3050 5700
 $Comp
-L GND #PWR013
+L GND-RESCUE-ponyser1 #PWR013
 U 1 1 53B054D0
 P 3050 5700
