File: rc_car/rc_car.sch (KiCad schematic (older format))
At the start: 27 parts, among them IC1 L293D, J1 Atmega328, m1_out1 CONN_2, m2_out1 CONN_2

Commit message: updates,rc_car
Connections:
- net 5V: now also i2c1.3 (P3); no longer i2c1.4 (P4)
- net GND: now also i2c1.2 (P2); no longer i2c1.1 (P1)
- net SCL: now also i2c1.1 (P1); no longer i2c1.2 (P2)
- net SDA: now also i2c1.4 (P4); no longer i2c1.3 (P3)
Changed lines of the file:
@@
 LIBS:valves
 LIBS:rc_car-cache
-LIBS:power_split-cache
 EELAYER 25 0
 EELAYER END
@@
 L GND #PWR03
 U 1 1 587A7D80
-P 3700 2100
-F 0 "#PWR03" H 3700 2100 30  0001 C CNN
-F 1 "GND" H 3700 2030 30  0001 C CNN
-F 2 "" H 3700 2100 60  0000 C CNN
-F 3 "" H 3700 2100 60  0000 C CNN
-	1    3700 2100
+P 3800 2200
+F 0 "#PWR03" H 3800 2200 30  0001 C CNN
+F 1 "GND" H 3800 2130 30  0001 C CNN
+F 2 "" H 3800 2200 60  0000 C CNN
+F 3 "" H 3800 2200 60  0000 C CNN
+	1    3800 2200
 	1    0    0    -1
 $EndComp
@@
 Text Label 5800 3700 0    60   ~ 0
 SDA
-Text Label 3800 2200 3    60   ~ 0
+Text Label 3700 2100 3    60   ~ 0
 SCL
-Text Label 4000 2200 3    60   ~ 0
+Text Label 4100 2100 3    60   ~ 0
 SDA
 Wire Wire Line
@@
 Wire Wire Line
 	2900 6250 2900 6150
-Text Label 4100 2100 3    60   ~ 0
+Text Label 4000 2200 3    60   ~ 0
 5V
 $Comp

Commit message: rc-car
Parts:
- removed C6: 470uF, Capacitors_ThroughHole:C_Radial_D6.3_L11.2_P2.5, symbol CP1
- added D1, D2, D3, D4: D, Discret:D4, symbol D
- added P1, P2: CONN_2, Connect:bornier2, symbol CONN_2
- added P3, P4: CONN_01X03, Pin_Headers:Pin_Header_Straight_1x03, symbol CONN_01X03
- added Q1, Q12, Q3, Q8: IRFU9024N, TO_SOT_Packages_THT:TO-251AA, symbol Q_PMOS_GDS
- added Q10, Q13, Q2, Q4, Q9: IRLU024N, TO_SOT_Packages_THT:TO-251AA, symbol Q_NMOS_GDS
- added Q11, Q14, Q7: Q_NMOS_SGD, TO_SOT_Packages_THT:TO-92_Inline_Narrow_Oval, symbol Q_NMOS_SGD
- added Q5, Q6: BC547, TO_SOT_Packages_THT:TO-92_Inline_Narrow_Oval, symbol BC547
- added R1, R11, R12, R13, R16, R17, R2, R6, R7, R8, R9: 10K, Discret:R1, symbol R
- added R10, R3, R4: 220R, Discret:R1, symbol R
- added R14, R15: 0R, Discret:R4, symbol R
- added R5: 10K, Discret:R4, symbol R
Connections:
- net labels added: GNDREF, MISO, MOSI, RST, SCK
- wire segments 116 -> 197
Other:
- moved on the sheet: C1, pwr_motor1

Commit message: fixes
Parts:
- removed D1, D2, D3, D4: D, Discret:D4, symbol D
- removed P1, P2: CONN_2, Connect:bornier2, symbol CONN_2
- removed Q1, Q12, Q3, Q8: IRFU9024N, TO_SOT_Packages_THT:TO-251AA, symbol Q_PMOS_GDS
- removed Q10, Q13, Q2, Q4, Q9: IRLU024N, TO_SOT_Packages_THT:TO-251AA, symbol Q_NMOS_GDS
- removed Q11, Q14, Q7: Q_NMOS_SGD, TO_SOT_Packages_THT:TO-92_Inline_Narrow_Oval, symbol Q_NMOS_SGD
- removed Q5, Q6: BC547, TO_SOT_Packages_THT:TO-92_Inline_Narrow_Oval, symbol BC547
- removed R1, R11, R12, R13, R16, R17, R2, R6, R7, R8: 10K, Discret:R1, symbol R
- removed R10, R3, R4: 220R, Discret:R1, symbol R
- removed R14, R15: 0R, Discret:R4, symbol R
- removed R5: 10K, Discret:R4, symbol R
Connections:
- wire segments 197 -> 126
- no-connect marks 4 -> 3
