File: v2/amp_box/power_ctrl/power_ctrl.kicad_pcb (KiCad board)
At the start: 2 copper layers, 239.4 x 199.7 mm, 174 parts, among them IC1 L293D, J1 Atmega328, J2 RJ12, P1 Msgeq7_1, P10 DIP05-2A72-21L, P11 DIP05-1A72-12L, P12 DIP05-2A72-21L, P13 DIP05-1A72-12L, P14 DIP05-2A72-21L, P15 DIP05-1A72-12L, P16 CONN_4, P17 CONN_02X04, P18 CONN_02X04, P19 CONN_01X03, P2 Msgeq7_1, P20 CONN_01X03, P21 DIP05-2A72-21L, P22 DIP05-2A72-21L, P23 CONN_01X03, P24 CONN_01X03, P25 CONN_01X02, P26 CONN_01X02, P27 CONN_01X02, P28 CONN_01X02, P29 CONN_01X02, P3 CONN_4, P30 CONN_01X02, P31 CONN_01X02, P32 CONN_01X02, P33 CONN_01X02, P34 CONN_01X02, P35 CONN_01X03, P36 CONN_01X03, P4 CONN_4, P5 CONN_4, P6 CONN_4, P7 DIP05-2A72-21L, P8 DIP05-2A72-21L, P9 DIP05-1A72-12L, Q1 BC547, Q10 BC547, Q11 BC547, Q12 Q_PMOS_GDS, Q2 BC547, Q3 BC547, Q4 BC547, Q5 BC547, Q6 Q_NJFET_DSG, Q7 Q_NJFET_DSG, Q8 Q_NJFET_DSG, Q9 Q_NJFET_DSG, U1 7805, U2 7809

Commit message: updates
Parts:
- added 12V_AUX1: CONN_2, Connect:bornier2, F.Cu at (-27.9, -128.9)
- added 12V_IN1: CONN_2, Connect:bornier2, F.Cu at (-27.9, -139.7)
- added 5V_AUX1: CONN_2, Connect:bornier2, F.Cu at (28.6, -148.0)
- added C1: 100nF, Capacitors_ThroughHole:C_Rect_L7_W2_P5, F.Cu at (0.64, -104.8)
- added C10: 100n, Capacitors_ThroughHole:C_Rect_L7_W2_P5, F.Cu at (0.64, -79.4)
- added C11: 100n, Capacitors_ThroughHole:C_Rect_L7_W2_P5, F.Cu at (27.3, -75.6)
- added C12: 100n, Capacitors_ThroughHole:C_Rect_L7_W2_P5, F.Cu at (1.91, -75.6)
- added C13: 470uF, Capacitors_ThroughHole:C_Rect_L7_W2_P5, F.Cu at (29.8, -85.1)
- added C2: 470uF, Capacitors_ThroughHole:C_Radial_D7.5_L11.2_P2.5, F.Cu at (-15.9, -139.7)
- added C3: 100nF, Capacitors_ThroughHole:C_Rect_L7_W2_P5, F.Cu at (-10.2, -136.5)
- added C34: 100n, Capacitors_ThroughHole:C_Rect_L7_W2_P5, F.Cu at (38.1, -88.3)
- added C4: 100nF, Capacitors_ThroughHole:C_Rect_L7_W2_P5, F.Cu at (-5.08, -136.5)
- added C5: 10uF, Capacitors_ThroughHole:C_Radial_D5_L6_P2.5, F.Cu at (0.00, -140.3)
- added C6: 100nF, Capacitors_ThroughHole:C_Rect_L7_W2_P5, F.Cu at (15.9, -106.0)
- added C7: 100nF, Capacitors_ThroughHole:C_Rect_L7_W2_P5, F.Cu at (5.08, -136.5)
- added C8: 10uF, Capacitors_ThroughHole:C_Radial_D5_L6_P2.5, F.Cu at (9.53, -139.1)
- added C9: 4.7uF, Capacitors_ThroughHole:C_Radial_D5_L11_P2.5, F.Cu at (-14.0, -103.5)
- added D1: DIODE, Diodes_ThroughHole:Diode_DO-35_SOD27_Horizontal_RM10, F.Cu at (-21.6, -134.6)
- added D2: DIODE, Diodes_ThroughHole:Diode_DO-35_SOD27_Horizontal_RM10, F.Cu at (-2.54, -148.6)
- added D3: LED, LEDs:LED-3MM, F.Cu at (18.4, -146.1)
- added FB1: FILTER, Discret:R4, F.Cu at (0.64, -118.1)
- added FB2: FILTER, Discret:R4, F.Cu at (21.0, -127.6)
- added FB3: FILTER, Discret:R4, F.Cu at (21.0, -133.3)
- added FB4: FILTER, Discret:R4, F.Cu at (5.08, -144.8)
- added FB5: FILTER, Discret:R4, F.Cu at (22.2, -111.1)
- added IC1: L293D, Housings_DIP:DIP-16_W7.62mm_LongPads, F.Cu at (5.71, -80.0)
- added J1: Atmega328, Housings_DIP:DIP-28_W7.62mm_LongPads, F.Cu at (4.45, -127.0)
- added J2: RJ12, Connect:RJ12_E, F.Cu at (44.5, -129.5)
- added P16: CONN_4, Pin_Headers:Pin_Header_Straight_1x04, F.Cu at (29.8, -125.7)
- added P17: CONN_02X04, Pin_Headers:Pin_Header_Straight_2x04, F.Cu at (29.2, -105.4)
- added P23: CONN_01X03, Pin_Headers:Pin_Header_Straight_1x03, F.Cu at (-17.8, -88.9)
- added P24: CONN_01X03, Pin_Headers:Pin_Header_Straight_1x03, F.Cu at (-12.7, -92.7)
- added P31: CONN_01X02, Pin_Headers:Pin_Header_Straight_1x02, F.Cu at (-22.2, -118.7)
- added P32: CONN_01X02, Pin_Headers:Pin_Header_Straight_1x02, F.Cu at (-22.2, -107.3)
- added P34: CONN_01X02, Pin_Headers:Pin_Header_Straight_1x02, F.Cu at (-8.26, -120.0)
- added P35: CONN_01X03, Pin_Headers:Pin_Header_Straight_1x03, F.Cu at (21.0, -123.8)
- added P36: CONN_01X03, Pin_Headers:Pin_Header_Straight_1x03, F.Cu at (21.0, -120.0)
- added P37: CONN_2, Connect:bornier2, F.Cu at (-138.4, 56.5)
- added P38: CONN_2, Connect:bornier2, F.Cu at (-108.6, 56.5)
- added P38: CONN_2, Connect:bornier2, F.Cu at (-116.2, 48.9)
- added P39: CONN_2, Connect:bornier2, F.Cu at (-162.6, 56.5)
- added P40: CONN_2, Connect:bornier2, F.Cu at (-130.8, 48.9)
- added P41: CONN_2, Connect:bornier2, F.Cu at (-97.8, 56.5)
- added P42: CONN_2, Connect:bornier2, F.Cu at (-105.4, 48.9)
- added P43: CONN_2, Connect:bornier2, F.Cu at (-149.2, 56.5)
- added P44: CONN_2, Connect:bornier2, F.Cu at (-141.6, 48.9)
- added Q1: BC547, TO_SOT_Packages_THT:TO-92_Inline_Wide, F.Cu at (-21.0, -114.9)
- added Q10: BC547, TO_SOT_Packages_THT:TO-92_Inline_Wide, F.Cu at (-21.0, -126.4)
- added Q2: BC547, TO_SOT_Packages_THT:TO-92_Inline_Wide, F.Cu at (-4.45, -81.9)
- added Q3: BC547, TO_SOT_Packages_THT:TO-92_Inline_Wide, F.Cu at (-8.89, -83.8)
- added Q4: BC547, TO_SOT_Packages_THT:TO-92_Inline_Wide, F.Cu at (-8.89, -99.1)
- added Q5: BC547, TO_SOT_Packages_THT:TO-92_Inline_Wide, F.Cu at (-6.99, -91.4)
- added R1: 680R, Discret:R4, F.Cu at (21.0, -141.6)
- added R10: 12K, Discret:R1, F.Cu at (-2.54, -97.2)
- added R2: 100R, Discret:R4, F.Cu at (-12.7, -107.3)
- added R25: 12K, Discret:R4, F.Cu at (-13.3, -123.2)
- added R6: 12K, Discret:R4, F.Cu at (-13.3, -111.1)
- added R7: 12K, Discret:R1, F.Cu at (0.64, -91.4)
- added R8: 12K, Discret:R1, F.Cu at (-1.27, -94.0)
- added R9: 12K, Discret:R1, F.Cu at (-4.45, -100.3)
- added U1: 7805, TO_SOT_Packages_THT:TO-220_Neutral123_Vertical_LargePads, F.Cu at (-7.62, -148.6)
- added ir1: CONN_4, Pin_Headers:Pin_Header_Straight_1x04, F.Cu at (-3.81, -112.4)
- added j_pwr1: CONN_2, Pin_Headers:Pin_Header_Straight_1x02, F.Cu at (34.9, -94.0)
- added motor_ctrl1: CONN_4, Pin_Headers:Pin_Header_Straight_1x04, F.Cu at (10.8, -75.6)
- added mute1: CONN_01X04, Pin_Headers:Pin_Header_Straight_1x04, F.Cu at (-3.17, -130.2)
- added pwr_motor1: CONN_2, Connect:bornier2, F.Cu at (34.9, -78.7)
- C15, C16, C26, C27: value 1uF -> 4.7uF
- R13, R14, R20, R21: value 10K -> 3K
- moved R17 4.26 mm to (-268.0, -94.0)
- moved R3 3.70 mm to (-267.3, -111.8)
- moved P27 3.18 mm to (-233.7, -154.3), turned to 90 degrees
- moved P28 3.17 mm to (-240.7, -151.8)
- moved P33 2.84 mm to (-226.1, -154.3), turned to 270 degrees
- moved R11 1.80 mm to (-273.1, -112.4)
- moved R18 1.80 mm to (-273.1, -93.3)
- moved C14 1.27 mm to (-262.9, -111.8)
- moved C17 1.27 mm to (-262.9, -94.0)
Routing:
- net /12V: track 41.0 -> 416.2 mm
- net /5V: track 498.4 -> 771.1 mm
- net /EQ7_STROBE: track 66.3 -> 105.2 mm
- net /VIN_MOTOR: track 28.3 -> 56.5 mm
- net /EQ7_RST: track 75.2 -> 103.4 mm
- net Net-(C2-Pad1): track 28.0 -> 56.0 mm
- net Net-(C4-Pad2): track 24.6 -> 49.1 mm
- net Net-(C6-Pad1): track 21.2 -> 42.3 mm
- net /EQ7_DATA_L: track 46.9 -> 67.5 mm
- net /PREAMP: track 17.5 -> 34.9 mm
- net /CH1_EN: track 81.6 -> 98.9 mm
- net /MOTOUT_R: track 17.3 -> 34.7 mm
- net /MOTOUT_L: track 17.3 -> 34.7 mm
- net /MOT_EN: track 17.0 -> 33.9 mm
- net Net-(FB3-Pad2): track 16.1 -> 32.1 mm
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Other:
- board size 239.4 x 199.7 mm -> 367 x 249.6 mm

Commit message: updates
Parts:
- removed the 12V_AUX1 at (-155.6, -129.5)
- removed the 12V_IN1 at (-155.6, -140.3)
- removed the 5V_AUX1 at (28.6, -148.0)
- removed the 5V_AUX1 at (-99.1, -148.6)
- removed the C1 at (-127.0, -105.4)
- removed C10 (x2), C11 (x2), C12 (x2), C34 (x2): 100n, Capacitors_ThroughHole:C_Rect_L7_W2_P5
- removed the C13 at (29.8, -85.1)
- removed the C13 at (-97.8, -85.7)
- removed the C2 at (-143.5, -140.3)
- removed the C3 at (-137.8, -137.2)
- removed the C4 at (-132.7, -137.2)
- removed the C5 at (-127.6, -141.0)
- removed the C6 at (-111.8, -106.7)
- removed the C7 at (-122.6, -137.2)
- removed the C8 at (-118.1, -139.7)
- removed the C9 at (-141.6, -104.1)
- removed the D1 at (-149.2, -135.3)
- removed the D2 at (-130.2, -149.2)
- removed the D3 at (-109.2, -146.7)
- removed the FB1 at (-127.0, -118.7)
- removed the FB2 at (-106.7, -128.3)
- removed the FB3 at (-106.7, -134.0)
- removed the FB4 at (-122.6, -145.4)
- removed the FB5 at (-105.4, -111.8)
- removed IC1 (x2): L293D, Housings_DIP:DIP-16_W7.62mm_LongPads
- removed the J1 at (-123.2, -127.6)
- removed the J2 at (-83.2, -130.2)
- removed the P16 at (29.8, -125.7)
- removed the P16 at (-97.8, -126.4)
- removed the P17 at (29.2, -105.4)
- removed the P17 at (-98.4, -106.0)
- removed the P23 at (-145.4, -89.5)
- removed the P24 at (-140.3, -93.3)
- removed the P31 at (-149.9, -119.4)
- removed the P32 at (-149.9, -108.0)
- removed the P34 at (-135.9, -120.7)
- removed the P35 at (-106.7, -124.5)
- removed the P36 at (-106.7, -120.7)
- removed the Q1 at (-148.6, -115.6)
- removed the Q10 at (-148.6, -127.0)
- removed the Q2 at (-132.1, -82.5)
- removed the Q3 at (-136.5, -84.5)
- removed the Q4 at (-136.5, -99.7)
- removed the Q5 at (-134.6, -92.1)
- removed the R1 at (-106.7, -142.2)
- removed the R10 at (-2.54, -97.2)
- removed the R10 at (-130.2, -97.8)
- removed the R2 at (-140.3, -108.0)
- removed the R25 at (-13.3, -123.2)
- removed the R25 at (-141.0, -123.8)
- removed the R6 at (-13.3, -111.1)
- removed the R6 at (-141.0, -111.8)
- removed the R7 at (0.64, -91.4)
- removed the R7 at (-127.0, -92.1)
- removed the R8 at (-1.27, -94.0)
- removed the R8 at (-128.9, -94.6)
- removed the R9 at (-4.45, -100.3)
- removed the R9 at (-132.1, -101.0)
- removed the U1 at (-135.3, -149.2)
- removed the ir1 at (-131.4, -113.0)
- removed the j_pwr1 at (34.9, -94.0)
- removed the j_pwr1 at (-92.7, -94.6)
- removed the motor_ctrl1 at (10.8, -75.6)
- removed the motor_ctrl1 at (-116.8, -76.2)
- removed the mute1 at (-3.17, -130.2)
- removed the mute1 at (-130.8, -130.8)
- removed the pwr_motor1 at (34.9, -78.7)
- removed the pwr_motor1 at (-92.7, -79.4)
- added 5V_AUX1: CONN_2, Connect:bornier2, F.Cu at (-378.5, -73.0)
- added C13: 470uF, Capacitors_ThroughHole:C_Rect_L7_W2_P5, F.Cu at (-367.0, -62.2)
- added C14: 0.1, Capacitors_ThroughHole:C_Rect_L7_W2_P5, F.Cu at (-360.7, -158.8)
- added C15: 4.7uF, Capacitors_ThroughHole:C_Radial_D5_L11_P2, F.Cu at (-348.0, -161.9)
- added C17: 0.1, Capacitors_ThroughHole:C_Rect_L7_W2_P5, F.Cu at (-360.7, -141.0)
- added C26: 4.7uF, Capacitors_ThroughHole:C_Radial_D5_L11_P2, F.Cu at (-348.0, -137.8)
- added C35: 10uF, Capacitors_ThroughHole:C_Radial_D5_L11_P2, F.Cu at (-365.1, -154.9)
- added C36: 10uF, Capacitors_ThroughHole:C_Radial_D5_L11_P2, F.Cu at (-365.1, -144.8)
- added C37: 100nF, Capacitors_ThroughHole:C_Rect_L7_W2_P5, F.Cu at (-2.54, -162.6)
- added C38: 100nF, Capacitors_ThroughHole:C_Rect_L7_W2_P5, F.Cu at (-24.1, -162.6)
- added C38: 100nF, Capacitors_ThroughHole:C_Rect_L7_W2_P5, F.Cu at (-34.9, -162.6)
- added C38: 100nF, Capacitors_ThroughHole:C_Rect_L7_W2_P5, F.Cu at (-45.7, -162.6)
- added C38: 100nF, Capacitors_ThroughHole:C_Rect_L7_W2_P5, F.Cu at (-13.3, -162.6)
- added C38: 100nF, Capacitors_ThroughHole:C_Rect_L7_W2_P5, F.Cu at (8.26, -162.6)
- added D5: DIODE, Discret:D3, F.Cu at (-51.4, -100.3)
- added D6: DIODE, Discret:D3, F.Cu at (-54.6, -100.3)
- added D7: DIODE, Discret:D3, F.Cu at (-9.53, -55.2)
- added D8: DIODE, Discret:D3, F.Cu at (-13.3, -55.2)
- added FB14: FILTER, Discret:R4, F.Cu at (-36.2, -111.8)
- added FB15: FILTER, Discret:R4, F.Cu at (-6.35, -111.8)
- added FB16: FILTER, Discret:R4, F.Cu at (8.89, -111.8)
- added FB17: FILTER, Discret:R4, F.Cu at (27.3, -68.6)
- added FB18: FILTER, Discret:R4, F.Cu at (26.7, -71.8)
- added FB19: FILTER, Discret:R4, F.Cu at (-3.81, -73.0)
- added FB20: FILTER, Discret:R4, F.Cu at (-15.2, -70.5)
- added FB21: FILTER, Discret:R4, F.Cu at (19.1, -163.8)
- added FB22: FILTER, Discret:R4, F.Cu at (19.1, -153.7)
- added FB7: FILTER, Discret:R4, F.Cu at (0.64, -152.4)
- added FB8: FILTER, Discret:R4, F.Cu at (-21.0, -152.4)
- added FB8: FILTER, Discret:R4, F.Cu at (-31.8, -152.4)
- added FB8: FILTER, Discret:R4, F.Cu at (-42.5, -152.4)
- added FB8: FILTER, Discret:R4, F.Cu at (-10.2, -152.4)
- added FB8: FILTER, Discret:R4, F.Cu at (11.4, -152.4)
- added FB9: FILTER, Discret:R4, F.Cu at (-51.4, -111.8)
- added P10: DIP05-2A72-21L, Housings_DIP:DIP-14_W7.62mm_LongPads, F.Cu at (-2.54, -106.7)
- added P11: DIP05-1A72-12L, Housings_DIP:DIP-14_W7.62mm_LongPads, F.Cu at (-17.8, -106.7)
- added P12: DIP05-2A72-21L, Housings_DIP:DIP-14_W7.62mm_LongPads, F.Cu at (-5.08, -61.6)
- added P13: DIP05-1A72-12L, Housings_DIP:DIP-14_W7.62mm_LongPads, F.Cu at (10.2, -61.6)
- added P14: DIP05-2A72-21L, Housings_DIP:DIP-14_W7.62mm_LongPads, F.Cu at (38.1, -61.6)
- added P15: DIP05-1A72-12L, Housings_DIP:DIP-14_W7.62mm_LongPads, F.Cu at (22.9, -61.6)
- added P16: CONN_4, Pin_Headers:Pin_Header_Straight_1x04, F.Cu at (-6.35, -162.6)
- added P16: CONN_4, Pin_Headers:Pin_Header_Straight_1x04, F.Cu at (-87.0, -126.4)
- added P17: CONN_02X04, Pin_Headers:Pin_Header_Straight_2x04, F.Cu at (-146.5, 72.3)
- added P19: CONN_01X03, Pin_Headers:Pin_Header_Straight_1x03, F.Cu at (-57.1, -92.7)
- added P20: CONN_01X03, Pin_Headers:Pin_Header_Straight_1x03, F.Cu at (-17.8, -48.9)
- added P3: CONN_4, Pin_Headers:Pin_Header_Straight_1x04, F.Cu at (-47.6, -114.3)
- added P4: CONN_4, Pin_Headers:Pin_Header_Straight_1x04, F.Cu at (-2.54, -114.3)
- added P45: CONN_4, Pin_Headers:Pin_Header_Straight_1x04, F.Cu at (-49.5, -162.6)
- added P45: CONN_4, Pin_Headers:Pin_Header_Straight_1x04, F.Cu at (-27.9, -162.6)
- added P45: CONN_4, Pin_Headers:Pin_Header_Straight_1x04, F.Cu at (-38.7, -162.6)
- added P45: CONN_4, Pin_Headers:Pin_Header_Straight_1x04, F.Cu at (-17.1, -162.6)
- added P45: CONN_4, Pin_Headers:Pin_Header_Straight_1x04, F.Cu at (4.45, -162.6)
- added P5: CONN_4, Pin_Headers:Pin_Header_Straight_1x04, F.Cu at (38.1, -68.6)
- added P6: CONN_4, Pin_Headers:Pin_Header_Straight_1x04, F.Cu at (2.54, -68.6)
- added P8: DIP05-2A72-21L, Housings_DIP:DIP-14_W7.62mm_LongPads, F.Cu at (-47.6, -106.7)
- added P9: DIP05-1A72-12L, Housings_DIP:DIP-14_W7.62mm_LongPads, F.Cu at (-32.4, -106.7)
- added Q6: Q_NJFET_DSG, TO_SOT_Packages_THT:TO-92_Inline_Wide, F.Cu at (-356.9, -164.5)
- added Q8: Q_NJFET_DSG, TO_SOT_Packages_THT:TO-92_Inline_Wide, F.Cu at (-356.2, -135.3)
- added R10: 12K, Discret:R4, F.Cu at (-99.7, -86.4)
- added R11: 2.2M, Discret:R1, F.Cu at (-370.8, -159.4)
- added R12: 2.2M, Discret:R1, F.Cu at (-369.6, -152.4)
- added R13: 3K, Discret:R4, F.Cu at (-352.4, -156.8)
- added R15: 100K, Discret:R1, F.Cu at (-348.0, -152.4)
- added R17: 10M, Discret:R1, F.Cu at (-365.8, -141.0)
- added R18: 2.2M, Discret:R1, F.Cu at (-370.8, -140.3)
- added R19: 2.2M, Discret:R1, F.Cu at (-369.6, -147.3)
- added R20: 3K, Discret:R4, F.Cu at (-352.4, -142.9)
- added R22: 100K, Discret:R1, F.Cu at (-348.0, -147.3)
- added R25: 12K, Discret:R1, F.Cu at (-115.6, -96.5)
- added R29: 10K, Discret:R4, F.Cu at (-118.1, -129.5)
- added R3: 10M, Discret:R1, F.Cu at (-365.1, -158.8)
- added R6: 12K, Discret:R1, F.Cu at (-115.6, -113.0)
- added R7: 12K, Discret:R4, F.Cu at (-113.7, -86.4)
- added R8: 12K, Discret:R1, F.Cu at (-117.5, -90.2)
- added R9: 12K, Discret:R4, F.Cu at (-96.5, -86.4)
- added buf_in1: CONN_4, Pin_Headers:Pin_Header_Straight_1x04, F.Cu at (-356.9, -153.7)
- added buf_out1: CONN_4, Pin_Headers:Pin_Header_Straight_1x04, F.Cu at (-344.2, -153.7)
- added buf_pwr1: CONN_4, Pin_Headers:Pin_Header_Straight_1x04, F.Cu at (-374.0, -146.1)
- added eq7_1: CONN_4, Pin_Headers:Pin_Header_Straight_1x04, F.Cu at (-87.0, -107.3)
- added eq7_1: CONN_4, Pin_Headers:Pin_Header_Straight_1x04, F.Cu at (-109.9, -33.0)
- added eq7_2: CONN_4, Pin_Headers:Pin_Header_Straight_1x04, F.Cu at (-87.0, -95.2)
- added eq7_2: CONN_4, Pin_Headers:Pin_Header_Straight_1x04, F.Cu at (-122.6, -38.7)
- added j_pwr1: CONN_2, Pin_Headers:Pin_Header_Straight_1x02, F.Cu at (-368.3, -54.6)
- added motor_ctrl1: CONN_4, Pin_Headers:Pin_Header_Straight_1x04, F.Cu at (-374.6, -59.1)
- added mute1: CONN_01X04, Pin_Headers:Pin_Header_Straight_1x04, F.Cu at (-379.7, -55.9)
- added pwr_motor1: CONN_2, Connect:bornier2, F.Cu at (-365.8, -74.3)
- added rid_out1: CONN_4, Pin_Headers:Pin_Header_Straight_1x04, F.Cu at (29.2, -38.1)
- added rid_out1: CONN_4, Pin_Headers:Pin_Header_Straight_1x04, F.Cu at (24.8, -38.1)
- added rid_out1: CONN_4, Pin_Headers:Pin_Header_Straight_1x04, F.Cu at (20.3, -38.1)
- added rid_out1: CONN_4, Pin_Headers:Pin_Header_Straight_1x04, F.Cu at (8.89, -102.2)
- P18: value CONN_02X04 -> CONN_01X02; footprint Pin_Headers:Pin_Header_Straight_2x04 -> Pin_Headers:Pin_Header_Straight_1x02
- moved FB13 255.2 mm to (-68.6, -25.4)
- moved D4 255.2 mm to (-53.3, -41.3)
- moved FB12 255.2 mm to (-69.2, -41.3)
- moved P7 255.2 mm to (-45.7, -37.5)
- moved mute_in1 255.2 mm to (-73.7, -37.5)
- moved P26 255.2 mm to (-52.1, -45.1)
- moved amp_out1 255.2 mm to (-78.1, -37.5)
- moved J2 220.4 mm to (-175.3, -147.3), turned to 180 degrees
- moved D12 173.8 mm to (-62.2, 3.17)
- moved P21 173.8 mm to (-65.4, 12.1)
- moved P22 173.8 mm to (-47.0, 12.1)
- moved P25 173.8 mm to (-58.4, 4.45)
- moved pre_buf_in1 173.8 mm to (-63.5, -8.26)
- moved pre_buf_out1 173.8 mm to (-64.1, 17.1)
- moved pre_buf_out2 173.8 mm to (-64.1, 21.6)
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Connections:
- J1 pad 1: /5V -> Net-(J1-Pad1)
- J1 pad 12: /CH3 -> /PREAMP
- J1 pad 15: /MOT_R -> /CH3
- J1 pad 16: /MOT_EN -> /CH4
- J1 pad 17: /MOT_L -> /IR_IN
- J1 pad 18: /EQ7_STROBE -> /EQ7_RST
- J1 pad 19: /EQ7_RST -> /EQ7_STROBE
- J1 pad 23: /EQ7_DATA_L -> /EQ7_DATA_R
- J1 pad 24: /EQ7_DATA_R -> /EQ7_DATA_L
- J1 pad 3: /SPK_MUTE_EN -> /PREAMP_PWR_EN
- J1 pad 6: /IR_IN -> /MUTE
- J2 pad 2: /SCL -> /SCL_OUT
- J2 pad 5: /SDA -> /SDA_OUT
- P18 pad 1: GND -> /SCL_OUT
- P18 pad 2: /5V -> /SDA_OUT
- P23 pad 1: /5V -> /CH1_EN
- P23 pad 2: /CH1_EN -> /5V
- P24 pad 2: /CH4_EN -> /5V
- P24 pad 3: /5V -> /CH4_EN
- P30 pad 1: /12V -> (no net)
- P34 pad 1: /PREAMP -> /PREAMP_PWR_EN
Routing:
- net /L_OUT: track 125.5 -> 246.8 mm, vias 0 -> 3
- net /5V: track 771.1 -> 654.1 mm
- net /R_OUT: track 94.4 -> 197.6 mm, vias 0 -> 4
- net +9V: track 181.9 -> 247.3 mm
- net /EQ7_STROBE: track 105.2 -> 43.2 mm
- net /VIN_MOTOR: track 56.5 -> 0.00 mm
- net /CH2_EN: track 46.4 -> 102.6 mm
- net /EQ7_RST: track 103.4 -> 48.7 mm
- net /SCL: track 22.1 -> 70.8 mm
- net /SDA: track 32.1 -> 80.5 mm
- net Net-(C38-Pad2): track 0.00 -> 34.9 mm
- net /MOTOUT_R: track 34.7 -> 0.00 mm
- net /MOTOUT_L: track 34.7 -> 0.00 mm
- net /MOT_EN: track 33.9 -> 0.00 mm
- net Net-(C2-Pad1): track 56.0 -> 23.7 mm
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Other:
- board size 367 x 249.6 mm -> 403.2 x 343.9 mm
- net class Default: via_dia 0.889 -> 1.3; via_drill 0.635 -> 0.8
- net class small added: clearance 0.5, trace_width 0.5, via_dia 0.889, via_drill 0.635

Commit message: updates,rc_car
Parts:
- moved 12V_AUX1 87.2 mm to (-202.6, -143.5)
- moved D5 46.4 mm to (-5.08, -97.8)
- moved FB14 46.4 mm to (10.2, -109.2)
- moved FB15 46.4 mm to (40.0, -109.2)
- moved FB9 46.4 mm to (-5.08, -109.2)
- moved P11 46.4 mm to (28.6, -104.1)
- moved D6 46.4 mm to (-8.26, -97.8)
- moved FB16 46.4 mm to (55.2, -109.2)
- moved P10 46.4 mm to (43.8, -104.1)
- moved P19 46.4 mm to (-10.8, -90.2)
- moved P3 46.4 mm to (-1.27, -111.8)
- moved P4 46.4 mm to (43.8, -111.8)
- moved P8 46.4 mm to (-1.27, -104.1)
- moved P9 46.4 mm to (14.0, -104.1)
- moved rid_out1 46.4 mm to (55.2, -99.7)
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Routing:
- net /PREAMP_EN: track 27.6 -> 28.9 mm
- net /5V: track 654.1 -> 655.4 mm
Other:
- board size 403.2 x 343.9 mm -> 434.3 x 343.9 mm

Commit message: fixes
Parts:
- removed the C38 at (-45.7, -162.6)
- removed the FB6 at (-270.2, -268.3)
- removed the FB6 at (-261.9, -219.4)
- removed the FB8 at (-21.0, -152.4)
- removed the FB8 at (-31.8, -152.4)
- removed the FB8 at (-42.5, -152.4)
- removed the FB8 at (-10.2, -152.4)
- removed the FB8 at (11.4, -152.4)
- removed the P45 at (-49.5, -162.6)
- added FB6: FILTER, Discret:R5, F.Cu at (-270.2, -268.3)
- added FB6: FILTER, Discret:R5, F.Cu at (-261.9, -219.4)
- added FB8: FILTER, Discret:R5, F.Cu at (-235.8, -104.9)
- added FB8: FILTER, Discret:R5, F.Cu at (-235.8, -94.1)
- added FB8: FILTER, Discret:R5, F.Cu at (-235.8, -115.7)
- added FB8: FILTER, Discret:R5, F.Cu at (-235.8, -136.8)
- added P46: CONN_01X04, Pin_Headers:Pin_Header_Straight_1x04, F.Cu at (-258.1, -127.8)
- added REF**: TO3, TO_SOT_Packages_THT:TO3, F.Cu at (-542.3, -154.3)
- FB1, FB10, FB11, FB12, FB13, FB14, FB15, FB16, FB17, FB18, FB19, FB2, FB20, FB21, FB22, FB3, FB4, FB5, FB7, FB9: footprint Discret:R4 -> Discret:R5
- P21, P22: value DIP05-2A72-21L -> DIP051C9051L
- P35, P36: value CONN_01X03 -> CONN_01X04; footprint Pin_Headers:Pin_Header_Straight_1x03 -> Pin_Headers:Pin_Header_Straight_1x04
- R8: footprint Discret:R1 -> Discret:R4
- moved FB19 490.2 mm to (-477.1, 54.6)
- moved P12 490.2 mm to (-478.4, 66.0)
- moved P13 490.2 mm to (-463.2, 66.0)
- moved P14 490.2 mm to (-435.2, 66.0)
- moved P15 490.2 mm to (-450.5, 66.0)
- moved P20 490.2 mm to (-491.1, 78.7)
- moved FB20 490.2 mm to (-488.6, 57.1)
- moved P5 490.2 mm to (-435.2, 59.1)
- moved P6 490.2 mm to (-470.8, 59.1)
- moved rid_out1 490.2 mm to (-444.1, 89.5)
- moved rid_out1 490.2 mm to (-448.6, 89.5)
- moved rid_out1 490.2 mm to (-453.0, 89.5)
- moved FB17 483.4 mm to (-438.8, 59.7), turned to 270 degrees
- moved FB18 469.5 mm to (-424.1, 59.7), turned to 270 degrees
- moved P16 366.9 mm to (-414.5, -13.2)
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Connections:
- J1 pad 12: /PREAMP -> /IR_IN
- J1 pad 13: /CH2 -> /CH1
- J1 pad 14: /CH1 -> /CH2
- J1 pad 15: /CH3 -> /CH4
- J1 pad 16: /CH4 -> /CH3
- J1 pad 3: /PREAMP_PWR_EN -> (no net)
- P10 pad 1: /L_IN2 -> /R_IN2
- P10 pad 14: /R_IN2 -> /L_IN2
- P10 pad 7: /L_OUT -> /R_OUT
- P10 pad 8: /R_OUT -> /L_OUT
- P35 pad 1: /5V -> GND
- P35 pad 3: /TEMP_R -> GND
- P36 pad 2: GND -> /5V
- P36 pad 3: /TEMP_L -> /5V
Routing:
- net /CH3_EN: track 62.9 -> 98.3 mm
- net /12V: track 399.9 -> 427.9 mm
- net /5V: track 655.4 -> 633.0 mm, vias 0 -> 6
- net /G_IN3: track 35.7 -> 54.5 mm
- net /SDA: track 80.5 -> 66.0 mm
- net /SCL: track 70.8 -> 59.7 mm
- net Net-(C9-Pad1): track 9.79 -> 20.0 mm
- net Net-(FB3-Pad2): track 15.8 -> 6.42 mm
- net /EQ7_DATA_R: track 23.7 -> 14.9 mm
- net /EQ7_DATA_L: track 44.7 -> 35.9 mm
- net /L_OUT: track 246.8 -> 238.2 mm
- net /EQ7_STROBE: track 43.2 -> 34.9 mm
- net /R_OUT_BUF2: track 27.5 -> 35.1 mm
- net Net-(FB17-Pad1): track 0.00 -> 7.19 mm
- net Net-(FB18-Pad1): track 0.00 -> 7.19 mm
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Other:
- board size 434.3 x 343.9 mm -> 365.4 x 458 mm
- net class pwr: via_dia 0.889 -> 1.5; via_drill 0.635 -> 1
