File: v2/amp_box/power_ctrl/power_ctrl.sch (KiCad schematic (older format))
At the start: 159 parts, among them IC1 L293D, J1 Atmega328, J2 RJ12, P1 Msgeq7_1, P10 DIP05-2A72-21L, P11 DIP05-1A72-12L, P12 DIP05-2A72-21L, P13 DIP05-1A72-12L, P14 DIP05-2A72-21L, P15 DIP05-1A72-12L, P16 CONN_4, P17 CONN_02X04, P18 CONN_02X04, P19 CONN_01X03, P2 Msgeq7_1, P20 CONN_01X03, P21 DIP05-2A72-21L, P22 DIP05-2A72-21L, P23 CONN_01X03, P24 CONN_01X03, P25 CONN_01X02, P26 CONN_01X02, P27 CONN_01X02, P28 CONN_01X02, P29 CONN_01X02, P3 CONN_4, P30 CONN_01X02, P31 CONN_01X02, P32 CONN_01X02, P33 CONN_01X02, P34 CONN_01X02, P35 CONN_01X03, P36 CONN_01X03, P4 CONN_4, P5 CONN_4, P6 CONN_4, P7 DIP05-2A72-21L, P8 DIP05-2A72-21L, P9 DIP05-1A72-12L, Q1 BC547, Q10 BC547, Q11 BC547, Q12 Q_PMOS_GDS, Q2 BC547, Q3 BC547, Q4 BC547, Q5 BC547, Q6 Q_NJFET_DSG, Q7 Q_NJFET_DSG, Q8 Q_NJFET_DSG, Q9 Q_NJFET_DSG, U1 7805, U2 7809

Commit message: updates
Parts:
- added P37, P38, P39, P40, P41, P42, P43, P44: CONN_2, Connect:bornier2, symbol CONN_2
- C15, C16, C26, C27: value 1uF -> 4.7uF
- R13, R14, R20, R21: value 10K -> 3K
Connections:
- net 12V: now also P37.1 (P1), P38.1 (P1), P39.1 (P1), P40.1 (P1), P41.1 (P1), P42.1 (P1), P43.1 (P1), P44.1 (P1)
- net GND: now also P37.2 (PM), P38.2 (PM), P39.2 (PM), P40.2 (PM), P41.2 (PM), P42.2 (PM), P43.2 (PM), P44.2 (PM)
Other:
- moved on the sheet: D12, P21, P22, Q10, R25

Commit message: updates
Parts:
- removed C10, C11, C12, C34: 100n, Capacitors_ThroughHole:C_Rect_L7_W2_P5, symbol C
- removed IC1: L293D, Housings_DIP:DIP-16_W7.62mm_LongPads, symbol L293D
- removed P18: CONN_02X04, Pin_Headers:Pin_Header_Straight_2x04, symbol CONN_02X04
- added C37, C38: 100nF, Capacitors_ThroughHole:C_Rect_L7_W2_P5, symbol C
- added FB14, FB15, FB16, FB17, FB18, FB19, FB20, FB21, FB22, FB7, FB8, FB9: FILTER, Discret:R4, symbol FILTER
- added P18: CONN_01X02, Pin_Headers:Pin_Header_Straight_1x02, symbol CONN_01X02
- added P45, eq7_1, eq7_2: CONN_4, Pin_Headers:Pin_Header_Straight_1x04, symbol CONN_4
- added R29: 10K, Discret:R4, symbol R-RESCUE-selector_ctrl
- D11, D3: symbol LED -> LED-RESCUE-power_ctrl
- R10, R7, R9: footprint Discret:R1 -> Discret:R4
- R25, R6: footprint Discret:R4 -> Discret:R1
Connections:
- net MOT_EN is gone; now on net CH4: J1.16
- net MOT_L is gone; now on net IR_IN: J1.17
- net MOT_R is gone; now on net CH3: J1.15
- net 12V: no longer P30.1 (P1)
- net 5V: now also P23.2 (P2), P24.2 (P2), FB7.2, FB8.2, R29.1, eq7_1.4 (P4); no longer J1.1, P16.3 (P3), P23.1 (P1), P24.3 (P3)
- net CH1_EN: now also P19.3 (P3), P23.1 (P1); no longer P19.2 (P2), P23.2 (P2)
- net CH2_EN: now also P19.2 (P2); no longer P19.3 (P3)
- net CH3: no longer J1.12
- net CH3_EN: now also P20.2 (P2); no longer P20.1 (P1)
- net CH4: no longer J1.11
- net CH4_EN: now also P20.1 (P1), P24.3 (P3); no longer P20.2 (P2), P24.2 (P2)
- net EQ7_DATA_L: now also J1.24, eq7_1.2 (P2); no longer J1.23
- net EQ7_DATA_R: now also J1.23, eq7_1.1 (P1); no longer J1.24
- net EQ7_RST: now also J1.18, eq7_2.2 (P2); no longer J1.19
- net EQ7_STROBE: now also J1.19, eq7_2.4 (P4); no longer J1.18
- net GND: now also C37.1, C38.1, P45.2 (P2), eq7_1.3 (P3), eq7_2.1 (P1), eq7_2.3 (P3)
- net IR_IN: no longer J1.6
- net L_IN1: now also FB9.2; no longer P3.1 (P1)
- net L_IN2: now also FB15.2; no longer P4.1 (P1)
- net L_IN3: now also FB17.2; no longer P5.1 (P1)
- net L_IN4: now also FB19.2; no longer P6.1 (P1)
- net MUTE: now also J1.6; no longer J1.5
- net PREAMP: now also J1.12; no longer J1.4, P34.1 (P1)
- net R_IN1: now also FB14.2; no longer P3.4 (P4)
- net R_IN2: now also FB16.2; no longer P4.4 (P4)
- net R_IN3: now also FB18.2; no longer P5.4 (P4)
- net R_IN4: now also FB20.2; no longer P6.4 (P4)
- net SCL: now also FB21.2, P45.1 (P1); no longer J2.2
- net SDA: now also FB22.1, P45.4 (P4); no longer J2.5
- net SPK_MUTE_EN: no longer J1.3
- new net: J1.1, R29.2
- new net: FB17.1, P5.1 (P1)
- new net: FB18.1, P5.4 (P4)
- new net: FB19.1, P6.1 (P1)
- new net: FB20.1, P6.4 (P4)
- new net: FB9.1, P3.1 (P1)
- new net: FB14.1, P3.4 (P4)
- new net: FB15.1, P4.1 (P1)
- new net: FB16.1, P4.4 (P4)
- new net: C37.2, FB7.1, P16.3 (P3)
- new net: C38.2, FB8.1, P45.3 (P3)
- new net 9V: P30.1 (P1)
- new net PREAMP_PWR_EN: J1.3, P34.1 (P1)
- new net SCL_OUT: FB21.1, J2.2, P18.1 (P1)
- new net SDA_OUT: FB22.2, J2.5, P18.2 (P2)
- no-connect marks 104 -> 105
Other:
- note added: "for IR receiver \nTSOP31238"
- moved on the sheet: C13, C18, C19, C20, C21, C22, C23, C24, C25, FB10, FB11, P1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

Commit message: updates,rc_car
Parts:
- P21, P22: value DIP05-2A72-21L -> DIP051C9051L
Changed lines of the file:
@@
 P 15100 26000
 F 0 "P21" H 15100 26400 60  0000 C CNN
-F 1 "DIP05-2A72-21L" V 15100 26000 50  0000 C CNN
+F 1 "DIP051C9051L" V 15100 26000 50  0000 C CNN
 F 2 "Housings_DIP:DIP-14_W7.62mm_LongPads" H 15100 26000 60  0001 C CNN
 F 3 "~" H 15100 26000 60  0000 C CNN
@@
 P 17800 25900
 F 0 "P22" H 17800 26300 60  0000 C CNN
-F 1 "DIP05-2A72-21L" V 17800 25900 50  0000 C CNN
+F 1 "DIP051C9051L" V 17800 25900 50  0000 C CNN
 F 2 "Housings_DIP:DIP-14_W7.62mm_LongPads" H 17800 25900 60  0001 C CNN
 F 3 "~" H 17800 25900 60  0000 C CNN

Commit message: fixes
Parts:
- removed P35, P36: CONN_01X03, Pin_Headers:Pin_Header_Straight_1x03, symbol CONN_01X03
- added P35, P36, P46: CONN_01X04, Pin_Headers:Pin_Header_Straight_1x04, symbol CONN_01X04
- FB1, FB10, FB11, FB12, FB13, FB14, FB15, FB16, FB17, FB18, FB19, FB2, FB20, FB21, FB22, FB3, FB4, FB5, FB6, FB7, FB8, FB9: footprint Discret:R4 -> Discret:R5
- R8: footprint Discret:R1 -> Discret:R4
Connections:
- net 5V: now also P36.1 (P1), P36.2 (P2), P36.3 (P3), P36.4 (P4)
- net CH1: now also J1.13; no longer J1.14
- net CH2: now also J1.14; no longer J1.13
- net CH3: now also J1.16; no longer J1.15
- net CH4: now also J1.15; no longer J1.16
- net EQ7_DATA_L: now also P46.3 (P3)
- net EQ7_DATA_R: now also P46.4 (P4)
- net GND: now also P35.1 (P1), P35.2 (P2), P35.3 (P3), P35.4 (P4)
- net IR_IN: now also J1.12; no longer J1.17
- net L_IN2: now also P10.14; no longer P10.1
- net L_OUT: now also P10.8; no longer P10.7
- net PREAMP: now also J1.5; no longer J1.12
- net PREAMP_PWR_EN: now also J1.4; no longer J1.3
- net R_IN2: now also P10.1; no longer P10.14
- net R_OUT: now also P10.7; no longer P10.8
- net TEMP_L: now also P46.2 (P2)
- net TEMP_R: now also P46.1 (P1)
