File: rc_car/h_bridge-1/rc_car.sch (KiCad schematic (older format))
At the start: 37 parts, among them J1 CONN_01X06, J2 CONN_01X02, J3 CONN_01X02, J4 CONN_01X02, J5 CONN_01X02, J6 CONN_01X02, J7 CONN_01X02, J8 CONN_01X02, J9 CONN_01X02, Q10 IRLU024N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

Commit message: cleanups
Parts:
- D10, D9: symbol LED -> LED-RESCUE-rc_car
Changed lines of the file:
@@
 EESchema Schematic File Version 2
+LIBS:rc_car-rescue
 LIBS:power
 LIBS:device
@@
 $EndComp
 $Comp
-L LED D9
+L LED-RESCUE-rc_car D9
 U 1 1 595A1DB7
 P 4850 3350
@@
 $EndComp
 $Comp
-L LED D10
+L LED-RESCUE-rc_car D10
 U 1 1 595A1EBB
 P 4850 3550
