File: rc_car/h_bridge-1/rc_car.kicad_pcb (KiCad board)
At the start: 2 copper layers, 94.9 x 46.4 mm, 38 parts, among them J1 CONN_01X06, J2 CONN_01X02, J3 CONN_01X02, J4 CONN_01X02, J5 CONN_01X02, J6 CONN_01X02, J7 CONN_01X02, J8 CONN_01X02, J9 CONN_01X02, Q10 IRLU024N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

Commit message: updates
Parts:
- moved J4 143.5 mm to (18.4, 52.8)
- moved J6 143.5 mm to (46.4, 62.4)
- moved J9 143.5 mm to (31.2, 52.8)
- moved C2 143.5 mm to (24.4, 63.1)
- moved C2 143.5 mm to (38.0, 63.1)
- moved J5 143.5 mm to (16.0, 62.4)
- moved J7 143.5 mm to (43.9, 52.8)
- moved R6 126.0 mm to (17.4, 40.8)
- moved D1 126.0 mm to (24.1, 35.9)
- moved D2 126.0 mm to (26.4, 35.9)
- moved D5 126.0 mm to (10.5, 23.0)
- moved D8 126.0 mm to (43.4, 23.0)
- moved J3 126.0 mm to (41.9, 6.10)
- moved Q10 126.0 mm to (19.6, 27.3)
- moved Q14 126.0 mm to (43.4, 42.0)
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Routing:
- net /VIN_MOTOR: track 240.8 -> 138.9 mm
- net /M2_OUT_L: track 90.5 -> 91.3 mm
- net Net-(D1-Pad1): track 16.7 -> 17.3 mm
Other:
- board outline removed
- net class Default removed
- net class mot removed
- net class pwr removed
- rule pad_to_mask_clearance: 0.2 -> 0
