File: amp_v2/7805/7805.sch (KiCad schematic (older format))
At the start: 16 parts, among them U1 7805

Commit message: updates
Parts:
- C1, C10, C16: symbol CP1 -> 7805-rescue:CP1
- C13, C4, C7: symbol C -> 7805-rescue:C
- D1, D2: symbol DIODE -> 7805-rescue:DIODE
- D3: symbol LED -> 7805-rescue:LED
- PowerIn1, PowerOut1, PowerOut2, PowerOut3: symbol CONN_2 -> 7805-rescue:CONN_2
- R1, R4: symbol R -> 7805-rescue:R
- U1: symbol 7805 -> 7805-rescue:7805
Changed lines of the file:
@@
-EESchema Schematic File Version 2
-LIBS:power
-LIBS:device
-LIBS:transistors
-LIBS:conn
-LIBS:linear
-LIBS:regul
-LIBS:74xx
-LIBS:cmos4000
-LIBS:adc-dac
-LIBS:memory
-LIBS:xilinx
-LIBS:special
-LIBS:microcontrollers
-LIBS:dsp
-LIBS:microchip
-LIBS:analog_switches
-LIBS:motorola
-LIBS:texas
-LIBS:intel
-LIBS:audio
-LIBS:interface
-LIBS:digital-audio
-LIBS:philips
-LIBS:display
-LIBS:cypress
-LIBS:siliconi
-LIBS:opto
-LIBS:atmel
-LIBS:contrib
-LIBS:valves
-LIBS:7805-cache
-EELAYER 27 0
+EESchema Schematic File Version 4
+EELAYER 30 0
 EELAYER END
 $Descr A4 11693 8268
@@
 $EndDescr
 $Comp
-L R R4
+L 7805-rescue:R R4
 U 1 1 54773478
 P 8400 3850
@@
 $EndComp
 $Comp
-L LED D3
+L 7805-rescue:LED D3
 U 1 1 54773479
 P 8400 4400
@@
 	8400 4200 8400 4100
 $Comp
-L GND #PWR01
+L 7805-rescue:GND #PWR01
 U 1 1 5477347A
 P 8400 4700
@@
 	8400 3600 8400 3500
 $Comp
-L CONN_2 PowerIn1
+L 7805-rescue:CONN_2 PowerIn1
 U 1 1 5477349A
 P 1300 3700
@@
 $EndComp
 $Comp
-L CP1 C1
+L 7805-rescue:CP1 C1
 U 1 1 5477349B
 P 3250 3800
@@
 $EndComp
 $Comp
-L 7805 U1
+L 7805-rescue:7805 U1
 U 1 1 5477349D
 P 4150 3650
@@
 $EndComp
 Wire Wire Line
-	2300 3600 3750 3600
-$Comp
-L CP1 C16
+	2300 3600 3250 3600
+$Comp
+L 7805-rescue:CP1 C16
 U 1 1 5477349F
 P 6300 3800
@@
 $EndComp
 $Comp
-L C C4
+L 7805-rescue:C C4
 U 1 1 547734A0
 P 3550 3800
@@
 	3550 4200 3550 4000
 Wire Wire Line
-	2800 4200 6750 4200
+	2800 4200 3250 4200
 Wire Wire Line
 	3250 4200 3250 4000
@@
 Connection ~ 4150 4200
 $Comp
-L CP1 C10
+L 7805-rescue:CP1 C10
 U 1 1 547734A1
 P 5000 3800
@@
 $EndComp
 $Comp
-L C C7
+L 7805-rescue:C C7
 U 1 1 547734A2
 P 4700 3800
@@
 Connection ~ 5000 3600
 $Comp
-L DIODE D2
+L 7805-rescue:DIODE D2
 U 1 1 5477284F
 P 4150 3250
@@
 	3750 3250 3750 3600
 $Comp
-L DIODE D1
+L 7805-rescue:DIODE D1
 U 1 1 5477293E
 P 2100 3600
@@
 $EndComp
 $Comp
-L R R1
+L 7805-rescue:R R1
 U 1 1 54772B42
 P 5600 3600
@@
 $EndComp
 Wire Wire Line
-	4550 3600 5350 3600
-Wire Wire Line
-	5000 4000 5000 4650
-$Comp
-L C C13
+	4550 3600 4700 3600
+Wire Wire Line
+	5000 4000 5000 4200
+$Comp
+L 7805-rescue:C C13
 U 1 1 54772D2C
 P 5950 3800
@@
 $EndComp
 Wire Wire Line
-	5850 3600 7300 3600
+	5850 3600 5950 3600
 Wire Wire Line
 	5950 4200 5950 4000
@@
 	1900 3600 1650 3600
 Wire Wire Line
-	1650 3800 2800 3800
-Wire Wire Line
 	2800 3800 2800 4200
 Text Label 1800 3600 1    60   ~ 0
@@
 Wire Wire Line
 	6750 4200 6750 4300
-Connection ~ 1750 3800
-$Comp
-L GND #PWR02
+$Comp
+L 7805-rescue:GND #PWR02
 U 1 1 5477395B
 P 6750 4300
@@
 $EndComp
 $Comp
-L CONN_2 PowerOut1
+L 7805-rescue:CONN_2 PowerOut1
 U 1 1 547747D9
 P 7700 3700
@@
 $EndComp
 $Comp
-L GND #PWR03
+L 7805-rescue:GND #PWR03
 U 1 1 547747E0
 P 7800 4200
@@
 	7300 4050 7600 4050
 Wire Wire Line
-	7300 3500 7300 4050
+	7300 3500 7300 3600
 Connection ~ 7300 3600
-Connection ~ 8400 3500
 Wire Wire Line
 	5000 3600 5000 3300
@@
 	5000 4650 6250 4650
 $Comp
-L AGND #PWR04
+L 7805-rescue:AGND #PWR04
 U 1 1 54839ED0
 P 6250 4700
@@
 AVCC
 $Comp
-L CONN_2 PowerOut2
+L 7805-rescue:CONN_2 PowerOut2
 U 1 1 54839FB8
 P 9250 3550
@@
 AVCC
 $Comp
-L AGND #PWR05
+L 7805-rescue:AGND #PWR05
 U 1 1 5483A0E6
 P 10000 4000
@@
 	9150 4050 9150 3900
 $Comp
-L CONN_2 PowerOut3
+L 7805-rescue:CONN_2 PowerOut3
 U 1 1 5483A362
 P 9850 3500
@@
 	9150 3900 9350 3900
 Wire Wire Line
-	9750 3850 10000 3850
+	9750 3850 9950 3850
 Wire Wire Line
 	10000 3850 10000 4000
 Connection ~ 9950 3850
+Wire Wire Line
+	3550 3600 3750 3600
+Wire Wire Line
+	3250 3600 3550 3600
+Wire Wire Line
+	3550 4200 4150 4200
+Wire Wire Line
+	4150 4200 4700 4200
+Wire Wire Line
+	4700 3600 5000 3600
+Wire Wire Line
+	4700 4200 5000 4200
+Wire Wire Line
+	5000 3600 5350 3600
+Wire Wire Line
+	5000 4200 5000 4650
+Wire Wire Line
+	5000 4200 5950 4200
+Wire Wire Line
+	5950 3600 6300 3600
+Wire Wire Line
+	5950 4200 6300 4200
+Wire Wire Line
+	3250 4200 3550 4200
+Wire Wire Line
+	6300 3600 7300 3600
+Wire Wire Line
+	6300 4200 6750 4200
+Wire Wire Line
+	7300 3600 7300 4050
+Wire Wire Line
+	9950 3850 10000 3850
+Wire Wire Line
+	1650 3800 2800 3800
 $EndSCHEMATC
