File: amp_v2/amp_box/power_ctrl/power_ctrl.kicad_pcb (KiCad board)
At the start: 2 copper layers, 365.4 x 458 mm, 253 parts, among them J1 Atmega328, J2 RJ12, P1 Msgeq7_1, P10 DIP05-2A72-21L, P11 DIP05-1A72-12L, P12 DIP05-2A72-21L, P13 DIP05-1A72-12L, P14 DIP05-2A72-21L, P15 DIP05-1A72-12L, P16 CONN_4, P17 CONN_02X04, P18 CONN_01X02, P19 CONN_01X03, P2 Msgeq7_1, P20 CONN_01X03, P21 DIP051C9051L, P22 DIP051C9051L, P23 CONN_01X03, P24 CONN_01X03, P25 CONN_01X02, P26 CONN_01X02, P27 CONN_01X02, P28 CONN_01X02, P29 CONN_01X02, P3 CONN_4, P30 CONN_01X02, P31 CONN_01X02, P32 CONN_01X02, P33 CONN_01X02, P34 CONN_01X02, P35 CONN_01X04, P36 CONN_01X04, P37 CONN_2, P38 CONN_2, P39 CONN_2, P4 CONN_4, P40 CONN_2, P41 CONN_2, P42 CONN_2, P43 CONN_2, P44 CONN_2, P45 CONN_4, P46 CONN_01X04, P5 CONN_4, P6 CONN_4, P7 DIP05-2A72-21L, P8 DIP05-2A72-21L, P9 DIP05-1A72-12L, Q1 BC547, Q10 BC547, Q11 BC547, Q12 Q_PMOS_GDS, Q2 BC547, Q3 BC547, Q4 BC547, Q5 BC547, Q6 Q_NJFET_DSG, Q7 Q_NJFET_DSG, Q8 Q_NJFET_DSG, Q9 Q_NJFET_DSG, U1 7805, U2 7809

Commit message: updates
Parts:
- removed the buf_in1 at (-358.1, -107.3)
- added REF**: JST_XH_B4B-XH-A_1x04_P2.50mm_Vertical, Connector_JST:JST_XH_B4B-XH-A_1x04_P2.50mm_Vertical, F.Cu at (-386.5, -96.0)
Other:
- net class Default removed
- net class pwr removed
- net class pwr12 removed
- net class small removed
