File: amp_v2/car_box/filters_dc/power_amp.sch (KiCad schematic (older format))
At the start: 12 parts

Commit message: updates
Parts:
- C10, C11, C13, C8: symbol CP1 -> power_amp-rescue:CP1
- C12, C14, C7, C9: symbol C -> power_amp-rescue:C
- DC_IN1, DC_OUT1: symbol CONN_3 -> power_amp-rescue:CONN_3
- F1, F3: symbol FUSE -> power_amp-rescue:FUSE
Changed lines of the file:
@@
-EESchema Schematic File Version 2
-LIBS:power
-LIBS:device
-LIBS:transistors
-LIBS:conn
-LIBS:linear
-LIBS:regul
-LIBS:74xx
-LIBS:cmos4000
-LIBS:adc-dac
-LIBS:memory
-LIBS:xilinx
-LIBS:special
-LIBS:microcontrollers
-LIBS:dsp
-LIBS:microchip
-LIBS:analog_switches
-LIBS:motorola
-LIBS:texas
-LIBS:intel
-LIBS:audio
-LIBS:interface
-LIBS:digital-audio
-LIBS:philips
-LIBS:display
-LIBS:cypress
-LIBS:siliconi
-LIBS:opto
-LIBS:atmel
-LIBS:contrib
-LIBS:valves
-LIBS:power_amp-cache
-EELAYER 27 0
+EESchema Schematic File Version 4
+EELAYER 30 0
 EELAYER END
 $Descr A4 11693 8268
@@
 $EndDescr
 $Comp
-L CONN_3 DC_IN1
+L power_amp-rescue:CONN_3 DC_IN1
 U 1 1 52497BBA
 P 4800 3750
@@
 $EndComp
 $Comp
-L CP1 C8
+L power_amp-rescue:CP1 C8
 U 1 1 52497D8D
 P 2250 3200
@@
 $EndComp
 $Comp
-L CP1 C10
+L power_amp-rescue:CP1 C10
 U 1 1 52497D9A
 P 3100 4300
@@
 $EndComp
 $Comp
-L C C7
+L power_amp-rescue:C C7
 U 1 1 52497DB4
 P 2550 3200
@@
 $EndComp
 $Comp
-L CONN_3 DC_OUT1
+L power_amp-rescue:CONN_3 DC_OUT1
 U 1 1 5249832A
 P 950 3750
@@
 $EndComp
 $Comp
-L FUSE F1
+L power_amp-rescue:FUSE F1
 U 1 1 52507074
 P 4450 3200
@@
 $EndComp
 $Comp
-L FUSE F3
+L power_amp-rescue:FUSE F3
 U 1 1 52507087
 P 4450 4300
@@
 $EndComp
 $Comp
-L CP1 C13
+L power_amp-rescue:CP1 C13
 U 1 1 5262630B
 P 3100 3200
@@
 $EndComp
 $Comp
-L C C14
+L power_amp-rescue:C C14
 U 1 1 52626311
 P 3400 3200
@@
 $EndComp
 $Comp
-L CP1 C11
+L power_amp-rescue:CP1 C11
 U 1 1 52626317
 P 2250 4300
@@
 $EndComp
 $Comp
-L C C9
+L power_amp-rescue:C C9
 U 1 1 52497DBA
 P 3400 4300
@@
 $EndComp
 $Comp
-L C C12
+L power_amp-rescue:C C12
 U 1 1 52626331
 P 2550 4300
@@
 $EndComp
 Wire Wire Line
-	2250 3000 2550 3000
+	2250 3000 2400 3000
 Connection ~ 2400 3000
 Wire Wire Line
@@
 	1450 3850 1450 4850
 Wire Wire Line
-	3100 3000 3400 3000
-Wire Wire Line
-	3100 3400 3400 3400
-Wire Wire Line
-	3100 4100 3400 4100
-Wire Wire Line
-	3100 4500 3400 4500
+	3100 3000 3250 3000
+Wire Wire Line
+	3100 3400 3250 3400
+Wire Wire Line
+	3100 4100 3250 4100
+Wire Wire Line
+	3100 4500 3250 4500
 Connection ~ 3250 3000
 Connection ~ 3250 3400
 Wire Wire Line
-	2250 4500 2550 4500
-Wire Wire Line
-	2250 4100 2550 4100
-Wire Wire Line
-	2250 3400 2550 3400
+	2250 4500 2400 4500
+Wire Wire Line
+	2250 4100 2400 4100
+Wire Wire Line
+	2250 3400 2400 3400
 Connection ~ 3250 4500
 Connection ~ 3250 4100
@@
 Connection ~ 2400 3400
 Wire Wire Line
-	3250 3400 3250 4100
-Wire Wire Line
-	2400 3400 2400 4100
+	3250 3400 3250 3750
+Wire Wire Line
+	2400 3400 2400 3750
 Connection ~ 3250 3750
 Connection ~ 2400 3750
@@
 Connection ~ 2400 2600
 Wire Wire Line
-	1450 4850 4450 4850
+	1450 4850 2400 4850
 Wire Wire Line
 	2400 4850 2400 4500
@@
 Connection ~ 3250 4850
 Wire Wire Line
-	1300 3750 4450 3750
+	1300 3750 2400 3750
 Wire Wire Line
 	1300 3850 1450 3850
@@
 	4450 2950 4450 2600
 Wire Wire Line
-	4450 2600 1450 2600
+	4450 2600 3250 2600
 Wire Wire Line
 	4450 4850 4450 4550
@@
 Wire Wire Line
 	4450 3850 4450 4050
+Wire Wire Line
+	2400 3000 2550 3000
+Wire Wire Line
+	3250 3000 3400 3000
+Wire Wire Line
+	3250 3400 3400 3400
+Wire Wire Line
+	3250 4500 3400 4500
+Wire Wire Line
+	3250 4100 3400 4100
+Wire Wire Line
+	2400 4100 2550 4100
+Wire Wire Line
+	2400 4500 2550 4500
+Wire Wire Line
+	2400 3400 2550 3400
+Wire Wire Line
+	3250 3750 3250 4100
+Wire Wire Line
+	3250 3750 4450 3750
+Wire Wire Line
+	2400 3750 2400 4100
+Wire Wire Line
+	2400 3750 3250 3750
+Wire Wire Line
+	3250 2600 2400 2600
+Wire Wire Line
+	2400 2600 1450 2600
+Wire Wire Line
+	2400 4850 3250 4850
+Wire Wire Line
+	3250 4850 4450 4850
 $EndSCHEMATC
