File: amp_v2/i2c_conn/i2c_conn.kicad_pcb (KiCad board)
At the start: 2 copper layers, 15 x 18.7 mm, 5 parts, among them J1 RJ12, P1 CONN_2, P2 CONN_2, P3 CONN_2, P4 CONN_2

Commit message: updates
Other:
- net class Default removed
- net class pwr removed
