File: amp_v2/power_box/soft_start/soft_start.sch (KiCad schematic (older format))
At the start: 26 parts, among them K1 CONN_3, P1 CONN_2, P2 CONN_2, P3 CONN_2, P4 CONN_2, P5 CONN_2, P6 CONN_2, P7 CONN_2, P8 CONN_2, Q1 BC547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

Commit message: updates
Parts:
- D1, D2, D3: symbol DIODE -> soft_start-rescue:DIODE
- K1: symbol CONN_3 -> soft_start-rescue:CONN_3
- P1, P2, P3, P4, P5, P6, P7, P8, R_A1, R_B1: symbol CONN_2 -> soft_start-rescue:CONN_2
- Q1, Q2, Q3: symbol BC547 -> soft_start-rescue:BC547
- R1, R2, R3, R4, R5, R6: symbol R-RESCUE-soft_start -> soft_start-rescue:R-RESCUE-soft_start
- RLY1, RLY2, RLY3: symbol RELAY_HJR-3FF_Z -> soft_start-rescue:RELAY_HJR-3FF_Z
Changed lines of the file:
@@
-EESchema Schematic File Version 2
-LIBS:soft_start-rescue
-LIBS:power
-LIBS:device
-LIBS:transistors
-LIBS:conn
-LIBS:linear
-LIBS:regul
-LIBS:74xx
-LIBS:cmos4000
-LIBS:adc-dac
-LIBS:memory
-LIBS:xilinx
-LIBS:special
-LIBS:microcontrollers
-LIBS:dsp
-LIBS:microchip
-LIBS:analog_switches
-LIBS:motorola
-LIBS:texas
-LIBS:intel
-LIBS:audio
-LIBS:interface
-LIBS:digital-audio
-LIBS:philips
-LIBS:display
-LIBS:cypress
-LIBS:siliconi
-LIBS:opto
-LIBS:atmel
-LIBS:contrib
-LIBS:valves
-LIBS:w_relay
-LIBS:soft_start-cache
-EELAYER 25 0
+EESchema Schematic File Version 4
+EELAYER 30 0
 EELAYER END
 $Descr A4 11693 8268
@@
 $EndDescr
 $Comp
-L RELAY_HJR-3FF_Z RLY1
+L soft_start-rescue:RELAY_HJR-3FF_Z RLY1
 U 1 1 53943E62
 P 2100 2250
@@
 $EndComp
 $Comp
-L RELAY_HJR-3FF_Z RLY2
+L soft_start-rescue:RELAY_HJR-3FF_Z RLY2
 U 1 1 53943E92
 P 2050 3700
@@
 $EndComp
 $Comp
-L DIODE D2
+L soft_start-rescue:DIODE D2
 U 1 1 53943E9A
 P 2800 2250
@@
 $EndComp
 $Comp
-L DIODE D1
+L soft_start-rescue:DIODE D1
 U 1 1 53943EA7
 P 2700 3700
@@
 Connection ~ 2700 3500
 $Comp
-L BC547 Q1
+L soft_start-rescue:BC547 Q1
 U 1 1 53943EBF
 P 3250 3800
@@
 $EndComp
 $Comp
-L BC547 Q2
+L soft_start-rescue:BC547 Q2
 U 1 1 53943ECC
 P 3250 2350
@@
 $EndComp
 $Comp
-L GND-RESCUE-soft_start #PWR2
+L soft_start-rescue:GND-RESCUE-soft_start #PWR2
 U 1 1 53943F3B
 P 3150 2650
@@
 $EndComp
 $Comp
-L GND-RESCUE-soft_start #PWR3
+L soft_start-rescue:GND-RESCUE-soft_start #PWR3
 U 1 1 53943F48
 P 3150 4100
@@
 EN_2
 $Comp
-L R-RESCUE-soft_start R1
+L soft_start-rescue:R-RESCUE-soft_start R1
 U 1 1 53944164
 P 3850 2350
@@
 $EndComp
 $Comp
-L R-RESCUE-soft_start R2
+L soft_start-rescue:R-RESCUE-soft_start R2
 U 1 1 53944171
 P 3850 3800
@@
 HOT_R
 $Comp
-L CONN_2 P1
+L soft_start-rescue:CONN_2 P1
 U 1 1 539443E8
 P 1250 1250
@@
 	900  1150 900  1600
 Wire Wire Line
-	900  1600 1350 1600
+	900  1600 1150 1600
 Connection ~ 1150 1600
 $Comp
-L CONN_2 P2
+L soft_start-rescue:CONN_2 P2
 U 1 1 53944432
 P 2200 1250
@@
 	1850 1150 1850 1600
 Wire Wire Line
-	1850 1600 2300 1600
+	1850 1600 2100 1600
 Connection ~ 2100 1600
 $Comp
-L CONN_2 P3
+L soft_start-rescue:CONN_2 P3
 U 1 1 539444AC
 P 3000 1250
@@
 	2650 1150 2650 1600
 Wire Wire Line
-	2650 1600 3100 1600
+	2650 1600 2900 1600
 Connection ~ 2900 1600
 Text Label 4900 2900 3    60   ~ 0
@@
 5V
 $Comp
-L GND-RESCUE-soft_start #PWR5
+L soft_start-rescue:GND-RESCUE-soft_start #PWR5
 U 1 1 5394462F
 P 4950 4950
@@
 	4950 4800 4950 4950
 $Comp
-L RELAY_HJR-3FF_Z RLY3
+L soft_start-rescue:RELAY_HJR-3FF_Z RLY3
 U 1 1 53FC72FF
 P 2000 5150
@@
 $EndComp
 $Comp
-L DIODE D3
+L soft_start-rescue:DIODE D3
 U 1 1 53FC7305
 P 2650 5150
@@
 $EndComp
 Wire Wire Line
-	2150 4950 2850 4950
+	2150 4950 2650 4950
 Wire Wire Line
 	2150 5350 2650 5350
 Connection ~ 2650 4950
 $Comp
-L BC547 Q3
+L soft_start-rescue:BC547 Q3
 U 1 1 53FC730E
 P 2750 5650
@@
 $EndComp
 $Comp
-L GND-RESCUE-soft_start #PWR1
+L soft_start-rescue:GND-RESCUE-soft_start #PWR1
 U 1 1 53FC7314
 P 2650 5950
@@
 EN_3
 $Comp
-L R-RESCUE-soft_start R3
+L soft_start-rescue:R-RESCUE-soft_start R3
 U 1 1 53FC7320
 P 3350 5650
@@
 	1450 2050 2000 2050
 Wire Wire Line
-	1950 2450 1950 3500
+	1950 2450 1950 2800
 Text Label 1650 2800 2    60   ~ 0
 L2
@@
 	3450 3800 3600 3800
 Wire Wire Line
-	1900 4950 1900 3900
+	1900 4950 1900 4550
 Wire Wire Line
 	1900 4550 1650 4550
@@
 	2950 5650 3100 5650
 $Comp
-L CONN_2 P4
+L soft_start-rescue:CONN_2 P4
 U 1 1 53FC7829
 P 5050 4450
@@
 	4700 2900 4700 2750
 $Comp
-L CONN_2 P5
+L soft_start-rescue:CONN_2 P5
 U 1 1 53FC7934
 P 3900 1250
@@
 	3550 1150 3550 1600
 Wire Wire Line
-	3550 1600 4000 1600
+	3550 1600 3800 1600
 Connection ~ 3800 1600
 Wire Wire Line
 	2700 3900 2700 4100
 Wire Wire Line
-	2200 3500 3150 3500
-$Comp
-L CONN_2 P6
+	2200 3500 2700 3500
+$Comp
+L soft_start-rescue:CONN_2 P6
 U 1 1 53FC7BD8
 P 4750 1250
@@
 	4400 1150 4400 1600
 Wire Wire Line
-	4400 1600 4850 1600
+	4400 1600 4650 1600
 Connection ~ 4650 1600
 Text Label 5600 2900 3    60   ~ 0
 5V
 $Comp
-L GND-RESCUE-soft_start #PWR6
+L soft_start-rescue:GND-RESCUE-soft_start #PWR6
 U 1 1 53FC8FA5
 P 5800 2900
@@
 	5800 2750 5800 2900
 $Comp
-L CONN_2 P8
+L soft_start-rescue:CONN_2 P8
 U 1 1 53FC8FAD
 P 5700 2400
@@
 $EndComp
 $Comp
-L CONN_3 K1
+L soft_start-rescue:CONN_3 K1
 U 1 1 53FC8FB9
 P 4800 2400
@@
 5V
 $Comp
-L GND-RESCUE-soft_start #PWR4
+L soft_start-rescue:GND-RESCUE-soft_start #PWR4
 U 1 1 53FC8FC7
 P 4800 2900
@@
 	4900 2750 4900 2900
 $Comp
-L CONN_2 P7
+L soft_start-rescue:CONN_2 P7
 U 1 1 53FC90C1
 P 4450 4300
@@
 	2800 2650 2750 2650
 $Comp
-L R-RESCUE-soft_start R4
+L soft_start-rescue:R-RESCUE-soft_start R4
 U 1 1 53FC9A1C
 P 8550 2250
@@
 $EndComp
 $Comp
-L R-RESCUE-soft_start R5
+L soft_start-rescue:R-RESCUE-soft_start R5
 U 1 1 53FC9A29
 P 8550 2500
@@
 $EndComp
 $Comp
-L R-RESCUE-soft_start R6
+L soft_start-rescue:R-RESCUE-soft_start R6
 U 1 1 53FC9A2F
 P 8550 2750
@@
 $EndComp
 Wire Wire Line
-	8300 2250 8300 2750
+	8300 2250 8300 2500
 Connection ~ 8300 2500
 Wire Wire Line
-	8800 2250 8800 2750
+	8800 2250 8800 2500
 Connection ~ 8800 2500
 Wire Wire Line
@@
 	8100 2500 8300 2500
 $Comp
-L CONN_2 R_A1
+L soft_start-rescue:CONN_2 R_A1
 U 1 1 53FC9CB3
 P 7750 2500
@@
 $EndComp
 $Comp
-L CONN_2 R_B1
+L soft_start-rescue:CONN_2 R_B1
 U 1 1 53FC9CB9
 P 9350 2500
@@
 $EndComp
 Wire Wire Line
-	8100 2400 8100 2600
+	8100 2400 8100 2500
 Connection ~ 8100 2500
 Wire Wire Line
-	9000 2400 9000 2600
+	9000 2400 9000 2500
 Connection ~ 9000 2500
+Wire Wire Line
+	2700 3500 3150 3500
+Wire Wire Line
+	1150 1600 1350 1600
+Wire Wire Line
+	2100 1600 2300 1600
+Wire Wire Line
+	2900 1600 3100 1600
+Wire Wire Line
+	2650 4950 2850 4950
+Wire Wire Line
+	1950 2800 1950 3500
+Wire Wire Line
+	1900 4550 1900 3900
+Wire Wire Line
+	3800 1600 4000 1600
+Wire Wire Line
+	4650 1600 4850 1600
+Wire Wire Line
+	8300 2500 8300 2750
+Wire Wire Line
+	8800 2500 8800 2750
+Wire Wire Line
+	8100 2500 8100 2600
+Wire Wire Line
+	9000 2500 9000 2600
 $EndSCHEMATC
