File: amp_v2/power_box_car/power_amp/power_amp.sch (KiCad schematic (older format))
At the start: 12 parts

Commit message: updates
Parts:
- C1, C12, C14, C2, C7, C9: symbol C -> power_amp-rescue:C
- C10, C11, C13, C8: symbol CP1 -> power_amp-rescue:CP1
- DCDC1, Power2: symbol CONN_3 -> power_amp-rescue:CONN_3
Changed lines of the file:
@@
-EESchema Schematic File Version 2
-LIBS:power
-LIBS:device
-LIBS:transistors
-LIBS:conn
-LIBS:linear
-LIBS:regul
-LIBS:74xx
-LIBS:cmos4000
-LIBS:adc-dac
-LIBS:memory
-LIBS:xilinx
-LIBS:special
-LIBS:microcontrollers
-LIBS:dsp
-LIBS:microchip
-LIBS:analog_switches
-LIBS:motorola
-LIBS:texas
-LIBS:intel
-LIBS:audio
-LIBS:interface
-LIBS:digital-audio
-LIBS:philips
-LIBS:display
-LIBS:cypress
-LIBS:siliconi
-LIBS:opto
-LIBS:atmel
-LIBS:contrib
-LIBS:valves
-LIBS:power_amp-cache
-EELAYER 27 0
+EESchema Schematic File Version 4
+EELAYER 30 0
 EELAYER END
 $Descr A4 11693 8268
@@
 $EndDescr
 $Comp
-L CONN_3 DCDC1
+L power_amp-rescue:CONN_3 DCDC1
 U 1 1 52497BBA
 P 6450 3700
@@
 $EndComp
 $Comp
-L C C1
+L power_amp-rescue:C C1
 U 1 1 52497C07
 P 4550 3450
@@
 $EndComp
 $Comp
-L C C2
+L power_amp-rescue:C C2
 U 1 1 52497C14
 P 4550 3950
@@
 $EndComp
 $Comp
-L CP1 C8
+L power_amp-rescue:CP1 C8
 U 1 1 52497D8D
 P 2250 3200
@@
 $EndComp
 $Comp
-L CP1 C10
+L power_amp-rescue:CP1 C10
 U 1 1 52497D9A
 P 3100 4300
@@
 $EndComp
 $Comp
-L C C7
+L power_amp-rescue:C C7
 U 1 1 52497DB4
 P 2550 3200
@@
 $EndComp
 $Comp
-L CONN_3 Power2
+L power_amp-rescue:CONN_3 Power2
 U 1 1 5249832A
 P 900 3750
@@
 $EndComp
 $Comp
-L CP1 C13
+L power_amp-rescue:CP1 C13
 U 1 1 5262630B
 P 3100 3200
@@
 $EndComp
 $Comp
-L C C14
+L power_amp-rescue:C C14
 U 1 1 52626311
 P 3400 3200
@@
 $EndComp
 $Comp
-L CP1 C11
+L power_amp-rescue:CP1 C11
 U 1 1 52626317
 P 2250 4300
@@
 $EndComp
 $Comp
-L C C9
+L power_amp-rescue:C C9
 U 1 1 52497DBA
 P 3400 4300
@@
 $EndComp
 $Comp
-L C C12
+L power_amp-rescue:C C12
 U 1 1 52626331
 P 2550 4300
@@
 $EndComp
 Wire Wire Line
-	4350 3250 6100 3250
-Wire Wire Line
-	4550 3650 4550 3750
+	4350 3250 4550 3250
+Wire Wire Line
+	4550 3650 4550 3700
 Connection ~ 4550 3700
 Connection ~ 4550 4150
 Wire Wire Line
-	2250 3000 2550 3000
+	2250 3000 2400 3000
 Connection ~ 2400 3000
 Connection ~ 4550 3250
@@
 	6100 3250 6100 3600
 Wire Wire Line
-	3800 3700 6100 3700
-Wire Wire Line
-	4350 4150 6100 4150
+	3800 3700 4550 3700
+Wire Wire Line
+	4350 4150 4550 4150
 Wire Wire Line
 	6100 4150 6100 3800
@@
 	4350 4850 4350 4150
 Wire Wire Line
-	3100 3000 3400 3000
-Wire Wire Line
-	3100 3400 3400 3400
-Wire Wire Line
-	3100 4100 3400 4100
-Wire Wire Line
-	3100 4500 3400 4500
+	3100 3000 3250 3000
+Wire Wire Line
+	3100 3400 3250 3400
+Wire Wire Line
+	3100 4100 3250 4100
+Wire Wire Line
+	3100 4500 3250 4500
 Connection ~ 3250 3000
 Connection ~ 3250 3400
 Wire Wire Line
-	2250 4500 2550 4500
-Wire Wire Line
-	2250 4100 2550 4100
-Wire Wire Line
-	2250 3400 2550 3400
+	2250 4500 2400 4500
+Wire Wire Line
+	2250 4100 2400 4100
+Wire Wire Line
+	2250 3400 2400 3400
 Connection ~ 3250 4500
 Connection ~ 3250 4100
@@
 Connection ~ 2400 3400
 Wire Wire Line
-	3250 3400 3250 4100
-Wire Wire Line
-	2400 3400 2400 4100
+	3250 3400 3250 3750
+Wire Wire Line
+	2400 3400 2400 3750
 Connection ~ 3250 3750
 Connection ~ 2400 3750
@@
 Connection ~ 2400 2600
 Wire Wire Line
-	1450 4850 4350 4850
+	1450 4850 2400 4850
 Wire Wire Line
 	2400 4850 2400 4500
@@
 	1250 3850 1450 3850
 Wire Wire Line
-	1250 3750 3800 3750
+	1250 3750 2400 3750
 Wire Wire Line
 	3800 3750 3800 3700
@@
 	1450 3650 1250 3650
 Wire Wire Line
-	1450 2600 4350 2600
+	1450 2600 2400 2600
+Wire Wire Line
+	4550 3700 4550 3750
+Wire Wire Line
+	4550 3700 6100 3700
+Wire Wire Line
+	4550 4150 6100 4150
+Wire Wire Line
+	2400 3000 2550 3000
+Wire Wire Line
+	4550 3250 6100 3250
+Wire Wire Line
+	3250 3000 3400 3000
+Wire Wire Line
+	3250 3400 3400 3400
+Wire Wire Line
+	3250 4500 3400 4500
+Wire Wire Line
+	3250 4100 3400 4100
+Wire Wire Line
+	2400 4100 2550 4100
+Wire Wire Line
+	2400 4500 2550 4500
+Wire Wire Line
+	2400 3400 2550 3400
+Wire Wire Line
+	3250 3750 3250 4100
+Wire Wire Line
+	3250 3750 3800 3750
+Wire Wire Line
+	2400 3750 2400 4100
+Wire Wire Line
+	2400 3750 3250 3750
+Wire Wire Line
+	3250 2600 4350 2600
+Wire Wire Line
+	2400 2600 3250 2600
+Wire Wire Line
+	2400 4850 3250 4850
+Wire Wire Line
+	3250 4850 4350 4850
 $EndSCHEMATC
