File: amp_v2/selector_box/selector_all/selector_ctrl.kicad_pcb (KiCad board)
At the start: 2 copper layers, 26.7 x 54 mm, 18 parts, among them J1 ATMEGA328P, P1 CONN_2, P2 CONN_2, P3 CONN_2, P4 CONN_2, P5 CONN_2

Commit message: updates
Other:
- net class Default removed
- net class sig removed
