File: amp_v2/selector_box/selector_ctrl_v2/selector_ctrl.sch (KiCad schematic (older format))
At the start: 59 parts, among them J1 ATMEGA328P, P1 CONN_4, P10 DIP05-1A72-12L, P11 Msgeq7_1, P12 Msgeq7_1, P16 DIP05-2A72-21L, P17 DIP05-2A72-21L, P18 DIP05-1A72-12L, P19 DIP05-1A72-12L, P2 CONN_4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

Commit message: updates
Parts:
- A_OUT1, IR1: symbol CONN_3 -> selector_ctrl-rescue:CONN_3
- C1, C3: symbol CP1-RESCUE-selector_ctrl -> selector_ctrl-rescue:CP1-RESCUE-selector_ctrl
- C10, C11, C12, C2, C4, C5, C6, C7, C8, C9: symbol C-RESCUE-selector_ctrl -> selector_ctrl-rescue:C-RESCUE-selector_ctrl
- D1, D2, D3, D4, D5: symbol DIODE -> selector_ctrl-rescue:DIODE
- FB1, FB2, FB3, FB4, FB5, FB6, FB7, FB8: symbol FILTER -> selector_ctrl-rescue:FILTER
- I2C1, P1, P2, P3, P4, RS1: symbol CONN_4 -> selector_ctrl-rescue:CONN_4
- J1: symbol SUPP28 -> selector_ctrl-rescue:SUPP28
- P10, P16, P17, P18, P19, P20, P6, P7, P9: symbol DIL14 -> selector_ctrl-rescue:DIL14
- P11, P12: symbol DIL8 -> selector_ctrl-rescue:DIL8
- Q1, Q2, Q3, Q4, Q5: symbol BC547 -> selector_ctrl-rescue:BC547
- R1, R2, R3, R4, R5, R6, R7, R8: symbol R-RESCUE-selector_ctrl -> selector_ctrl-rescue:R-RESCUE-selector_ctrl
- VDC1: symbol CONN_2 -> selector_ctrl-rescue:CONN_2
Connections:
- wire segments 233 -> 255
