File: led_segments1/led_segments.sch (KiCad schematic (older format))
At the start: 86 parts, among them J1 Conn_01x06_Female, J10 Conn_01x02, J11 Conn_01x02, J12 Conn_01x02, J13 Conn_01x02, J14 Conn_01x02, J15 Conn_01x02, J16 Conn_01x04, J2 Conn_01x01, J5 Conn_01x02, J6 Conn_01x02, J7 Conn_01x03, J8 Conn_01x02, J9 Conn_01x02, Q1 BC547, Q10 IRFU9024N, Q11 BC547, Q12 IRFU9024N, Q13 IRLU024N, Q14 IRLU024N, Q15 IRLU024N, Q16 IRLU024N, Q17 BC547, Q18 IRFU9024N, Q2 IRFU9024N, Q3 BC547, Q4 IRFU9024N, Q5 BC547, Q6 IRFU9024N, Q7 BC547, Q8 IRFU9024N, Q9 BC547, U1 MCP23017, U2 NodeMCU1.0(ESP-12E)

Commit message: updates
Parts:
- removed J2: Conn_01x01, Pin_Headers:Pin_Header_Straight_1x01_Pitch2.54mm, symbol Conn_01x01
- C1, C2: symbol CP -> led_segments-rescue:CP
- C3: symbol C -> led_segments-rescue:C
- D1, D10, D11, D12, D13, D14, D15, D16, D17, D18, D19, D2, D20, D21, D22, D23, D24, D25, D26, D27, D28, D3, D4, D5, D6, D7, D8, D9: symbol LED_Series -> led_segments-rescue:LED_Series
- J1: symbol Conn_01x06_Female -> led_segments-rescue:Conn_01x06_Female
- J10, J11, J12, J13, J14, J15, J5, J6, J8, J9: symbol Conn_01x02 -> led_segments-rescue:Conn_01x02
- J16: symbol Conn_01x04 -> led_segments-rescue:Conn_01x04
- J7: symbol Conn_01x03 -> led_segments-rescue:Conn_01x03
- Q1, Q11, Q17, Q3, Q5, Q7, Q9: symbol BC547 -> led_segments-rescue:BC547
- Q10, Q12, Q18, Q2, Q4, Q6, Q8: symbol Q_PMOS_GDS -> led_segments-rescue:Q_PMOS_GDS
- Q13, Q14, Q15, Q16: symbol Q_NMOS_GDS -> led_segments-rescue:Q_NMOS_GDS
- R1, R10, R11, R12, R13, R14, R15, R16, R17, R18, R2, R21, R3, R4, R5, R6, R7, R8, R9: symbol R -> led_segments-rescue:R
- R19, R20: value 4.7K -> 2.2K; symbol R -> led_segments-rescue:R
- U1: symbol MCP23017 -> led_segments-rescue:MCP23017
- U2: symbol NodeMCU1.0(ESP-12E) -> led_segments-rescue:NodeMCU1.0(ESP-12E)
Connections:
- wire segments 206 -> 256
- no-connect marks 23 -> 25
