File: rc_car/h_bridge/rc_car.sch (KiCad schematic (older format))
At the start: 20 parts, among them J1 CONN_01X06, Q10 IRLU024N, Q11 Q_NMOS_SGD, Q12 IRFU9024N, Q13 IRLU024N, Q14 Q_NMOS_SGD, Q7 Q_NMOS_SGD, Q8 IRFU9024N

Commit message: updates
Parts:
- D1, D2, D3, D4: symbol D -> rc_car-rescue:D
- J1: symbol CONN_01X06 -> rc_car-rescue:CONN_01X06
- Q10, Q13: symbol Q_NMOS_GDS -> rc_car-rescue:Q_NMOS_GDS
- Q11, Q14, Q7: symbol Q_NMOS_SGD -> rc_car-rescue:Q_NMOS_SGD
- Q12, Q8: symbol Q_PMOS_GDS -> rc_car-rescue:Q_PMOS_GDS
- R11, R12, R13, R16, R17, R6, R7, R8: symbol R -> rc_car-rescue:R
Changed lines of the file:
@@
-EESchema Schematic File Version 2
-LIBS:power
-LIBS:device
-LIBS:transistors
-LIBS:conn
-LIBS:linear
-LIBS:regul
-LIBS:74xx
-LIBS:cmos4000
-LIBS:adc-dac
-LIBS:memory
-LIBS:xilinx
-LIBS:microcontrollers
-LIBS:dsp
-LIBS:microchip
-LIBS:analog_switches
-LIBS:motorola
-LIBS:texas
-LIBS:intel
-LIBS:audio
-LIBS:interface
-LIBS:digital-audio
-LIBS:philips
-LIBS:display
-LIBS:cypress
-LIBS:siliconi
-LIBS:opto
-LIBS:atmel
-LIBS:contrib
-LIBS:valves
+EESchema Schematic File Version 4
 LIBS:rc_car-cache
-EELAYER 25 0
+EELAYER 30 0
 EELAYER END
 $Descr A4 11693 8268
@@
 M2_R
 $Comp
-L GND #PWR01
+L rc_car-rescue:GND #PWR01
 U 1 1 588961A1
 P 6400 4250
@@
 VIN_MOTOR
 $Comp
-L R R7
+L rc_car-rescue:R R7
 U 1 1 5889617A
 P 5250 2800
@@
 $EndComp
 $Comp
-L Q_NMOS_GDS Q13
+L rc_car-rescue:Q_NMOS_GDS Q13
 U 1 1 58896165
 P 7200 3850
@@
 $EndComp
 $Comp
-L Q_NMOS_GDS Q10
+L rc_car-rescue:Q_NMOS_GDS Q10
 U 1 1 5889615F
 P 5600 3850
@@
 $EndComp
 $Comp
-L Q_PMOS_GDS Q12
+L rc_car-rescue:Q_PMOS_GDS Q12
 U 1 1 58896159
 P 7200 3100
@@
 $EndComp
 $Comp
-L Q_PMOS_GDS Q8
+L rc_car-rescue:Q_PMOS_GDS Q8
 U 1 1 58896153
 P 5600 3100
@@
 Connection ~ 7100 3450
 Wire Wire Line
-	7100 3300 7100 3650
+	7100 3300 7100 3450
 Connection ~ 5700 3450
 Wire Wire Line
-	5700 3300 5700 3650
-Wire Wire Line
-	5250 2950 5250 3850
-$Comp
-L D D1
+	5700 3300 5700 3450
+Wire Wire Line
+	5250 2950 5250 3300
+$Comp
+L rc_car-rescue:D D1
 U 1 1 5895349F
 P 5100 3300
@@
 Connection ~ 5250 3300
 $Comp
-L D D2
+L rc_car-rescue:D D2
 U 1 1 58953890
 P 5100 3600
@@
 Connection ~ 5250 3600
 $Comp
-L R R12
+L rc_car-rescue:R R12
 U 1 1 58896173
 P 7500 2800
@@
 $EndComp
 $Comp
-L R R13
+L rc_car-rescue:R R13
 U 1 1 5895668B
 P 4650 2800
@@
 $EndComp
 $Comp
-L R R11
+L rc_car-rescue:R R11
 U 1 1 58956B2F
 P 3750 2800
@@
 $EndComp
 $Comp
-L Q_NMOS_SGD Q11
+L rc_car-rescue:Q_NMOS_SGD Q11
 U 1 1 58956DE3
 P 3650 4800
@@
 $EndComp
 Connection ~ 4950 3300
-Connection ~ 4950 3600
 Wire Wire Line
 	4950 3600 4950 4600
 $Comp
-L Q_NMOS_SGD Q7
+L rc_car-rescue:Q_NMOS_SGD Q7
 U 1 1 5895A373
 P 4550 3500
@@
 $EndComp
 $Comp
-L R R8
+L rc_car-rescue:R R8
 U 1 1 5895A83E
 P 3300 4950
@@
 $EndComp
 $Comp
-L R R6
+L rc_car-rescue:R R6
 U 1 1 5895ABC1
 P 4250 3650
@@
 M2_EN
 Wire Wire Line
-	7500 2950 7500 3850
-$Comp
-L D D3
+	7500 2950 7500 3250
+$Comp
+L rc_car-rescue:D D3
 U 1 1 5895E5B7
 P 7650 3250
@@
 $EndComp
 $Comp
-L D D4
+L rc_car-rescue:D D4
 U 1 1 5895E95A
 P 7650 3500
@@
 Connection ~ 7500 3500
 $Comp
-L R R16
+L rc_car-rescue:R R16
 U 1 1 5895EFFF
 P 7950 2800
@@
 	7950 3250 7950 2950
 $Comp
-L Q_NMOS_SGD Q14
+L rc_car-rescue:Q_NMOS_SGD Q14
 U 1 1 5895F95A
 P 8050 3450
@@
 Connection ~ 7950 3250
 $Comp
-L R R17
+L rc_car-rescue:R R17
 U 1 1 5895FF0B
 P 8250 3750
@@
 	5250 3850 5400 3850
 Wire Wire Line
-	3750 4600 7800 4600
+	3750 4600 4950 4600
 Wire Wire Line
 	7400 3100 7800 3100
@@
 	8250 3900 8250 4000
 $Comp
-L GND #PWR02
+L rc_car-rescue:GND #PWR02
 U 1 1 58ABDC0F
 P 7950 3750
@@
 $EndComp
 $Comp
-L GND #PWR03
+L rc_car-rescue:GND #PWR03
 U 1 1 58ABDD34
 P 8250 4000
@@
 $EndComp
 Wire Wire Line
-	5700 4150 7100 4150
+	5700 4150 6400 4150
 Wire Wire Line
 	6400 4150 6400 4250
 Connection ~ 6400 4150
 Wire Wire Line
-	3750 2550 7950 2550
+	3750 2550 4650 2550
 Wire Wire Line
 	5250 2550 5250 2650
@@
 Connection ~ 5250 2550
 $Comp
-L GND #PWR04
+L rc_car-rescue:GND #PWR04
 U 1 1 58AC0E7B
 P 4650 3800
@@
 	4650 3800 4650 3700
 $Comp
-L GND #PWR05
+L rc_car-rescue:GND #PWR05
 U 1 1 58AC11BE
 P 4250 3900
@@
 	4250 3900 4250 3800
 Wire Wire Line
-	4000 3500 4350 3500
+	4000 3500 4250 3500
 Connection ~ 4950 4600
 Wire Wire Line
@@
 M2_L
 Wire Wire Line
-	3100 4800 3450 4800
+	3100 4800 3300 4800
 Connection ~ 3300 4800
 $Comp
-L GND #PWR06
+L rc_car-rescue:GND #PWR06
 U 1 1 58AC2F66
 P 3300 5150
@@
 $EndComp
 $Comp
-L GND #PWR07
+L rc_car-rescue:GND #PWR07
 U 1 1 58AC2FFE
 P 3750 5150
@@
 	6800 3450 7100 3450
 $Comp
-L CONN_01X06 J1
+L rc_car-rescue:CONN_01X06 J1
 U 1 1 5953AFBA
 P 5350 5000
@@
 	5300 5200 5200 5200
 Wire Wire Line
-	5200 5200 5200 5850
+	5200 5200 5200 5750
 Wire Wire Line
 	5400 5350 5400 5200
@@
 Connection ~ 5200 5750
 $Comp
-L GND #PWR08
+L rc_car-rescue:GND #PWR08
 U 1 1 5953B5BA
 P 5200 5850
@@
 	1    0    0    -1
 $EndComp
+Wire Wire Line
+	7100 3450 7100 3650
+Wire Wire Line
+	5700 3450 5700 3650
+Wire Wire Line
+	5250 3300 5250 3600
+Wire Wire Line
+	5250 3600 5250 3850
+Wire Wire Line
+	7500 3250 7500 3500
+Wire Wire Line
+	7500 3500 7500 3850
+Wire Wire Line
+	6400 4150 7100 4150
+Wire Wire Line
+	5700 2550 6400 2550
+Wire Wire Line
+	7100 2550 7500 2550
+Wire Wire Line
+	7500 2550 7950 2550
+Wire Wire Line
+	6400 2550 7100 2550
+Wire Wire Line
+	5250 2550 5700 2550
+Wire Wire Line
+	4950 4600 7800 4600
+Wire Wire Line
+	4650 2550 5250 2550
+Wire Wire Line
+	4250 3500 4350 3500
+Wire Wire Line
+	3300 4800 3450 4800
+Wire Wire Line
+	5200 5750 5200 5850
 $EndSCHEMATC
