File: amp_v2/selector_box/rid_relay_audio/selector_rid_ground.kicad_pcb (KiCad board)
At the start: 2 copper layers, 33 x 30.5 mm, 8 parts, among them K1 CONN_3, P1 CONN_4, P2 CONN_4, P3 DIP05-2A72-21L, P4 DIP05-1A72-12L, Q1 BC547

Commit message: update_v3
Parts:
- removed K1: CONN_3, Pin_Headers:Pin_Header_Straight_1x03
- removed P3: DIP05-2A72-21L, Housings_DIP:DIP-14_W7.62mm_LongPads
- removed P4: DIP05-1A72-12L, Housings_DIP:DIP-14_W7.62mm_LongPads
- added D2: DIODE, Diode_THT:D_A-405_P7.62mm_Horizontal, F.Cu at (237.5, 188.0)
- added J1: Conn_01x02_Pin, Connector_PinHeader_2.54mm:PinHeader_1x02_P2.54mm_Vertical, F.Cu at (232.9, 176.4)
- added J2: Conn_01x02_Pin, Connector_PinHeader_2.54mm:PinHeader_1x02_P2.54mm_Vertical, F.Cu at (229.4, 176.4)
- added J3: Conn_01x03_Pin, Connector_JST:JST_XH_B3B-XH-A_1x03_P2.50mm_Vertical, F.Cu at (250.2, 136.4)
- added J4: Conn_01x03_Pin, Connector_JST:JST_XH_B3B-XH-A_1x03_P2.50mm_Vertical, F.Cu at (245.2, 144.8)
- added Q2: 2N7000, Package_TO_SOT_THT:TO-92L_Inline_Wide, F.Cu at (232.9, 183.6)
- added R2: 10K, Resistor_THT:R_Axial_DIN0207_L6.3mm_D2.5mm_P7.62mm_Horizontal, F.Cu at (255.3, 139.7)
- added R3: 0R, Resistor_THT:R_Axial_DIN0207_L6.3mm_D2.5mm_P7.62mm_Horizontal, F.Cu at (229.9, 166.4)
- added R4: 0R, Resistor_THT:R_Axial_DIN0207_L6.3mm_D2.5mm_P7.62mm_Horizontal, F.Cu at (229.9, 191.8)
- added R5: 680, Resistor_THT:R_Axial_DIN0207_L6.3mm_D2.5mm_P7.62mm_Horizontal, F.Cu at (247.7, 172.7)
- added R6: 3.3K, Resistor_THT:R_Axial_DIN0207_L6.3mm_D2.5mm_P7.62mm_Horizontal, F.Cu at (247.7, 198.1)
- added R7: 680, Resistor_THT:R_Axial_DIN0204_L3.6mm_D1.6mm_P2.54mm_Vertical, F.Cu at (250.2, 174.0)
- added R8: 3.3K, Resistor_THT:R_Axial_DIN0204_L3.6mm_D1.6mm_P2.54mm_Vertical, F.Cu at (250.2, 199.4)
- D1: footprint Diodes_ThroughHole:Diode_DO-35_SOD27_Horizontal_RM10 -> Diode_THT:D_A-405_P7.62mm_Horizontal
- P1, P2: value CONN_4 -> DIP05-2A72-21L; footprint Pin_Headers:Pin_Header_Straight_1x04 -> Package_DIP:DIP-14_W7.62mm_Socket_LongPads
- Q1: value BC547 -> 2N7000; footprint TO_SOT_Packages_THT:TO-92_Inline_Narrow_Oval -> Package_TO_SOT_THT:TO-92L_Inline_Wide
- R1: value 12K -> 10K; footprint Discret:R4 -> Resistor_THT:R_Axial_DIN0207_L6.3mm_D2.5mm_P7.62mm_Horizontal
- moved P2 57.1 mm to (242.6, 177.8), turned to 0 degrees
- moved P1 35.5 mm to (242.6, 152.4)
- moved R1 31.9 mm to (240.0, 147.3)
- moved Q1 28.6 mm to (232.9, 170.7)
- moved D1 28.1 mm to (237.5, 162.6)
Connections:
- D1 pad 1: Net-(D1-Pad1) -> Net-(D1-A)
- P1 pad 1: /VCC -> /L_OUT
- P1 pad 2: GND -> /VCC
- P2 pad 1: /L_IN1 -> /L_OUT
- P2 pad 2: /G_IN1 -> /VCC
- Q1 pad 1: Net-(D1-Pad1) -> GND
- Q1 pad 2: Net-(Q1-Pad2) -> /EN_1
- Q1 pad 3: GND -> Net-(Q1-D)
- R1 pad 1: Net-(Q1-Pad2) -> /L_OUT
- R1 pad 2: /EN1 -> /L_IN
Routing:
- net /AGND: track 0.00 -> 72.7 mm
- net /L_OUT: track 6.24 -> 73.3 mm
- net /R_OUT: track 6.24 -> 70.0 mm
- net /G_IN1: track 32.6 -> 0.00 mm
- net Net-(D1-Pad1): track 29.6 -> 0.00 mm
- net /G_OUT: track 25.0 -> 0.00 mm
- net GND: track 0.00 -> 13.0 mm
- net /VCC: track 27.5 -> 37.2 mm
- net Net-(D2-A): track 0.00 -> 9.41 mm
- net Net-(D1-A): track 0.00 -> 9.41 mm
- net Net-(Q2-D): track 0.00 -> 8.97 mm
- net Net-(Q1-Pad2): track 8.67 -> 0.00 mm
- net /EN_1: track 0.00 -> 7.82 mm
- net /EN_2: track 0.00 -> 7.66 mm
- net /R_IN1: track 6.98 -> 0.00 mm
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- removed copper zone on B.Cu, net GND
Other:
- board outline removed
- net class Default removed
- net class Power removed
