File: amp_v3/jfet_buffer1/jfet_buffer.kicad_pcb (KiCad board)
At the start: 2 copper layers, 70.5 x 43.2 mm, 36 parts, among them J1 Conn_01x04_Pin, J2 Signal Input, J3 SIG_OUT_L1, J4 SIG_OUT_R_1, J5 SIG_OUT_L2, J6 SIG_OUT_R2, Q1 2N5457 DSG, Q2 2N5457, Q3 2N5457 DSG, Q4 2N5457 DSG

Commit message: update
Parts:
- removed the C4 at (92.5, 52.2)
- removed the C7 at (92.5, 72.5)
- moved C4 2.78 mm to (94.9, 58.6), turned to 180 degrees
- moved C5 2.75 mm to (94.9, 66.2), turned to 180 degrees
- renumbered C12 to C10, C5 to C4, C6 to C5, C8 to C6, C9 to C7, C10 to C8, C11 to C9
Routing:
- net +20V: track 224.1 -> 194.4 mm
- net GND_IN_L: track 125.8 -> 123.2 mm
- net GND_IN_R: track 122.5 -> 120.3 mm
