File: amp_v3/jfet_buffer1/jfet_buffer.kicad_pcb (KiCad board)
At the start: 2 copper layers, 70.5 x 43.2 mm, 34 parts, among them J1 Conn_01x04_Pin, J2 Signal Input, J3 SIG_OUT_L1, J4 SIG_OUT_R_1, J5 SIG_OUT_L2, J6 SIG_OUT_R2, Q1 2N5457 DSG, Q2 2N5457, Q3 2N5457 DSG, Q4 2N5457 DSG

Commit message: update
Parts:
- added C1: 100nF, Capacitor_THT:C_Rect_L7.2mm_W2.5mm_P5.00mm_FKS2_FKP2_MKS2_MKP2, F.Cu at (36.5, 55.4)
- added C2: 100nF, Capacitor_THT:C_Rect_L7.2mm_W2.5mm_P5.00mm_FKS2_FKP2_MKS2_MKP2, F.Cu at (36.5, 69.3)
- R1, R2, R3, R4: value 100K -> 1M
- moved R1 11.3 mm to (40.4, 49.7), turned to 180 degrees
- moved R2 5.46 mm to (32.7, 75.1), turned to 0 degrees
- moved R8 2.01 mm to (43.5, 49.7)
- moved R7 2.01 mm to (43.5, 75.1)
- moved R6 1.52 mm to (55.6, 50.3)
- moved R5 1.50 mm to (55.6, 74.4)
- moved C9 0.26 mm to (52.2, 71.2)
- moved C10 0.25 mm to (52.2, 53.5)
- moved C3 0.13 mm to (45.9, 55.4)
- moved C4 0.13 mm to (45.9, 69.3)
- renumbered C8 to C10, C9 to C11, C10 to C12, C1 to C3, C2 to C4, C3 to C5, C4 to C6, C5 to C7, C6 to C8, C7 to C9, J3 to J2, J2 to J3
Routing:
- net +20V: track 194.4 -> 217.9 mm
- net /VBIAS_OUT_L: track 39.3 -> 21.3 mm
- net /VBIAS_L: track 19.4 -> 6.13 mm
- net /VBIAS_R: track 18.8 -> 5.51 mm
- net /VBIAS_OUT_R: track 31.8 -> 21.6 mm
- net Net-(Q1-G): track 6.04 -> 0.00 mm
- net GND_IN_L: track 123.2 -> 127.8 mm
- net Net-(Q2-G): track 5.14 -> 4.50 mm
- net GND_IN_R: track 120.3 -> 120.9 mm
- added copper zone on B.Cu, net /L_IN
- added copper zone on B.Cu, net /R_IN
- added copper zone on B.Cu, net /VBIAS_L
- added copper zone on B.Cu, net /VBIAS_OUT_L
- added copper zone on B.Cu, net /VBIAS_OUT_R
- added copper zone on B.Cu, net /VBIAS_R
- added copper zone on B.Cu, net GND_IN_L
- added copper zone on B.Cu, net GND_IN_R
Other:
- board size 70.5 x 43.2 mm -> 74.9 x 43.2 mm
