File: amp_v3/jfet_buffer1/jfet_buffer.kicad_sch (KiCad schematic)
At the start: 36 parts, among them J1 Conn_01x04_Pin, J2 Signal Input, J3 SIG_OUT_L1, J4 SIG_OUT_R_1, J5 SIG_OUT_L2, J6 SIG_OUT_R2, Q1 2N5457 DSG, Q2 2N5457, Q3 2N5457 DSG, Q4 2N5457 DSG

Commit message: update
Parts:
- removed C4, C7: 100nF, Capacitor_THT:C_Rect_L7.2mm_W2.5mm_P5.00mm_FKS2_FKP2_MKS2_MKP2, symbol Device:C
- renumbered C12 to C10, C5 to C4, C6 to C5, C8 to C6, C9 to C7, C10 to C8, C11 to C9
Changed lines of the file:
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@@
 	)
 	(junction
-		(at 35.56 63.5)
-		(diameter 0)
-		(color 0 0 0 0)
-	)
-	(junction
 		(at 119.38 33.02)
 		(diameter 0)
@@
 	)
 	(junction
-		(at 22.86 63.5)
-		(diameter 0)
-		(color 0 0 0 0)
-	)
-	(junction
 		(at 123.19 83.82)
 		(diameter 0)
@@
 	)
 	(junction
-		(at 35.56 55.88)
-		(diameter 0)
-		(color 0 0 0 0)
-	)
-	(junction
 		(at 165.1 127)
 		(diameter 0)
@@
 	)
 	(junction
-		(at 22.86 55.88)
-		(diameter 0)
-		(color 0 0 0 0)
-	)
-	(junction
 		(at 265.43 100.33)
 		(diameter 0)
@@
 	(wire
 		(pts
-			(xy 35.56 55.88) (xy 44.45 55.88)
-		)
-		(stroke
-			(width 0)
-			(type default)
-		)
-	)
-	(wire
-		(pts
 			(xy 265.43 49.53) (xy 270.51 49.53)
 		)
@@
 	(wire
 		(pts
-			(xy 35.56 63.5) (xy 44.45 63.5)
-		)
-		(stroke
-			(width 0)
-			(type default)
-		)
-	)
-	(wire
-		(pts
 			(xy 209.55 81.28) (xy 217.17 81.28)
 		)
@@
 	(wire
 		(pts
-			(xy 13.97 63.5) (xy 22.86 63.5)
-		)
-		(stroke
-			(width 0)
-			(type default)
-		)
-	)
-	(wire
-		(pts
 			(xy 195.58 31.75) (xy 195.58 34.29)
 		)
@@
 	(wire
 		(pts
-			(xy 13.97 55.88) (xy 22.86 55.88)
-		)
-		(stroke
-			(width 0)
-			(type default)
-		)
-	)
-	(wire
-		(pts
 			(xy 66.04 111.76) (xy 66.04 115.57)
 		)
@@
 		(in_pos_files yes)
 		(dnp no)
-		(property "Reference" "C5"
+		(property "Reference" "C4"
 			(at 24.384 62.992 0)
 			(show_name no)
@@
 			(project "jfet_buffer"
 				(path "/4a69c903-ca61-4bf4-abb9-de13d0f3d285"
-					(reference "C5")
+					(reference "C4")
 					(unit 1)
 				)
@@
 		(dnp no)
 		(fields_autoplaced yes)
-		(property "Reference" "C8"
+		(property "Reference" "C6"
 			(at 172.72 58.4199 0)
 			(show_name no)
@@
 			(project "jfet_buffer"
 				(path "/4a69c903-ca61-4bf4-abb9-de13d0f3d285"
-					(reference "C8")
+					(reference "C6")
 					(unit 1)
 				)
@@
 		(dnp no)
 		(fields_autoplaced yes)
-		(property "Reference" "C12"
+		(property "Reference" "C10"
 			(at 172.72 107.9499 0)
 			(show_name no)
@@
 			(project "jfet_buffer"
 				(path "/4a69c903-ca61-4bf4-abb9-de13d0f3d285"
-					(reference "C12")
+					(reference "C10")
 					(unit 1)
 				)
@@
 		(in_pos_files yes)
 		(dnp no)
-		(property "Reference" "C10"
+		(property "Reference" "C8"
 			(at 121.92 84.455 0)
 			(show_name no)
@@
 			(project "jfet_buffer"
 				(path "/4a69c903-ca61-4bf4-abb9-de13d0f3d285"
-					(reference "C10")
+					(reference "C8")
 					(unit 1)
 				)
@@
 		(in_pos_files yes)
 		(dnp no)
-		(property "Reference" "C9"
+		(property "Reference" "C7"
 			(at 208.28 81.915 0)
 			(show_name no)
@@
 			(project "jfet_buffer"
 				(path "/4a69c903-ca61-4bf4-abb9-de13d0f3d285"
-					(reference "C9")
+					(reference "C7")
 					(unit 1)
 				)
@@
 	)
 	(symbol
-		(lib_id "Device:C")
-		(at 13.97 59.69 0)
-		(unit 1)
-		(body_style 1)
-		(exclude_from_sim no)
-		(in_bom yes)
-		(on_board yes)
-		(in_pos_files yes)
-		(dnp no)
-		(property "Reference" "C4"
-			(at 10.668 56.642 0)
-			(show_name no)
-			(do_not_autoplace no)
-			(effects
-				(font
-					(size 1.27 1.27)
-				)
-				(justify left)
-			)
-		)
-		(property "Value" "100nF"
-			(at 7.62 62.23 0)
-			(show_name no)
-			(do_not_autoplace no)
-			(effects
-				(font
-					(size 1.27 1.27)
-				)
-				(justify left)
-			)
-		)
-		(property "Footprint" "Capacitor_THT:C_Rect_L7.2mm_W2.5mm_P5.00mm_FKS2_FKP2_MKS2_MKP2"
-			(at 14.9352 63.5 0)
-			(hide yes)
-			(show_name no)
-			(do_not_autoplace no)
-			(effects
-				(font
-					(size 1.27 1.27)
-				)
-			)
-		)
-		(property "Datasheet" ""
-			(at 13.97 59.69 0)
-			(hide yes)
-			(show_name no)
-			(do_not_autoplace no)
-			(effects
-				(font
-					(size 1.27 1.27)
-				)
-			)
-		)
-		(property "Description" "Unpolarized capacitor"
-			(at 13.97 59.69 0)
-			(hide yes)
-			(show_name no)
-			(do_not_autoplace no)
-			(effects
-				(font
-					(size 1.27 1.27)
-				)
-			)
-		)
-		(pin "1"
-		)
-		(pin "2"
-		)
-		(instances
-			(project "jfet_buffer"
-				(path "/4a69c903-ca61-4bf4-abb9-de13d0f3d285"
-					(reference "C4")
-					(unit 1)
-				)
-			)
-		)
-	)
-	(symbol
 		(lib_id "power_ctrl-rescue:GNDA")
 		(at 119.38 44.45 0)
@@
 		(in_pos_files yes)
 		(dnp no)
-		(property "Reference" "C6"
+		(property "Reference" "C5"
 			(at 39.878 60.706 90)
 			(show_name no)
@@
 			(project "jfet_buffer"
 				(path "/4a69c903-ca61-4bf4-abb9-de13d0f3d285"
-					(reference "C6")
-					(unit 1)
-				)
-			)
-		)
-	)
-	(symbol
-		(lib_id "Device:C")
-		(at 44.45 59.69 0)
-		(unit 1)
-		(body_style 1)
-		(exclude_from_sim no)
-		(in_bom yes)
-		(on_board yes)
-		(in_pos_files yes)
-		(dnp no)
-		(fields_autoplaced yes)
-		(property "Reference" "C7"
-			(at 48.26 58.4199 0)
-			(show_name no)
-			(do_not_autoplace no)
-			(effects
-				(font
-					(size 1.27 1.27)
-				)
-				(justify left)
-			)
-		)
-		(property "Value" "100nF"
-			(at 48.26 60.9599 0)
-			(show_name no)
-			(do_not_autoplace no)
-			(effects
-				(font
-					(size 1.27 1.27)
-				)
-				(justify left)
-			)
-		)
-		(property "Footprint" "Capacitor_THT:C_Rect_L7.2mm_W2.5mm_P5.00mm_FKS2_FKP2_MKS2_MKP2"
-			(at 45.4152 63.5 0)
-			(hide yes)
-			(show_name no)
-			(do_not_autoplace no)
-			(effects
-				(font
-					(size 1.27 1.27)
-				)
-			)
-		)
-		(property "Datasheet" ""
-			(at 44.45 59.69 0)
-			(hide yes)
-			(show_name no)
-			(do_not_autoplace no)
-			(effects
-				(font
-					(size 1.27 1.27)
-				)
-			)
-		)
-		(property "Description" "Unpolarized capacitor"
-			(at 44.45 59.69 0)
-			(hide yes)
-			(show_name no)
-			(do_not_autoplace no)
-			(effects
-				(font
-					(size 1.27 1.27)
-				)
-			)
-		)
-		(pin "1"
-		)
-		(pin "2"
-		)
-		(instances
-			(project "jfet_buffer"
-				(path "/4a69c903-ca61-4bf4-abb9-de13d0f3d285"
-					(reference "C7")
+					(reference "C5")
 					(unit 1)
 				)
@@
 		(dnp no)
 		(fields_autoplaced yes)
-		(property "Reference" "C11"
+		(property "Reference" "C9"
 			(at 274.32 102.8699 0)
 			(show_name no)
@@
 			(project "jfet_buffer"
 				(path "/4a69c903-ca61-4bf4-abb9-de13d0f3d285"
-					(reference "C11")
+					(reference "C9")
 					(unit 1)
 				)
