File: amp_v3/jfet_buffer1/jfet_buffer.kicad_sch (KiCad schematic)
At the start: 34 parts, among them J1 Conn_01x04_Pin, J2 Signal Input, J3 SIG_OUT_L1, J4 SIG_OUT_R_1, J5 SIG_OUT_L2, J6 SIG_OUT_R2, Q1 2N5457 DSG, Q2 2N5457, Q3 2N5457 DSG, Q4 2N5457 DSG

Commit message: update
Parts:
- added C1, C2: 100nF, Capacitor_THT:C_Rect_L7.2mm_W2.5mm_P5.00mm_FKS2_FKP2_MKS2_MKP2, symbol Device:C
- R1, R2, R3, R4: value 100K -> 1M
- renumbered C8 to C10, C9 to C11, C10 to C12, C1 to C3, C2 to C4, C3 to C5, C4 to C6, C5 to C7, C6 to C8, C7 to C9, J3 to J2, J2 to J3
Connections:
- net +20V: now also C1.1, C2.1
- net GND_IN_L: now also C1.2
- net GND_IN_R: now also C2.2
Other:
- moved on the sheet: J2, J3, J4, J5, J6
