File: amp_v3/jfet_buffer3/jfet_buffer.kicad_sch (KiCad schematic)
At the start: 21 parts, among them J1 SIG_OUT_L1, J2 SIG_OUT_L1, J3 SIG_OUT_L1, J4 SIG_OUT_L2, Q1 2N5457, Q2 2N5457 DSG

Commit message: updates
Parts:
- added H3, H4: MountingHole_Pad, Connector_PinHeader_2.54mm:PinHeader_1x01_P2.54mm_Vertical, symbol Mechanical:MountingHole_Pad
- added R7: 0R, Resistor_THT:R_Axial_DIN0207_L6.3mm_D2.5mm_P5.08mm_Vertical, symbol power_ctrl-rescue:R
- renumbered R7 to R8
Connections:
- net +20V: now also H3.1, H4.1
- net GND_IN_L: now also R7.2
- new net SH_GND: R7.1
Other:
- moved on the sheet: H1, H2, J2
