File: amp_v3/jfet_buffer4/jfet_buffer.kicad_sch (KiCad schematic)
At the start: 21 parts, among them J1 SIG_OUT_L1, J2 SIG_OUT_L1, J3 SIG_OUT_L1, J4 SIG_OUT_L2, Q1 2N5457, Q2 2N5457 DSG

Commit message: updates
Parts:
- removed H1, H2: MountingHole_Pad, Connector_PinHeader_2.54mm:PinHeader_1x01_P2.54mm_Vertical, symbol Mechanical:MountingHole_Pad
- added R7: 0R, Resistor_THT:R_Axial_DIN0207_L6.3mm_D2.5mm_P2.54mm_Vertical, symbol power_ctrl-rescue:R
- renumbered R7 to R8
Connections:
- net GND_IN_L: now also R7.2
- new net SH_GND: R7.1
Other:
- moved on the sheet: J2

Commit message: update
Parts:
- J1: value SIG_OUT_L1 -> PWR
- J2: value SIG_OUT_L1 -> INPUT
- J3: value SIG_OUT_L1 -> OUT1
- J4: value SIG_OUT_L2 -> OUT2
- Q2: value 2N5457 DSG -> 2N5457
- renumbered R8 to R7, R7 to R8
Connections:
- net GND_IN_L renamed GND
- net L_IN renamed INPUT
- net L_OUT_BUF1 renamed OUT1
- net L_OUT_BUF2 renamed OUT2
- net VBIAS_L renamed VBIAS
- net VBIAS_OUT_L renamed VBIAS_OUT
Other:
- moved on the sheet: C2, C5, Q1, Q2, R2, R4, R6, R7, R8
