File: delta/power_top/power_top.kicad_pcb (KiCad board)
At the start: 2 copper layers, 44.5 x 54 mm, 12 parts, among them J1 PWR_PANEL, J2 FAN_SSR_PANEL, J3 48V_EZ3, J4 24V_EZ3, J5 FAN_SSR_EZ3, J6 GND_ENCLOSURE, J7 GND_ENCLOSURE, J8 PWR_ENCLOSURE

Commit message: updates
Other:
- board size 44.5 x 54 mm -> 39.1 x 41.1 mm
Changed lines of the file:
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@@
 		(capping no)
 		(filling no)
-		(zone_defaults)
 		(grid_origin 63.5 51.435)
 		(pcbplotparams
-			(layerselection 0x00000000_00000000_55555555_5755f5ff)
+			(layerselection 0x00000000_00000000_55555555_57555550)
 			(plot_on_all_layers_selection 0x00000000_00000000_00000000_00000000)
 			(disableapertmacros no)
@@
 			(crossoutdnponfab yes)
 			(subtractmaskfromsilk no)
-			(outputformat 1)
+			(outputformat 5)
 			(mirror no)
-			(drillshape 1)
+			(drillshape 0)
 			(scaleselection 1)
 			(outputdirectory "")
@@
 		)
 		(fill no)
-		(layer "Edge.Cuts")
+		(layer "Dwgs.User")
 	)
 	(gr_circle
