File: delta/12v_pwr/12v_pwr.kicad_sch (KiCad schematic)
At the start: 11 parts, among them J1 GND_ENCLOSURE, J10 FAN_OUT_PANEL_4, J2 24V_PANEL, J3 GND_ENCLOSURE, J4 FAN_IN_EZ3_1, J5 FAN_IN_EZ3_2, J6 12V_ENCLOSURE, J7 FAN_OUT_PANEL_1, J8 FAN_OUT_PANEL_2, J9 FAN_OUT_PANEL_3

Commit message: updates
Parts:
- removed J1, J3: GND_ENCLOSURE, Connector_TE-Connectivity:TE_826576-2_1x02_P3.96mm_Vertical, symbol Connector:Conn_01x02_Socket
- added J10, J9: FAN_OUT_PANEL_2, Connector_JST:JST_XH_B2B-XH-A_1x02_P2.50mm_Vertical, symbol Connector:Conn_01x02_Socket
- added J12: FAN_OUT_PANEL_3, Connector_JST:JST_XH_B2B-XH-A_1x02_P2.50mm_Vertical, symbol Connector:Conn_01x02_Socket
- added J15: FAN_OUT_PANEL_4, Connector_JST:JST_XH_B2B-XH-A_1x02_P2.50mm_Vertical, symbol Connector:Conn_01x02_Socket
- added J6, J7: FAN_OUT_PANEL_1, Connector_JST:JST_XH_B2B-XH-A_1x02_P2.50mm_Vertical, symbol Connector:Conn_01x02_Socket
- J1: renamed from J2; footprint Connector_TE-Connectivity:TE_826576-2_1x02_P3.96mm_Vertical -> TerminalBlock_Phoenix:TerminalBlock_Phoenix_PT-1,5-2-5.0-H_1x02_P5.00mm_Horizontal
- J11: renamed from J9; footprint Connector_TE-Connectivity:TE_826576-2_1x02_P3.96mm_Vertical -> Connector_JST:JST_XH_B2B-XH-A_1x02_P2.50mm_Vertical
- J14: renamed from J10; footprint Connector_TE-Connectivity:TE_826576-2_1x02_P3.96mm_Vertical -> Connector_JST:JST_XH_B2B-XH-A_1x02_P2.50mm_Vertical
- J4: renamed from J6; footprint Connector_TE-Connectivity:TE_826576-2_1x02_P3.96mm_Vertical -> TerminalBlock_Phoenix:TerminalBlock_Phoenix_PT-1,5-2-5.0-H_1x02_P5.00mm_Horizontal
- J5: renamed from J7; footprint Connector_TE-Connectivity:TE_826576-2_1x02_P3.96mm_Vertical -> Connector_JST:JST_XH_B2B-XH-A_1x02_P2.50mm_Vertical
- J8: footprint Connector_TE-Connectivity:TE_826576-2_1x02_P3.96mm_Vertical -> Connector_JST:JST_XH_B2B-XH-A_1x02_P2.50mm_Vertical
- renumbered J4 to J2, J5 to J3
Connections:
- net +12V: now also J10.1 (Pin_1), J12.1 (Pin_1), J15.1 (Pin_1), J6.1 (Pin_1), J7.1 (Pin_1), J9.1 (Pin_1); no longer J4.2 (Pin_2)
- net FAN1_NEG: now also J6.2 (Pin_2), J7.2 (Pin_2)
- net FAN2_NEG: now also J10.2 (Pin_2), J9.2 (Pin_2)
- net FAN3_NEG: now also J12.2 (Pin_2)
- net FAN4_NEG: now also J15.2 (Pin_2)
- net GND: now also J4.2 (Pin_2)
