File: amp_v3/ldr_volume/board#3.kicad_sch (KiCad schematic)
At the start: 42 parts, among them J11 5v_in_b3, J12 TFT_PWR, J13 TFT_L, J14 BOARD2.L, J15 TFT_PWR, J16 TFT_R, J17 BOARD2.R, Q1 2N7000, Q2 2N7000, Q3 2N7000, Q4 2N7000, Q5 2N7000, Q6 2N7000

Commit message: updates
Parts:
- removed J14: BOARD2.L, Connector_JST:JST_XH_B5B-XH-A_1x05_P2.50mm_Vertical, symbol Connector:Conn_01x05_Pin
- removed J17: BOARD2.R, Connector_JST:JST_XH_B5B-XH-A_1x05_P2.50mm_Vertical, symbol Connector:Conn_01x05_Pin
- added J14: BOARD2.L, Connector_JST:JST_XH_B6B-XH-A_1x06_P2.50mm_Vertical, symbol Connector:Conn_01x06_Pin
- added J17: BOARD2.R, Connector_JST:JST_XH_B6B-XH-A_1x06_P2.50mm_Vertical, symbol Connector:Conn_01x06_Pin
Connections:
- net COIL_L: now also J14.2 (Pin_2)
- net COIL_R: now also J17.2 (Pin_2)
- net SCL_L: now also J14.3 (Pin_3)
- net SCL_R: now also J17.4 (Pin_4)
- net SDA_L: now also J14.4 (Pin_4)
- net SDA_R: now also J17.3 (Pin_3)
- net SERIAL_L: now also J14.5 (Pin_5)
- net SERIAL_R: now also J17.5 (Pin_5)
- net SHUNT_L: now also J14.6 (Pin_6)
- net SHUNT_R: now also J17.6 (Pin_6)
- new net CABLE_SHD: J14.1 (Pin_1), J17.1 (Pin_1)
Changed lines of the file:
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@@
 	(wire
 		(pts
-			(xy -24.13 168.91) (xy -24.13 172.72)
+			(xy -22.86 166.37) (xy -22.86 170.18)
 		)
 		(stroke
@@
 	(wire
 		(pts
-			(xy -26.67 168.91) (xy -26.67 172.72)
+			(xy -25.4 166.37) (xy -25.4 170.18)
 		)
 		(stroke
@@
 	(wire
 		(pts
-			(xy -31.75 168.91) (xy -31.75 172.72)
+			(xy -30.48 166.37) (xy -30.48 170.18)
 		)
 		(stroke
@@
 	(wire
 		(pts
+			(xy -17.78 166.37) (xy -17.78 170.18)
+		)
+		(stroke
+			(width 0)
+			(type default)
+		)
+	)
+	(wire
+		(pts
 			(xy 33.02 171.45) (xy 39.37 171.45)
 		)
@@
 	(wire
 		(pts
-			(xy -21.59 168.91) (xy -21.59 172.72)
+			(xy -20.32 166.37) (xy -20.32 170.18)
 		)
 		(stroke
@@
 	(wire
 		(pts
-			(xy -29.21 168.91) (xy -29.21 172.72)
+			(xy -27.94 166.37) (xy -27.94 170.18)
 		)
 		(stroke
@@
 	(wire
 		(pts
+			(xy -19.05 198.12) (xy -19.05 201.93)
+		)
+		(stroke
+			(width 0)
+			(type default)
+		)
+	)
+	(wire
+		(pts
 			(xy 273.05 38.1) (xy 273.05 39.37)
 		)
@@
 		)
 	)
+	(label "CABLE_SHD"
+		(at -17.78 170.18 270)
+		(effects
+			(font
+				(size 1.27 1.27)
+			)
+			(justify right bottom)
+		)
+	)
 	(label "5v_display"
 		(at 153.67 147.32 90)
@@
 	)
 	(label "SHUNT_L"
-		(at -31.75 172.72 270)
+		(at -30.48 170.18 270)
 		(effects
 			(font
@@
 	)
 	(label "SDA_L"
-		(at -26.67 172.72 270)
+		(at -25.4 170.18 270)
 		(effects
 			(font
@@
 		)
 	)
+	(label "CABLE_SHD"
+		(at -19.05 201.93 270)
+		(effects
+			(font
+				(size 1.27 1.27)
+			)
+			(justify right bottom)
+		)
+	)
 	(label "TFT_CS_L"
 		(at 134.62 152.4 270)
@@
 	)
 	(label "COIL_L"
-		(at -21.59 172.72 270)
+		(at -20.32 170.18 270)
 		(effects
 			(font
@@
 	)
 	(label "SERIAL_L"
-		(at -29.21 172.72 270)
+		(at -27.94 170.18 270)
 		(effects
 			(font
@@
 	)
 	(label "SCL_L"
-		(at -24.13 172.72 270)
+		(at -22.86 170.18 270)
 		(effects
 			(font
@@
 	)
 	(symbol
-		(lib_id "Connector:Conn_01x05_Pin")
-		(at -26.67 163.83 270)
-		(unit 1)
-		(body_style 1)
-		(exclude_from_sim no)
-		(in_bom yes)
-		(on_board yes)
-		(in_pos_files yes)
-		(dnp no)
-		(fields_autoplaced yes)
-		(property "Reference" "J14"
-			(at -26.67 158.75 90)
-			(show_name no)
-			(do_not_autoplace no)
-			(effects
-				(font
-					(size 1.27 1.27)
-				)
-			)
-		)
-		(property "Value" "BOARD2.L"
-			(at -26.67 161.29 90)
-			(show_name no)
-			(do_not_autoplace no)
-			(effects
-				(font
-					(size 1.27 1.27)
-				)
-			)
-		)
-		(property "Footprint" "Connector_JST:JST_XH_B5B-XH-A_1x05_P2.50mm_Vertical"
-			(at -26.67 163.83 0)
-			(hide yes)
-			(show_name no)
-			(do_not_autoplace no)
-			(effects
-				(font
-					(size 1.27 1.27)
-				)
-			)
-		)
-		(property "Datasheet" ""
-			(at -26.67 163.83 0)
-			(hide yes)
-			(show_name no)
-			(do_not_autoplace no)
-			(effects
-				(font
-					(size 1.27 1.27)
-				)
-			)
-		)
-		(property "Description" "Generic connector, single row, 01x05, script generated"
-			(at -26.67 163.83 0)
-			(hide yes)
-			(show_name no)
-			(do_not_autoplace no)
-			(effects
-				(font
-					(size 1.27 1.27)
-				)
-			)
-		)
-		(pin "1"
-		)
-		(pin "4"
-		)
-		(pin "5"
-		)
-		(pin "3"
-		)
-		(pin "2"
-		)
-		(instances
-			(project "ldr_volume"
-				(path "/94f77547-2e48-4baf-b2d8-b5c6eb42fd6e"
-					(reference "J14")
-					(unit 1)
-				)
-			)
-		)
-	)
-	(symbol
 		(lib_id "Device:R")
 		(at 210.82 154.94 0)
@@
 	)
 	(symbol
+		(lib_id "Connector:Conn_01x06_Pin")
+		(at -22.86 161.29 270)
+		(unit 1)
+		(body_style 1)
+		(exclude_from_sim no)
+		(in_bom yes)
+		(on_board yes)
+		(in_pos_files yes)
+		(dnp no)
+		(fields_autoplaced yes)
+		(property "Reference" "J14"
+			(at -24.13 156.21 90)
+			(show_name no)
+			(do_not_autoplace no)
+			(effects
+				(font
+					(size 1.27 1.27)
+				)
+			)
+		)
+		(property "Value" "BOARD2.L"
+			(at -24.13 158.75 90)
+			(show_name no)
+			(do_not_autoplace no)
+			(effects
+				(font
+					(size 1.27 1.27)
+				)
+			)
+		)
+		(property "Footprint" "Connector_JST:JST_XH_B6B-XH-A_1x06_P2.50mm_Vertical"
+			(at -22.86 161.29 0)
+			(hide yes)
+			(show_name no)
+			(do_not_autoplace no)
+			(effects
+				(font
+					(size 1.27 1.27)
+				)
+			)
+		)
+		(property "Datasheet" ""
+			(at -22.86 161.29 0)
+			(hide yes)
+			(show_name no)
+			(do_not_autoplace no)
+			(effects
+				(font
+					(size 1.27 1.27)
+				)
+			)
+		)
+		(property "Description" "Generic connector, single row, 01x06, script generated"
+			(at -22.86 161.29 0)
+			(hide yes)
+			(show_name no)
+			(do_not_autoplace no)
+			(effects
+				(font
+					(size 1.27 1.27)
+				)
+			)
+		)
+		(pin "6"
+		)
+		(pin "5"
+		)
+		(pin "4"
+		)
+		(pin "1"
+		)
+		(pin "3"
+		)
+		(pin "2"
+		)
+		(instances
+			(project "ldr_volume"
+				(path "/94f77547-2e48-4baf-b2d8-b5c6eb42fd6e"
+					(reference "J14")
+					(unit 1)
+				)
+			)
+		)
+	)
+	(symbol
 		(lib_id "Transistor_FET:2N7000")
 		(at 67.31 68.58 0)
@@
 	)
 	(symbol
-		(lib_id "Connector:Conn_01x05_Pin")
-		(at -26.67 193.04 270)
-		(unit 1)
-		(body_style 1)
-		(exclude_from_sim no)
-		(in_bom yes)
-		(on_board yes)
-		(in_pos_files yes)
-		(dnp no)
-		(fields_autoplaced yes)
-		(property "Reference" "J17"
-			(at -26.67 187.96 90)
-			(show_name no)
-			(do_not_autoplace no)
-			(effects
-				(font
-					(size 1.27 1.27)
-				)
-			)
-		)
-		(property "Value" "BOARD2.R"
-			(at -26.67 190.5 90)
-			(show_name no)
-			(do_not_autoplace no)
-			(effects
-				(font
-					(size 1.27 1.27)
-				)
-			)
-		)
-		(property "Footprint" "Connector_JST:JST_XH_B5B-XH-A_1x05_P2.50mm_Vertical"
-			(at -26.67 193.04 0)
-			(hide yes)
-			(show_name no)
-			(do_not_autoplace no)
-			(effects
-				(font
-					(size 1.27 1.27)
-				)
-			)
-		)
-		(property "Datasheet" ""
-			(at -26.67 193.04 0)
-			(hide yes)
-			(show_name no)
-			(do_not_autoplace no)
-			(effects
-				(font
-					(size 1.27 1.27)
-				)
-			)
-		)
-		(property "Description" "Generic connector, single row, 01x05, script generated"
-			(at -26.67 193.04 0)
-			(hide yes)
-			(show_name no)
-			(do_not_autoplace no)
-			(effects
-				(font
-					(size 1.27 1.27)
-				)
-			)
-		)
-		(pin "1"
-		)
-		(pin "4"
-		)
-		(pin "5"
-		)
-		(pin "3"
-		)
-		(pin "2"
-		)
-		(instances
-			(project "ldr_volume"
-				(path "/94f77547-2e48-4baf-b2d8-b5c6eb42fd6e"
-					(reference "J17")
-					(unit 1)
-				)
-			)
-		)
-	)
-	(symbol
 		(lib_id "Device:D")
 		(at 57.15 111.76 90)
@@
 					(unit 1)
 				)
+			)
+		)
+	)
+	(symbol
+		(lib_id "Connector:Conn_01x06_Pin")
+		(at -24.13 193.04 270)
+		(unit 1)
+		(body_style 1)
+		(exclude_from_sim no)
+		(in_bom yes)
+		(on_board yes)
+		(in_pos_files yes)
+		(dnp no)
+		(fields_autoplaced yes)
+		(property "Reference" "J17"
+			(at -25.4 187.96 90)
+			(show_name no)
+			(do_not_autoplace no)
+			(effects
+				(font
+					(size 1.27 1.27)
+				)
+			)
+		)
+		(property "Value" "BOARD2.R"
+			(at -25.4 190.5 90)
+			(show_name no)
+			(do_not_autoplace no)
+			(effects
+				(font
+					(size 1.27 1.27)
+				)
+			)
+		)
+		(property "Footprint" "Connector_JST:JST_XH_B6B-XH-A_1x06_P2.50mm_Vertical"
+			(at -24.13 193.04 0)
+			(hide yes)
+			(show_name no)
+			(do_not_autoplace no)
+			(effects
+				(font
+					(size 1.27 1.27)
+				)
+			)
+		)
+		(property "Datasheet" ""
+			(at -24.13 193.04 0)
+			(hide yes)
+			(show_name no)
+			(do_not_autoplace no)
+			(effects
+				(font
+					(size 1.27 1.27)
+				)
+			)
+		)
+		(property "Description" "Generic connector, single row, 01x06, script generated"
+			(at -24.13 193.04 0)
+			(hide yes)
+			(show_name no)
+			(do_not_autoplace no)
+			(effects
+				(font
+					(size 1.27 1.27)
+				)
+			)
+		)
+		(pin "6"
+		)
+		(pin "5"
+		)
+		(pin "4"
+		)
+		(pin "1"
+		)
+		(pin "3"
+		)
+		(pin "2"
+		)
+		(instances
+			(project "ldr_volume"
+				(path "/94f77547-2e48-4baf-b2d8-b5c6eb42fd6e"
+					(reference "J17")
+					(unit 1)
+				)

Commit message: updates
Parts:
- removed C17: 100uF low, Capacitor_THT:CP_Radial_D6.3mm_P2.50mm, symbol Device:C_Polarized
- removed J12, J15: TFT_PWR, Connector_JST:JST_XH_B2B-XH-A_1x02_P2.50mm_Vertical, symbol Connector:Conn_01x02_Pin
- removed J13: TFT_L, Connector_JST:JST_XH_B5B-XH-A_1x05_P2.50mm_Vertical, symbol Connector:Conn_01x05_Pin
- removed J16: TFT_R, Connector_JST:JST_XH_B5B-XH-A_1x05_P2.50mm_Vertical, symbol Connector:Conn_01x05_Pin
- added J12: Conn_01x03_Pin, Connector_JST:JST_XH_B3B-XH-A_1x03_P2.50mm_Vertical, symbol Connector:Conn_01x03_Pin
- added J13: 5v_in_b3, Connector_JST:JST_XH_B2B-XH-A_1x02_P2.50mm_Vertical, symbol Connector:Conn_01x02_Pin
- added NT3, NT4: NetTie_2, nettie 1.0:NetTie-2_SMD_Pad1.0o, symbol Device:NetTie_2
- added R23: 100R, Resistor_THT:R_Axial_DIN0207_L6.3mm_D2.5mm_P7.62mm_Horizontal, symbol Device:R
- added U5: 4N25, Package_DIP:DIP-6_W7.62mm, symbol Isolator:4N25
- renumbered J17 to J15
Connections:
- net 3.3V_PICO: now also R23.2
- net CABLE_SHD: now also NT3.1, NT4.1
- net GNDD: now also J12.1 (Pin_1), NT3.2, NT4.2, U5.2
- net UART_RX: now reaches A1.21 (GPIO16)
- net UART_RX: now also J12.3 (Pin_3)
- net TFT_CS_L renamed UART_TX
- net UART_TX: now also J12.2 (Pin_2)
- net TFT_CS_R: no longer names the net of A1.26 (GPIO20)
- net TFT_DC_RS: no longer names the net of A1.27 (GPIO21)
- net TFT_MOSI: no longer names the net of A1.25 (GPIO19)
- net TFT_RST_RES: no longer names the net of A1.29 (GPIO22)
- net TFT_SCK renamed MUTE_CTRL
- net MUTE_CTRL: now also R23.1, U5.1
- new net AMP_GND_PIN: J13.1 (Pin_1), U5.4
- new net AMP_MUTE_PIN: J13.2 (Pin_2), U5.5

Commit message: updates
Parts:
- removed J12: Conn_01x03_Pin, Connector_JST:JST_XH_B3B-XH-A_1x03_P2.50mm_Vertical, symbol Connector:Conn_01x03_Pin
- removed J13: 5v_in_b3, Connector_JST:JST_XH_B2B-XH-A_1x02_P2.50mm_Vertical, symbol Connector:Conn_01x02_Pin
- removed R2, R23: 100R, Resistor_THT:R_Axial_DIN0207_L6.3mm_D2.5mm_P7.62mm_Horizontal, symbol Device:R
- added C13, C14, C25, C26: 100nF, Capacitor_THT:C_Disc_D5.0mm_W2.5mm_P5.00mm, symbol Device:C
- added J11: UART_EXT1, Connector_JST:JST_XH_B5B-XH-A_1x05_P2.50mm_Vertical, symbol Connector:Conn_01x05_Pin
- added J12: EXT2, Connector_JST:JST_XH_B4B-XH-A_1x04_P2.50mm_Vertical, symbol Connector:Conn_01x04_Pin
- added J13: MUTE, Connector_JST:JST_XH_B3B-XH-A_1x03_P2.50mm_Vertical, symbol Connector:Conn_01x03_Pin
- added NT8: NetTie_2, nettie 1.0:NetTie-2_SMD_Pad1.0o, symbol Device:NetTie_2
- added Q7: 2N7000, Package_TO_SOT_THT:TO-92_Inline_Wide, symbol Transistor_FET:2N7000
- added R15: 240, Resistor_THT:R_Axial_DIN0207_L6.3mm_D2.5mm_P7.62mm_Horizontal, symbol Device:R
- added R17: 10K, Resistor_THT:R_Axial_DIN0207_L6.3mm_D2.5mm_P7.62mm_Horizontal, symbol Device:R
- added R3: 100R, Resistor_THT:R_Axial_DIN0207_L6.3mm_D2.5mm_P7.62mm_Horizontal, symbol Device:R
- C1, C15, C16, C2: value 1uF -> 100nF; footprint Capacitor_THT:C_Disc_D7.5mm_W2.5mm_P5.00mm -> Capacitor_THT:C_Disc_D5.0mm_W2.5mm_P5.00mm
- C28: renamed from C14; footprint Capacitor_THT:C_Rect_L7.2mm_W2.5mm_P5.00mm_FKS2_FKP2_MKS2_MKP2 -> Capacitor_THT:C_Disc_D5.0mm_W2.5mm_P5.00mm
- J15: renamed from J11; value 5v_in_b3 -> PWR_IN
- R10, R13, R14, R9: value 10K -> 4.7K
- R5, R6, R7, R8: value 100R -> 4.7K
- renumbered C13 to C27, J15 to J23, R21 to R16, R15 to R18, R22 to R19, R3 to R2, R16 to R20, R17 to R21, R18 to R22, R19 to R23, R20 to R31
Connections:
- net 3.3V_PICO: now also R17.1
- net 5V_board1: now also U5.1, R3.1
- net AMP_GND_PIN: now also J13.2 (Pin_2)
- net AMP_MUTE_PIN: now also J13.3 (Pin_3)
- net CABLE_SHD: now also J13.1 (Pin_1), NT8.1
- net COIL_L: now also J14.6 (Pin_6), Q5.3 (D); no longer J14.2 (Pin_2), Q6.3 (D)
- net COIL_R: now also J23.6 (Pin_6), Q6.3 (D); no longer J23.2 (Pin_2), Q5.3 (D)
- net GNDD: now also C13.2, C14.2, C25.2, C26.2, J11.3 (Pin_3), J12.2 (Pin_2), NT8.2, Q7.1 (S); no longer R10.2, R13.2, R14.2, R9.2, U5.2
- net MUTE_CTRL: now also A1.32 (GPIO27_ADC1), Q7.2 (G), R17.2; no longer A1.24 (GPIO18), U5.1
- net PWM_SER_L: no longer R9.1
- net PWM_SER_R: now also R7.1; no longer R10.1, R6.1
- net PWM_SHUNT_L: now also A1.1 (GPIO0), R9.1; no longer A1.4 (GPIO2), R13.1, R7.1
- net PWM_SHUNT_R: now also A1.20 (GPIO15), R13.1; no longer A1.17 (GPIO13), R14.1, R8.1
- net SCL_L: now also J14.5 (Pin_5); no longer J14.3 (Pin_3)
- net SDA_R: now also J23.5 (Pin_5); no longer J23.3 (Pin_3)
- net SERIAL_L: now also J14.3 (Pin_3); no longer C15.1, J14.5 (Pin_5)
- net SERIAL_R: now also J23.3 (Pin_3), R1.2; no longer C16.1, J23.5 (Pin_5), R4.2
- net SHUNT_L: now also J14.2 (Pin_2), R3.2; no longer C1.1, J14.6 (Pin_6), R1.2
- net SHUNT_R: now also J23.2 (Pin_2), R4.2; no longer C2.1, J23.6 (Pin_6)
- net SPI0_TX: now reaches A1.25 (GPIO19)
- net SPI0_TX: now also J11.1 (Pin_1)
- net GP20: now reaches A1.26 (GPIO20)
- net GP20: now also J12.4 (Pin_4)
- net GP21: now reaches A1.27 (GPIO21)
- net GP21: now also J12.3 (Pin_3)
- net GP22: now reaches A1.29 (GPIO22)
- net GP22: now also J12.1 (Pin_1)
- net at R8.2: now also Q2.2 (G), C14.1; no longer Q4.2 (G)
- net at Q5.2 (G): now also R16.2; no longer R18.2
- net at Q1.2 (G): now also C2.1, R6.2; no longer R5.2
- net at Q3.2 (G): now also C16.1, R10.2; no longer R7.2
- net at Q6.2 (G): now also R18.2; no longer R16.2
- net UART_RX renamed SPI0_RX
- net SPI0_RX: now also J11.5 (Pin_5)
- net UART_TX renamed SPI0_CSN
- net SPI0_CSN: now also J11.4 (Pin_4)
- new net: C15.1, R10.1, R9.2
- new net: C13.1, R7.2, R8.1
- new net: C26.1, Q4.2 (G), R14.2
- new net: C25.1, R13.2, R14.1
- new net: Q7.3 (D), R15.1
- new net: R15.2, U5.2
- new net: C1.1, R5.2, R6.1
- new net SPI0_SCK: A1.24 (GPIO18), J11.2 (Pin_2)
Other:
- moved on the sheet: A1, C27, C28, D2, J14, J15, J23, NT3, NT4, R16, R18, R19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

Commit message: updates
Parts:
- removed C15, C16, C25, C26: 100nF, Capacitor_THT:C_Disc_D5.0mm_W2.5mm_P5.00mm, symbol Device:C
- removed J14: BOARD2.L, Connector_JST:JST_XH_B6B-XH-A_1x06_P2.50mm_Vertical, symbol Connector:Conn_01x06_Pin
- removed J23: BOARD2.R, Connector_JST:JST_XH_B6B-XH-A_1x06_P2.50mm_Vertical, symbol Connector:Conn_01x06_Pin
- removed Q1, Q2, Q3, Q4: 2N7000, Package_TO_SOT_THT:TO-92_Inline_Wide, symbol Transistor_FET:2N7000
- added J14: LDR_R, Connector_JST:JST_XH_B4B-XH-A_1x04_P2.50mm_Vertical, symbol Connector:Conn_01x04_Pin
- added J15: LDR_L, Connector_JST:JST_XH_B4B-XH-A_1x04_P2.50mm_Vertical, symbol Connector:Conn_01x04_Pin
- added J24, J25: I2C, Connector_JST:JST_XH_B2B-XH-A_1x02_P2.50mm_Vertical, symbol Connector:Conn_01x02_Pin
- added Q1, Q3, Q5, Q7: BC547, Package_TO_SOT_THT:TO-92_Inline_Wide, symbol Transistor_BJT:BC547
- added Q2, Q4, Q6, Q8: BC557, Package_TO_SOT_THT:TO-92_Inline_Wide, symbol Transistor_BJT:BC557
- C1, C13, C14, C2: value 100nF -> 1uF
- R1, R2: value 100R -> 110
- R10, R14, R6: value 4.7K -> 10K
- R13, R5, R9: value 4.7K -> 100K; footprint Resistor_THT:R_Axial_DIN0207_L6.3mm_D2.5mm_P7.62mm_Horizontal -> Resistor_THT:R_Axial_DIN0207_L6.3mm_D2.5mm_P2.54mm_Vertical
- R3: value 100R -> 100K; footprint Resistor_THT:R_Axial_DIN0207_L6.3mm_D2.5mm_P7.62mm_Horizontal -> Resistor_THT:R_Axial_DIN0207_L6.3mm_D2.5mm_P2.54mm_Vertical
- R4: value 100R -> 10K
- R7, R8: value 4.7K -> 110
- renumbered C27 to C15, C28 to C16, J15 to J23, Q5 to Q11, Q7 to Q12, Q6 to Q13, R17 to R16, R16 to R17
Connections:
- net 5V_board1: now also R1.2, R2.2, R7.2, R8.2; no longer R1.1, R2.1, R3.1, R4.1
- net CABLE_SHD: now also J14.1 (Pin_1), J15.1 (Pin_1)
- net COIL_CTRL_L: now also A1.5 (GPIO3); no longer A1.9 (GPIO6)
- net COIL_CTRL_R: now also A1.16 (GPIO12); no longer A1.12 (GPIO9)
- net COIL_L: now also J15.4 (Pin_4)
- net COIL_R: now also J14.4 (Pin_4)
- net PWM_SER_L: now also A1.9 (GPIO6), R4.2; no longer A1.5 (GPIO3), R5.1
- net PWM_SER_R: now also A1.12 (GPIO9), R10.2; no longer A1.16 (GPIO12), R7.1
- net PWM_SHUNT_L: now also A1.2 (GPIO1), R6.2; no longer A1.1 (GPIO0), R9.1
- net PWM_SHUNT_R: now also A1.19 (GPIO14), R14.2; no longer A1.20 (GPIO15), R13.1
- net SCL_L: now also J24.1 (Pin_1)
- net SCL_R: now also J25.1 (Pin_1)
- net SDA_L: now also J24.2 (Pin_2)
- net SDA_R: now also J25.2 (Pin_2)
- net SERIAL_L: now also J15.2 (Pin_2), Q2.1 (C); no longer R2.2
- net SERIAL_R: now also J14.2 (Pin_2), Q6.1 (C); no longer R1.2
- net SHUNT_L: now also J15.3 (Pin_3), Q4.1 (C); no longer R3.2
- net SHUNT_R: now also J14.3 (Pin_3), Q8.1 (C); no longer R4.2
- net at C14.1: now also R14.1, Q7.2 (B); no longer R8.2
- net at R10.1: now also C13.1, Q5.2 (B); no longer R9.2
- net at R13.2: now also R8.1, Q7.3 (E), Q8.3 (E); no longer R14.1
- net at C2.1: now also R6.1, Q3.2 (B); no longer R6.2
- new net: Q1.1 (C), Q2.2 (B), R3.1
- new net: C1.1, Q1.2 (B), R4.1
- new net: Q1.3 (E), Q2.3 (E), R1.1, R3.2
- new net: Q7.1 (C), Q8.2 (B), R13.1
- new net: Q3.1 (C), Q4.2 (B), R5.1
- new net: Q3.3 (E), Q4.3 (E), R2.1, R5.2
- new net: Q5.1 (C), Q6.2 (B), R9.1
- new net: Q5.3 (E), Q6.3 (E), R7.1, R9.2
Other:
- moved on the sheet: Q12, R15, R16, U5

Commit message: updataes
Parts:
- C1, C13, C14, C2: value 1uF -> 100nF
- R1, R2, R7, R8: value 110 -> 120
- renumbered R31 to R29
Changed lines of the file:
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@@
 			)
 		)
-		(property "Value" "1uF"
+		(property "Value" "100nF"
 			(at 61.976 -144.78 0)
 			(show_name no)
@@
 			)
 		)
-		(property "Value" "110"
+		(property "Value" "120"
 			(at 117.856 -222.25 90)
 			(show_name no)
@@
 			)
 		)
-		(property "Value" "110"
+		(property "Value" "120"
 			(at 116.586 -161.29 90)
 			(show_name no)
@@
 			)
 		)
-		(property "Value" "1uF"
+		(property "Value" "100nF"
 			(at 63.246 -205.74 0)
 			(show_name no)
@@
 			)
 		)
-		(property "Value" "110"
+		(property "Value" "120"
 			(at 41.656 -227.33 90)
 			(show_name no)
@@
 			)
 		)
-		(property "Value" "1uF"
+		(property "Value" "100nF"
 			(at 139.446 -200.66 0)
 			(show_name no)
@@
 		(in_pos_files yes)
 		(dnp no)
-		(property "Reference" "R31"
+		(property "Reference" "R29"
 			(at 255.016 50.546 0)
 			(show_name no)
@@
 			(project "ldr_volume"
 				(path "/94f77547-2e48-4baf-b2d8-b5c6eb42fd6e"
-					(reference "R31")
+					(reference "R29")
 					(unit 1)
 				)
@@
 			)
 		)
-		(property "Value" "1uF"
+		(property "Value" "100nF"
 			(at 138.176 -139.7 0)
 			(show_name no)
@@
 			)
 		)
-		(property "Value" "110"
+		(property "Value" "120"
 			(at 40.386 -166.37 90)
 			(show_name no)

Commit message: updates
Parts:
- removed J24, J25: I2C, Connector_JST:JST_XH_B2B-XH-A_1x02_P2.50mm_Vertical, symbol Connector:Conn_01x02_Pin
- removed NT4, NT8: NetTie_2, nettie 1.0:NetTie-2_SMD_Pad1.0o, symbol Device:NetTie_2
- added J24: I2C_L, Connector_JST:JST_XH_B3B-XH-A_1x03_P2.50mm_Vertical, symbol Connector:Conn_01x03_Pin
- added J25: I2C_R, Connector_JST:JST_XH_B3B-XH-A_1x03_P2.50mm_Vertical, symbol Connector:Conn_01x03_Pin
- C1, C2: value 100nF -> 10nF
- C11: renamed from C13; value 100nF -> 10nF
- C12: renamed from C14; value 100nF -> 10nF
- NT3: value NetTie_2 -> mute_cable
- renumbered C15 to C13, C16 to C14
Connections:
- net CABLE_SHD: no longer J14.1 (Pin_1), J15.1 (Pin_1)
- net GNDD: now also J14.2 (Pin_2), J15.2 (Pin_2), J24.1 (Pin_1), J25.1 (Pin_1)
- net PWM_SER_L: now also A1.2 (GPIO1), R6.2; no longer A1.9 (GPIO6), R4.2
- net PWM_SER_R: now also A1.19 (GPIO14), R14.2; no longer A1.12 (GPIO9), R10.2
- net PWM_SHUNT_L: now also A1.9 (GPIO6), R4.2; no longer A1.2 (GPIO1), R6.2
- net PWM_SHUNT_R: now also A1.12 (GPIO9), R10.2; no longer A1.19 (GPIO14), R14.2
- net SCL_L: now also J24.2 (Pin_2)
- net SCL_R: now also J25.3 (Pin_3)
- net SDA_L: now also J24.3 (Pin_3)
- net SDA_R: now also J25.2 (Pin_2)
- net SERIAL_L: now also J15.3 (Pin_3), Q4.1 (C); no longer J15.2 (Pin_2), Q2.1 (C)
- net SERIAL_R: now also J14.3 (Pin_3), Q8.1 (C); no longer J14.2 (Pin_2), Q6.1 (C)
- net SHUNT_L: now also J15.1 (Pin_1), Q2.1 (C); no longer J15.3 (Pin_3), Q4.1 (C)
- net SHUNT_R: now also J14.1 (Pin_1), Q6.1 (C); no longer J14.3 (Pin_3), Q8.1 (C)
Other:
- note added: "Non-twisted wire 3 wires + shield LiYCY 3 x 0.34mm2 For LDR + relay coil interconnect, shield goes to GNDD on board#3. No other gnd connection needed"
- note added: "Twisted wire 1 pair + shield LiYCY 1x2x0.5mm2 For main board interconnect +5V and GND , shield connects to board#1 only"
- note added: "Twisted wires 2 pairs + shield - LiYCY paar 2x2x 0.25mm2 For i2c interconnect, Pairs - SDA+GND, SCL+GND Shield connected on board#3 only together with both pairs gnd return. Both gnd pairs connect together on board#2 and connect to gnda"

Commit message: updates
Parts:
- renumbered J13 to J11, J11 to J12, J12 to J13
Connections:
- net AMP_GND_PIN: now also J11.3 (Pin_3); no longer J11.2 (Pin_2)
- net AMP_MUTE_PIN: now also J11.2 (Pin_2); no longer J11.3 (Pin_3)
Other:
- moved on the sheet: C13, C14, J11, NT3, R21, R22, R23, R29

Commit message: update
Parts:
- removed J13: EXT2, Connector_JST:JST_XH_B4B-XH-A_1x04_P2.50mm_Vertical, symbol Connector:Conn_01x04_Pin
- removed Q12: 2N7000, Package_TO_SOT_THT:TO-92_Inline_Wide, symbol Transistor_FET:2N7000
- R15: value 240 -> 300; footprint Resistor_THT:R_Axial_DIN0207_L6.3mm_D2.5mm_P7.62mm_Horizontal -> Resistor_THT:R_Axial_DIN0207_L6.3mm_D2.5mm_P2.54mm_Vertical
- renumbered Q13 to Q12, R17 to R16, R18 to R17, R19 to R18, R20 to R19, R16 to R20, U5 to U4
Connections:
- net 3.3V_PICO: now also R15.2; no longer R20.1
- net 5V_board1: no longer U4.1
- net GNDD: now also R20.2
- net MUTE_CTRL: now also R20.1, U4.2; no longer R20.2
- net at R15.1: now also U4.1
- net GP20: no longer names the net of A1.26 (GPIO20)
- net GP21: no longer names the net of A1.27 (GPIO21)
- net GP22: no longer names the net of A1.29 (GPIO22)
Other:
- note added: "Operational Verification At Boot (GPIO = Input/Hi-Z): Current flows: 3.3V → 300Ω → LED → Junction → 10kΩ Pull-Down → GND. Since 10kΩ is much larger than 300Ω, it does not significantly limit current. Result: LED is ON (~7mA). To Turn OFF (GPIO = Output High/3.3V): The MCU drives the Junction to 3.3V. Voltage across LED = 3.3V (Anode) - 3.3V (Cathode) = 0V. Result: LED is OFF (0mA current draw). T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"
- moved on the sheet: R15, R20, U4
