File: amp_v3/ldr_volume/testboard.kicad_sch (KiCad schematic)
At the start: 7 parts, among them Q10 BC557, Q9 BC547, U6 NSL-32-SR3-Rshunt

Commit message: updataes
Parts:
- C24: value 1uF -> 100nF
- U6: value NSL-32-SR3-Rshunt -> NSL-32-SR3
Changed lines of the file:
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@@
 			)
 		)
-		(property "Value" "NSL-32-SR3-Rshunt"
+		(property "Value" "NSL-32-SR3"
 			(at 52.832 98.806 0)
 			(show_name no)
@@
 			)
 		)
-		(property "Value" "1uF"
+		(property "Value" "100nF"
 			(at 114.046 76.2 0)
 			(show_name no)

Commit message: update
Parts:
- added C30: 100nF, Capacitor_THT:C_Disc_D5.0mm_W2.5mm_P5.00mm, symbol Device:C
- added J13: NTC, Connector_JST:JST_XH_B2B-XH-A_1x02_P2.50mm_Vertical, symbol Connector:Conn_01x02_Pin
- added NT4: GNDD_TO_GNDA, nettie 1.0:NetTie-2_SMD_Pad1.0o, symbol Device:NetTie_2
- added R30: 10K, Resistor_THT:R_Axial_DIN0207_L6.3mm_D2.5mm_P7.62mm_Horizontal, symbol Device:R
Connections:
- net GNDD: now also NT4.1
- new net 3.3V_PICO: J13.2 (Pin_2)
- new net GNDA: C30.2, NT4.2, R30.2
- new net TEMP_IN: C30.1, J13.1 (Pin_1), R30.1

Commit message: updates
Parts:
- added C27: 4.7uF, symbol selector_ctrl-rescue:CP1
- added J27: IR, Connector_JST:JST_XH_B3B-XH-A_1x03_P2.50mm_Vertical, symbol Connector:Conn_01x03_Pin
- added R34: 100R, symbol selector_ctrl-rescue:R
- renumbered C30 to C26, R32 to R30, R33 to R31, R34 to R32, R30 to R33, U6 to U5
Connections:
- net 3.3V_PICO: now also R34.1
- new net: C27.1, J27.2 (Pin_2), R34.2
- new net GND: C27.2, J27.1 (Pin_1)
- new net IR: J27.3 (Pin_3)
Other:
- note added: "TSOP31238"

Commit message: update
Parts:
- removed C27: 4.7uF, symbol selector_ctrl-rescue:CP1
- removed J27: IR, Connector_JST:JST_XH_B3B-XH-A_1x03_P2.50mm_Vertical, symbol Connector:Conn_01x03_Pin
- removed R34: 100R, symbol selector_ctrl-rescue:R
Other:
- note removed: "TSOP31238"
