File: amp_v3/ldr_volume/board#1.kicad_sch (KiCad schematic)
At the start: 8 parts, among them J6 Conn_01x02_Pin, J7 Conn_01x02_Pin, J8 Conn_01x02_Pin, J9 Conn_01x02_Pin, U4 IRM-20-5

Commit message: updates
Parts:
- added C12: 100nF, Capacitor_THT:C_Rect_L7.2mm_W2.5mm_P5.00mm_FKS2_FKP2_MKS2_MKP2, symbol Device:C
- added J9: Conn_01x02_Pin, Connector_JST:JST_XH_B2B-XH-A_1x02_P2.50mm_Vertical, symbol Connector:Conn_01x02_Pin
- C18: renamed from C12; value 100uF -> 470uF; footprint Capacitor_THT:CP_Radial_D6.3mm_P2.50mm -> Capacitor_THT:CP_Radial_D8.0mm_P3.80mm
- renumbered J9 to J18
Connections:
- net 5V_board1: now also J9.2 (Pin_2)
- net GNDD: now also C12.2, J9.1 (Pin_1)
- net at C11.1, L1.1, U4.4 (+Vo): now also C12.1

Commit message: updates
Parts:
- C12: footprint Capacitor_THT:C_Rect_L7.2mm_W2.5mm_P5.00mm_FKS2_FKP2_MKS2_MKP2 -> Capacitor_THT:C_Disc_D5.0mm_W2.5mm_P5.00mm
- L1: footprint Inductor_THT:L_Radial_D9.5mm_P5.00mm_Fastron_07HVP -> Inductor_THT:L_Radial_D8.7mm_P5.00mm_Fastron_07HCP
Changed lines of the file:
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@@
 			)
 		)
-		(property "Footprint" "Inductor_THT:L_Radial_D9.5mm_P5.00mm_Fastron_07HVP"
+		(property "Footprint" "Inductor_THT:L_Radial_D8.7mm_P5.00mm_Fastron_07HCP"
 			(at 97.79 48.26 0)
 			(hide yes)
@@
 			)
 		)
-		(property "Footprint" "Capacitor_THT:C_Rect_L7.2mm_W2.5mm_P5.00mm_FKS2_FKP2_MKS2_MKP2"
+		(property "Footprint" "Capacitor_THT:C_Disc_D5.0mm_W2.5mm_P5.00mm"
 			(at 88.5952 58.42 0)
 			(hide yes)

Commit message: updates
Parts:
- J6: value Conn_01x02_Pin -> PWR1
- J7: value Conn_01x02_Pin -> PWR2
- J8: value Conn_01x02_Pin -> PWR3
- J9: value Conn_01x02_Pin -> PWR4
- renumbered C11 to C3, C12 to C4, C18 to C5
Changed lines of the file:
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@@
 		(dnp no)
 		(fields_autoplaced yes)
-		(property "Reference" "#PWR026"
+		(property "Reference" "#PWR020"
 			(at 125.73 38.1 0)
 			(hide yes)
@@
 			(project "ldr_volume"
 				(path "/4c316523-e3a9-424b-9fb2-25fa254a8a5b"
-					(reference "#PWR026")
+					(reference "#PWR020")
 					(unit 1)
 				)
@@
 		(in_pos_files yes)
 		(dnp no)
-		(property "Reference" "C11"
+		(property "Reference" "C3"
 			(at 81.28 60.452 0)
 			(show_name no)
@@
 			(project "ldr_volume"
 				(path "/4c316523-e3a9-424b-9fb2-25fa254a8a5b"
-					(reference "C11")
+					(reference "C3")
 					(unit 1)
 				)
@@
 			)
 		)
-		(property "Value" "Conn_01x02_Pin"
+		(property "Value" "PWR3"
 			(at 99.06 24.7649 90)
 			(show_name no)
@@
 			)
 		)
-		(property "Value" "Conn_01x02_Pin"
+		(property "Value" "PWR2"
 			(at 71.12 24.7649 90)
 			(show_name no)
@@
 		(in_pos_files yes)
 		(dnp no)
-		(property "Reference" "C12"
+		(property "Reference" "C4"
 			(at 86.614 60.452 0)
 			(show_name no)
@@
 			(project "ldr_volume"
 				(path "/4c316523-e3a9-424b-9fb2-25fa254a8a5b"
-					(reference "C12")
+					(reference "C4")
 					(unit 1)
 				)
@@
 		(dnp no)
 		(fields_autoplaced yes)
-		(property "Reference" "C18"
+		(property "Reference" "C5"
 			(at 115.57 52.4509 0)
 			(show_name no)
@@
 			(project "ldr_volume"
 				(path "/4c316523-e3a9-424b-9fb2-25fa254a8a5b"
-					(reference "C18")
+					(reference "C5")
 					(unit 1)
 				)
@@
 		(dnp no)
 		(fields_autoplaced yes)
-		(property "Reference" "#PWR045"
+		(property "Reference" "#PWR025"
 			(at 97.79 68.58 0)
 			(hide yes)
@@
 			(project "ldr_volume"
 				(path "/4c316523-e3a9-424b-9fb2-25fa254a8a5b"
-					(reference "#PWR045")
+					(reference "#PWR025")
 					(unit 1)
 				)
@@
 			)
 		)
-		(property "Value" "Conn_01x02_Pin"
+		(property "Value" "PWR4"
 			(at 127 24.7649 90)
 			(show_name no)
@@
 		(dnp no)
 		(fields_autoplaced yes)
-		(property "Reference" "#PWR025"
+		(property "Reference" "#PWR019"
 			(at 97.79 38.1 0)
 			(hide yes)
@@
 			(project "ldr_volume"
 				(path "/4c316523-e3a9-424b-9fb2-25fa254a8a5b"
-					(reference "#PWR025")
+					(reference "#PWR019")
 					(unit 1)
 				)
@@
 			)
 		)
-		(property "Value" "Conn_01x02_Pin"
+		(property "Value" "PWR1"
 			(at 43.18 24.7649 90)
 			(show_name no)

Commit message: updates
Parts:
- C5: value 470uF -> 100uF; footprint Capacitor_THT:CP_Radial_D8.0mm_P3.80mm -> Capacitor_THT:CP_Radial_D6.3mm_P2.50mm
- J18: value Conn_01x02_Pin -> AC_IN; footprint TerminalBlock_Phoenix:TerminalBlock_Phoenix_MKDS-3-2-5.08_1x02_P5.08mm_Horizontal -> TerminalBlock_Phoenix:TerminalBlock_Phoenix_PT-1,5-2-5.0-H_1x02_P5.00mm_Horizontal
Changed lines of the file:
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@@
 			)
 		)
-		(property "Value" "Conn_01x02_Pin"
+		(property "Value" "AC_IN"
 			(at 27.305 50.8 0)
 			(show_name no)
@@
 			)
 		)
-		(property "Footprint" "TerminalBlock_Phoenix:TerminalBlock_Phoenix_MKDS-3-2-5.08_1x02_P5.08mm_Horizontal"
+		(property "Footprint" "TerminalBlock_Phoenix:TerminalBlock_Phoenix_PT-1,5-2-5.0-H_1x02_P5.00mm_Horizontal"
 			(at 26.67 53.34 0)
 			(hide yes)
@@
 			)
 		)
-		(property "Value" "470uF"
+		(property "Value" "100uF"
 			(at 115.57 54.9909 0)
 			(show_name no)
@@
 			)
 		)
-		(property "Footprint" "Capacitor_THT:CP_Radial_D8.0mm_P3.80mm"
+		(property "Footprint" "Capacitor_THT:CP_Radial_D6.3mm_P2.50mm"
 			(at 112.7252 58.42 0)
 			(hide yes)

Commit message: updates
Parts:
- removed U4: IRM-20-5, Converter_ACDC:Converter_ACDC_MeanWell_IRM-20-xx_THT, symbol Converter_ACDC:IRM-20-5
- added C22, C25, C27, C29: 100nF, Capacitor_THT:C_Disc_D5.0mm_W2.5mm_P5.00mm, symbol Device:C
- added C26, C28, C5: 100uF, Capacitor_THT:CP_Radial_D6.3mm_P2.50mm, symbol Device:C_Polarized
- added J26: 5V_IN, Connector_JST:JST_XH_B2B-XH-A_1x02_P2.50mm_Vertical, symbol Connector:Conn_01x02_Pin
- added L2, L3: L_Coupled, Inductor_THT:Choke_Schaffner_RN202-04-8.8x18.2mm, symbol Device:L_Coupled
- J18: value AC_IN -> 5V_IN; footprint TerminalBlock_Phoenix:TerminalBlock_Phoenix_PT-1,5-2-5.0-H_1x02_P5.00mm_Horizontal -> Connector_JST:JST_XH_B2B-XH-A_1x02_P2.50mm_Vertical
- renumbered C5 to C23
Connections:
- net 5V_board1: now also C28.1, C29.1, L3.2; no longer C23.1, J8.2 (Pin_2), J9.2 (Pin_2), L1.2
- net GNDD: now also C22.2, C25.2, C28.2, C29.2, C5.2, L2.4, L3.4; no longer C3.2, C4.2
- net 5V_IRM: now reaches J18.1 (Pin_1)
- net 5V_IRM: now also C3.1, C4.1, C26.1, C27.1, J26.1 (Pin_1), L2.1, L3.1
- net GND_IRM: now reaches J18.2 (Pin_2)
- net GND_IRM: now also C3.2, C4.2, C26.2, C27.2, J26.2 (Pin_2), L2.3, L3.3
- new net: C22.1, C5.1, L1.1, L2.2
- new net 5V_analog: C23.1, C25.1, J8.2 (Pin_2), J9.2 (Pin_2), L1.2
Other:
- moved on the sheet: C23, C3, C4, L1

Commit message: updates
Parts:
- removed C22, C27, C29: 100nF, Capacitor_THT:C_Disc_D5.0mm_W2.5mm_P5.00mm, symbol Device:C
- removed C26, C28, C3, C5: 100uF, Capacitor_THT:CP_Radial_D6.3mm_P2.50mm, symbol Device:C_Polarized
- added C22: 100uF (low esr), Capacitor_THT:CP_Radial_D6.3mm_P2.50mm, symbol Device:C_Polarized
- added C23: 10uF, Capacitor_THT:C_Disc_D5.0mm_W2.5mm_P5.00mm, symbol Device:C
- added C25: 100nF (X7R), Capacitor_THT:C_Disc_D5.0mm_W2.5mm_P5.00mm, symbol Device:C
- added L3: 10uH, Inductor_THT:L_Radial_D8.7mm_P5.00mm_Fastron_07HCP, symbol Device:L
- C3: renamed from C23; value 100uF -> 100uF (low esr)
- C4: value 100nF -> 10uF
- C5: renamed from C25; value 100nF -> 100nF (X7R)
- L1: value 4.7uH -> 10uH
- L2: value L_Coupled -> RN202-0.3-02-12M
- L4: renamed from L3; value L_Coupled -> RN-202-1/02
Connections:
- net 5V_IRM: no longer C4.1
- net 5V_analog: now also C4.1
- net 5V_board1: now also C22.1, C23.1, C25.1, L3.2; no longer L4.2
- net GNDD: now also C4.2, C22.2, C23.2, C25.2
- net GND_IRM: no longer C4.2
- new net: L3.1, L4.2
Other:
- moved on the sheet: C3, J18, J26, L1

Commit message: updates
Parts:
- added J18: PWR3, Connector_JST:JST_XH_B2B-XH-A_1x02_P2.50mm_Vertical, symbol Connector:Conn_01x02_Pin
- added J25: PWR4, Connector_JST:JST_XH_B2B-XH-A_1x02_P2.50mm_Vertical, symbol Connector:Conn_01x02_Pin
- added J26: Conn_01x03_Pin, Connector_JST:JST_XH_B3B-XH-A_1x03_P2.50mm_Vertical, symbol Connector:Conn_01x03_Pin
- added U7: IRM-10-5, Converter_ACDC:Converter_ACDC_MeanWell_IRM-10-xx_THT, symbol Converter_ACDC:IRM-10-5
- L1, L3: footprint Inductor_THT:L_Radial_D8.7mm_P5.00mm_Fastron_07HCP -> Inductor_THT:L_Radial_D7.8mm_P5.00mm_Fastron_07HCP
- renumbered J18 to J27, J26 to J28
Connections:
- net 5V_IRM: now also J18.2 (Pin_2), J25.2 (Pin_2), U7.4 (+Vo)
- net GND_IRM: now also J18.1 (Pin_1), J25.1 (Pin_1), U7.3 (-Vo)
- new net: J26.1 (Pin_1), U7.2 (AC/L)
- new net: J26.3 (Pin_3), U7.1 (AC/N)
- no-connect marks 0 -> 1
