File: amp_v3/ldr_volume/board#5.kicad_sch (KiCad schematic)
At the start: 18 parts, among them J16 5v_in_b3, J17 Conn_01x03_Pin, J20 LEFT_TFT, J23 RIGHT_TFT, J24 TFT_PWR, J25 TFT_PWR

Commit message: updates
Parts:
- C19: footprint Capacitor_THT:C_Rect_L7.2mm_W2.5mm_P5.00mm_FKS2_FKP2_MKS2_MKP2 -> Capacitor_THT:C_Disc_D5.0mm_W2.5mm_P5.00mm
- renumbered J20 to J19, J23 to J20, J24 to J21, J25 to J22
Connections:
- net UART_RX: no longer A2.21 (GPIO16)
- net UART_TX: no longer A2.22 (GPIO17)
- net TFT_DC_R: now reaches A2.24 (GPIO18)
- net TFT_DC_R: now also J20.6 (Pin_6)
- net TFT_RES_R: now reaches A2.25 (GPIO19)
- net TFT_RES_R: now also J20.5 (Pin_5)
- net TFT_SCL_R: now reaches A2.26 (GPIO20)
- net TFT_SCL_R: now also J20.3 (Pin_3)
- net TFT_SDA_R: now reaches A2.27 (GPIO21)
- net TFT_SDA_R: now also J20.4 (Pin_4)
- net TFT_SCL_L: now reaches A2.4 (GPIO2)
- net TFT_SCL_L: now also J19.3 (Pin_3)
- net TFT_SDA_L: now reaches A2.5 (GPIO3)
- net TFT_SDA_L: now also J19.4 (Pin_4)
- net TFT_RES_L: now reaches A2.6 (GPIO4)
- net TFT_RES_L: now also J19.5 (Pin_5)
- net TFT_DC_L: now reaches A2.7 (GPIO5)
- net TFT_DC_L: now also J19.6 (Pin_6)
- net TFT_CS_L: now reaches A2.9 (GPIO6)
- net TFT_CS_L: now also J19.7 (Pin_7)
- net TFT_BL renamed TFT_BL_L
- net TFT_BL_L: no longer J20.8 (Pin_8)
- net TFT_CS renamed TFT_CS_R
- net TFT_CS_R: now also A2.22 (GPIO17); no longer J19.7 (Pin_7)
- removed net TFT_DC: J19.6 (Pin_6), J20.6 (Pin_6)
- net TFT_GND renamed TFT_GND_L
- net TFT_GND_L: no longer J20.1 (Pin_1)
- removed net TFT_RES: J19.5 (Pin_5), J20.5 (Pin_5)
- removed net TFT_SCL: J19.3 (Pin_3), J20.3 (Pin_3)
- removed net TFT_SDA: J19.4 (Pin_4), J20.4 (Pin_4)
- net TFT_VDD renamed TFT_VDD_L
- net TFT_VDD_L: no longer J20.2 (Pin_2)
- new net TFT_BL_R: J20.8 (Pin_8)
- new net TFT_GND_R: J20.1 (Pin_1)
- new net TFT_VDD_R: J20.2 (Pin_2)
Changed lines of the file:
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@@
+	(wire
+		(pts
+			(xy 43.18 81.28) (xy 48.26 81.28)
+		)
+		(stroke
+			(width 0)
+			(type default)
+		)
+	)
 	(wire
 		(pts
@@
 	(wire
 		(pts
+			(xy 43.18 76.2) (xy 48.26 76.2)
+		)
+		(stroke
+			(width 0)
+			(type default)
+		)
+	)
+	(wire
+		(pts
 			(xy 24.13 156.21) (xy 24.13 160.02)
 		)
@@
 	(wire
 		(pts
+			(xy 43.18 86.36) (xy 48.26 86.36)
+		)
+		(stroke
+			(width 0)
+			(type default)
+		)
+	)
+	(wire
+		(pts
 			(xy 49.53 163.83) (xy 49.53 165.1)
 		)
@@
 	(wire
 		(pts
+			(xy 43.18 78.74) (xy 48.26 78.74)
+		)
+		(stroke
+			(width 0)
+			(type default)
+		)
+	)
+	(wire
+		(pts
 			(xy 26.67 45.72) (xy 26.67 49.53)
 		)
@@
 		(pts
 			(xy 93.98 78.74) (xy 104.14 78.74)
+		)
+		(stroke
+			(width 0)
+			(type default)
+		)
+	)
+	(wire
+		(pts
+			(xy 43.18 83.82) (xy 48.26 83.82)
 		)
 		(stroke
@@
 		)
 	)
-	(label "TFT_CS"
+	(label "TFT_SDA_L"
+		(at 43.18 78.74 180)
+		(effects
+			(font
+				(size 1.27 1.27)
+			)
+			(justify right bottom)
+		)
+	)
+	(label "TFT_CS_L"
 		(at -21.59 90.17 180)
 		(effects
@@
 		)
 	)
+	(label "TFT_SCL_L"
+		(at 43.18 76.2 180)
+		(effects
+			(font
+				(size 1.27 1.27)
+			)
+			(justify right bottom)
+		)
+	)
+	(label "TFT_SCL_R"
+		(at 104.14 83.82 0)
+		(effects
+			(font
+				(size 1.27 1.27)
+			)
+			(justify left bottom)
+		)
+	)
 	(label "AUDIO_L"
 		(at 21.59 160.02 270)
@@
 		)
 	)
+	(label "TFT_DC_R"
+		(at 104.14 78.74 0)
+		(effects
+			(font
+				(size 1.27 1.27)
+			)
+			(justify left bottom)
+		)
+	)
 	(label "AUDIO_L"
 		(at 35.56 165.1 180)
@@
 	)
 	(label "UART_TX"
-		(at 104.14 76.2 0)
+		(at 116.84 54.61 0)
 		(effects
 			(font
@@
 		)
 	)
-	(label "TFT_RES"
+	(label "TFT_RES_L"
 		(at -21.59 85.09 180)
 		(effects
@@
 		)
 	)
-	(label "TFT_GND"
+	(label "TFT_DC_L"
+		(at 43.18 83.82 180)
+		(effects
+			(font
+				(size 1.27 1.27)
+			)
+			(justify right bottom)
+		)
+	)
+	(label "TFT_GND_R"
 		(at -15.24 120.65 0)
 		(effects
@@
 	)
 	(label "UART_RX"
-		(at 104.14 73.66 0)
+		(at 116.84 52.07 0)
 		(effects
 			(font
@@
 		)
 	)
-	(label "TFT_BL"
+	(label "TFT_BL_R"
 		(at -15.24 102.87 0)
 		(effects
@@
 		)
 	)
-	(label "TFT_GND"
+	(label "TFT_SDA_R"
+		(at 104.14 86.36 0)
+		(effects
+			(font
+				(size 1.27 1.27)
+			)
+			(justify left bottom)
+		)
+	)
+	(label "TFT_GND_L"
 		(at -21.59 74.93 180)
 		(effects
@@
 		)
 	)
-	(label "TFT_SDA"
+	(label "TFT_SDA_L"
 		(at -21.59 82.55 180)
 		(effects
@@
 		)
 	)
+	(label "TFT_CS_R"
+		(at 104.14 76.2 0)
+		(effects
+			(font
+				(size 1.27 1.27)
+			)
+			(justify left bottom)
+		)
+	)
 	(label "5v_local"
 		(at 41.91 49.53 0)
@@
 		)
 	)
-	(label "TFT_DC"
+	(label "TFT_DC_L"
 		(at -21.59 87.63 180)
 		(effects
@@
 		)
 	)
-	(label "TFT_CS"
+	(label "TFT_CS_R"
 		(at -15.24 105.41 0)
 		(effects
@@
 		)
 	)
-	(label "TFT_SCL"
+	(label "TFT_RES_R"
+		(at 104.14 81.28 0)
+		(effects
+			(font
+				(size 1.27 1.27)
+			)
+			(justify left bottom)
+		)
+	)
+	(label "TFT_SCL_R"
 		(at -15.24 115.57 0)
 		(effects
@@
 			)
 			(justify left bottom)
+		)
+	)
+	(label "TFT_CS_L"
+		(at 43.18 86.36 180)
+		(effects
+			(font
+				(size 1.27 1.27)
+			)
+			(justify right bottom)
 		)
 	)
@@
 		)
 	)
-	(label "TFT_DC"
+	(label "TFT_DC_R"
 		(at -15.24 107.95 0)
 		(effects
@@
 			)
 			(justify left bottom)
+		)
+	)
+	(label "TFT_RES_L"
+		(at 43.18 81.28 180)
+		(effects
+			(font
+				(size 1.27 1.27)
+			)
+			(justify right bottom)
 		)
 	)
@@
 		)
 	)
-	(label "TFT_BL"
+	(label "TFT_BL_L"
 		(at -21.59 92.71 180)
 		(effects
@@
 		)
 	)
-	(label "TFT_VDD"
+	(label "TFT_VDD_R"
 		(at -15.24 118.11 0)
 		(effects
@@
 		)
 	)
-	(label "TFT_SCL"
+	(label "TFT_SCL_L"
 		(at -21.59 80.01 180)
 		(effects
@@
 		)
 	)
-	(label "TFT_RES"
+	(label "TFT_RES_R"
 		(at -15.24 110.49 0)
 		(effects
@@
 		)
 	)
-	(label "TFT_VDD"
+	(label "TFT_VDD_L"
 		(at -21.59 77.47 180)
 		(effects
@@
 		)
 	)
-	(label "TFT_SDA"
+	(label "TFT_SDA_R"
 		(at -15.24 113.03 0)
 		(effects
@@
 		(dnp no)
 		(fields_autoplaced yes)
-		(property "Reference" "#PWR051"
+		(property "Reference" "#PWR050"
 			(at 71.12 138.43 0)
 			(hide yes)
@@
 			(project "ldr_volume"
 				(path "/c16a8161-991e-4f32-8346-3bac9962e2d7"
-					(reference "#PWR051")
+					(reference "#PWR050")
 					(unit 1)
 				)
@@
 		(dnp no)
 		(fields_autoplaced yes)
-		(property "Reference" "J20"
+		(property "Reference" "J19"
 			(at -10.16 82.5499 0)
 			(show_name no)
@@
 			(project "ldr_volume"
 				(path "/c16a8161-991e-4f32-8346-3bac9962e2d7"
-					(reference "J20")
+					(reference "J19")
 					(unit 1)
 				)
@@
 		(dnp no)
 		(fields_autoplaced yes)
-		(property "Reference" "J24"
+		(property "Reference" "J21"
 			(at 67.31 149.2249 90)
 			(show_name no)
@@
 			(project "ldr_volume"
 				(path "/c16a8161-991e-4f32-8346-3bac9962e2d7"
-					(reference "J24")
+					(reference "J21")
 					(unit 1)
 				)
@@
 		(dnp no)
 		(fields_autoplaced yes)
-		(property "Reference" "J23"
+		(property "Reference" "J20"
 			(at -26.67 113.0301 0)
 			(show_name no)
@@
 			(project "ldr_volume"
 				(path "/c16a8161-991e-4f32-8346-3bac9962e2d7"
-					(reference "J23")
+					(reference "J20")
 					(unit 1)
 				)
@@
 		(dnp no)
 		(fields_autoplaced yes)
-		(property "Reference" "J25"
+		(property "Reference" "J22"
 			(at 25.4 150.4949 90)
 			(show_name no)
@@
 			(project "ldr_volume"
 				(path "/c16a8161-991e-4f32-8346-3bac9962e2d7"
-					(reference "J25")
+					(reference "J22")
 					(unit 1)
 				)
@@
 			)
 		)
-		(property "Footprint" "Capacitor_THT:C_Rect_L7.2mm_W2.5mm_P5.00mm_FKS2_FKP2_MKS2_MKP2"
+		(property "Footprint" "Capacitor_THT:C_Disc_D5.0mm_W2.5mm_P5.00mm"
 			(at 33.9852 59.69 0)
 			(hide yes)
@@
 		(dnp no)
 		(fields_autoplaced yes)
-		(property "Reference" "#PWR048"
+		(property "Reference" "#PWR049"
 			(at 30.48 71.12 0)
 			(hide yes)
@@
 			(project "ldr_volume"
 				(path "/c16a8161-991e-4f32-8346-3bac9962e2d7"
-					(reference "#PWR048")
+					(reference "#PWR049")
 					(unit 1)
 				)
@@
 		(dnp no)
 		(fields_autoplaced yes)
-		(property "Reference" "#PWR049"
+		(property "Reference" "#PWR048"
 			(at 138.43 36.83 0)
 			(hide yes)
@@
 			(project "ldr_volume"
 				(path "/c16a8161-991e-4f32-8346-3bac9962e2d7"
-					(reference "#PWR049")
+					(reference "#PWR048")
 					(unit 1)
 				)

Commit message: updates
Parts:
- added C32: 1uF, Capacitor_THT:C_Rect_L7.2mm_W2.5mm_P5.00mm_FKS2_FKP2_MKS2_MKP2, symbol Device:C
- added R35: 1K, Resistor_THT:R_Axial_DIN0207_L6.3mm_D2.5mm_P7.62mm_Horizontal, symbol Device:R
- added R36: 10K, Resistor_THT:R_Axial_DIN0207_L6.3mm_D2.5mm_P7.62mm_Horizontal, symbol Device:R
- J21: value TFT_PWR -> S_AIN_R
- J22: value TFT_PWR -> S_AIN_L
- R25, R26, R27, R28: value 4k -> 10K
Connections:
- net 3.3V_PICO: now also R36.1
- net ADC_R: now also R35.2; no longer C20.2, R25.2, R27.1
- net GNDD: now also C32.1
- net TFT_RES_R: now also C32.2, R36.2
- new net: C20.2, R25.2, R27.1, R35.1
Other:
- moved on the sheet: C20, C21, J21, J22, NT5, NT6, R25, R26, R27, R28

Commit message: update
Parts:
- removed C20, C21: 2.2uF, Capacitor_THT:C_Rect_L7.2mm_W2.5mm_P5.00mm_FKS2_FKP2_MKS2_MKP2, symbol Device:C
- removed C32: 1uF, Capacitor_THT:C_Rect_L7.2mm_W2.5mm_P5.00mm_FKS2_FKP2_MKS2_MKP2, symbol Device:C
- removed J21: S_AIN_R, Connector_JST:JST_XH_B2B-XH-A_1x02_P2.50mm_Vertical, symbol Connector:Conn_01x02_Pin
- removed J22: S_AIN_L, Connector_JST:JST_XH_B2B-XH-A_1x02_P2.50mm_Vertical, symbol Connector:Conn_01x02_Pin
- removed NT5, NT6: NetTie_2, nettie 1.0:NetTie-2_SMD_Pad1.0o, symbol Device:NetTie_2
- removed R25, R26, R27, R28, R36: 10K, Resistor_THT:R_Axial_DIN0207_L6.3mm_D2.5mm_P7.62mm_Horizontal, symbol Device:R
- removed R35: 1K, Resistor_THT:R_Axial_DIN0207_L6.3mm_D2.5mm_P7.62mm_Horizontal, symbol Device:R
- renumbered J19 to J21, J20 to J22

Commit message: updates
Parts:
- removed C17: 100uF low, Capacitor_THT:CP_Radial_D6.3mm_P2.50mm, symbol Device:C_Polarized
- removed C19: 100nF, Capacitor_THT:C_Disc_D5.0mm_W2.5mm_P5.00mm, symbol Device:C
- removed D3: 1n5819, Diode_THT:D_DO-41_SOD81_P7.62mm_Horizontal, symbol Device:D
- removed J16: 5v_in_b3, Connector_JST:JST_XH_B2B-XH-A_1x02_P2.50mm_Vertical, symbol Connector:Conn_01x02_Pin
- removed J17: Conn_01x03_Pin, Connector_JST:JST_XH_B3B-XH-A_1x03_P2.50mm_Vertical, symbol Connector:Conn_01x03_Pin
- removed J21: LEFT_TFT, Connector_PinHeader_2.54mm:PinHeader_1x08_P2.54mm_Vertical, symbol Connector:Conn_01x08_Socket
- removed J22: RIGHT_TFT, Connector_PinHeader_2.54mm:PinHeader_1x08_P2.54mm_Vertical, symbol Connector:Conn_01x08_Socket
- added C13: 100uF low, Capacitor_THT:CP_Radial_D6.3mm_P2.50mm, symbol Device:C_Polarized
- added C21, C27, C31, C32, C33: 100nF, Capacitor_THT:C_Disc_D5.0mm_W2.5mm_P5.00mm, symbol Device:C
- added C28, C29: 2.2uF, Capacitor_THT:C_Rect_L7.2mm_W2.5mm_P5.00mm_FKS2_FKP2_MKS2_MKP2, symbol Device:C
- added C30: 4.7uF, Capacitor_THT:CP_Radial_D6.3mm_P2.50mm, symbol Device:C_Polarized
- added D2: 1n5819, Diode_THT:D_DO-41_SOD81_P7.62mm_Horizontal, symbol Device:D
- added J14: Conn_02x04_Counter_Clockwise, Connector_PinHeader_2.54mm:PinHeader_2x04_P2.54mm_Vertical, symbol Connector_Generic:Conn_02x04_Counter_Clockwise
- added J15: PWR_IN, Connector_JST:JST_XH_B2B-XH-A_1x02_P2.50mm_Vertical, symbol Connector:Conn_01x02_Pin
- added J24: UART, Connector_JST:JST_XH_B3B-XH-A_1x03_P2.50mm_Vertical, symbol Connector:Conn_01x03_Pin
- added J29: TFT, Connector_PinHeader_2.54mm:PinHeader_1x08_P2.54mm_Horizontal, symbol Connector:Conn_01x08_Pin
- added J30, J33: IR, Connector_JST:JST_XH_B3B-XH-A_1x03_P2.50mm_Vertical, symbol Connector:Conn_01x03_Pin
- added J31: S_AIN_L, Connector_JST:JST_XH_B2B-XH-A_1x02_P2.50mm_Vertical, symbol Connector:Conn_01x02_Pin
- added J32: S_AIN_R, Connector_JST:JST_XH_B2B-XH-A_1x02_P2.50mm_Vertical, symbol Connector:Conn_01x02_Pin
- added J34: SDA, Connector_JST:JST_XH_B4B-XH-A_1x04_P2.50mm_Vertical, symbol Connector:Conn_01x04_Pin
- added J35: BTN_VOL, Connector_PinHeader_2.54mm:PinHeader_1x03_P2.54mm_Horizontal, symbol Connector:Conn_01x03_Pin
- added J38: BTN_MENU, Connector_PinHeader_2.54mm:PinHeader_1x03_P2.54mm_Horizontal, symbol Connector:Conn_01x03_Pin
- added J40: BTN_EXT1, Connector_PinHeader_2.54mm:PinHeader_1x03_P2.54mm_Horizontal, symbol Connector:Conn_01x03_Pin
- added J41: BTN_EXT2, Connector_PinHeader_2.54mm:PinHeader_1x03_P2.54mm_Horizontal, symbol Connector:Conn_01x03_Pin
- added NT7, NT8: NetTie_2, nettie 1.0:NetTie-2_SMD_Pad1.0o, symbol Device:NetTie_2
- added R21, R35, R36, R37, R38: 10K, Resistor_THT:R_Axial_DIN0207_L6.3mm_D2.5mm_P2.54mm_Vertical, symbol Device:R
- added R39, R40: 4.7K, Resistor_THT:R_Axial_DIN0207_L6.3mm_D2.5mm_P7.62mm_Horizontal, symbol Device:R
- added R41, R42, R43, R44: 1k, Resistor_THT:R_Axial_DIN0207_L6.3mm_D2.5mm_P7.62mm_Horizontal, symbol Device:R
- added SW1, SW2, SW3, SW4: SW_Push, Button_Switch_THT:SW_SPST_Omron_B3F-50xx, symbol Switch:SW_Push
- added U6: TSOP312xx, OptoDevice:Vishay_CAST-3Pin, symbol Interface_Optical:TSOP312xx
Connections:
- net 3.3V_PICO: now also J14.1 (Pin_1), J14.2 (Pin_2), J29.1 (Pin_1), J30.2 (Pin_2), J33.2 (Pin_2), J34.4 (Pin_4), R21.1, R35.1, R38.2, R39.1, R40.1
- net 5V_board1: now also C13.1, C21.1, D2.2 (A), J15.2 (Pin_2)
- net ADC_L: now also A2.34 (GPIO28_ADC2), C28.2, R21.2, R36.1; no longer A2.31 (GPIO26_ADC0)
- net ADC_R: now also C29.2, R35.2, R37.1
- net AGND_PICO: now also NT7.2, NT8.2
- net GNDD: now also C13.2, C21.2, C27.2, C30.2, C31.2, C32.2, C33.2, J14.3 (Pin_3), J14.4 (Pin_4), J14.8 (Pin_8), J15.1 (Pin_1), J24.1 (Pin_1), J29.4 (Pin_4), J30.3 (Pin_3), J33.3 (Pin_3), J34.1 (Pin_1), J35.2 (Pin_2), J38.2 (Pin_2), J40.2 (Pin_2), J41.2 (Pin_2), SW1.2, SW2.2, SW3.2, SW4.2, U6.1 (GND)
- net UART_RX: now also A2.17 (GPIO13), J24.2 (Pin_2)
- net UART_TX: now also A2.16 (GPIO12), J24.3 (Pin_3)
- net BTN_UP: now reaches A2.1 (GPIO0)
- net BTN_UP: now also J38.3 (Pin_3), J40.1 (Pin_1), R41.1
- net TFT_RST: now reaches A2.10 (GPIO7)
- net TFT_RST: now also J29.2 (Pin_2)
- net PWR_CTRL: now reaches A2.12 (GPIO9)
- net PWR_CTRL: now also J14.6 (Pin_6)
- net EXT_1: now reaches A2.14 (GPIO10)
- net EXT_1: now also J14.7 (Pin_7)
- net EXT_2: now reaches A2.15 (GPIO11)
- net EXT_2: now also J14.5 (Pin_5)
- net BTN_DN: now reaches A2.19 (GPIO14)
- net BTN_DN: now also J35.3 (Pin_3), J41.3 (Pin_3), R42.1
- net BTN_RT: now reaches A2.2 (GPIO1)
- net BTN_RT: now also J38.1 (Pin_1), J40.3 (Pin_3), R44.1
- net BTN_LT: now reaches A2.20 (GPIO15)
- net BTN_LT: now also J35.1 (Pin_1), J41.1 (Pin_1), R43.1
- net SDA: now reaches A2.21 (GPIO16)
- net SDA: now also J34.3 (Pin_3), R39.2
- net at A2.39 (VSYS): now also D2.1 (K)
- net TFT_CS_L renamed TFT_DC
- net TFT_DC: now also J29.3 (Pin_3)
- net TFT_CS_R renamed SCL
- net SCL: now also J34.2 (Pin_2), R40.2
- net TFT_DC_L renamed TFT_CS
- net TFT_CS: now also J29.5 (Pin_5)
- net TFT_DC_R renamed IR
- net IR: now also J30.1 (Pin_1), J33.1 (Pin_1), U6.3 (OUT)
- net TFT_RES_L renamed TFT_BLK
- net TFT_BLK: now also J29.6 (Pin_6)
- net TFT_RES_R: no longer names the net of A2.25 (GPIO19)
- net TFT_SCL_L renamed TFT_SCL
- net TFT_SCL: now also J29.8 (Pin_8)
- net TFT_SCL_R: no longer names the net of A2.26 (GPIO20)
- net TFT_SDA_L renamed TFT_SDA
- net TFT_SDA: now also J29.7 (Pin_7)
- net TFT_SDA_R: no longer names the net of A2.27 (GPIO21)
- new net: C32.1, R43.2, SW3.1
- new net: C30.1, R38.1, U6.2 (Vs)
- new net: C31.1, R42.2, SW2.1
- new net: C33.1, R44.2, SW4.1
- new net: C27.1, R41.2, SW1.1
- new net AGND_L: J31.1 (Pin_1), NT8.1, R36.2
- new net AGND_R: J32.2 (Pin_2), NT7.1, R37.2
- new net AUDIO_L: C28.1, J31.2 (Pin_2)
- new net AUDIO_R: C29.1, J32.1 (Pin_1)
Other:
- note added: "Twisted wire 1 pair + shield LiYCY 1x2x0.5mm2 For main board interconnect +5V and GND , shield connects to board#1 only"

Commit message: updates
Parts:
- removed C30: 4.7uF, Capacitor_THT:CP_Radial_D6.3mm_P2.50mm, symbol Device:C_Polarized
- added C34: 100nF, Capacitor_THT:C_Disc_D5.0mm_W2.5mm_P5.00mm, symbol Device:C
- added C35, C36: 10nF, Capacitor_THT:C_Disc_D5.0mm_W2.5mm_P5.00mm, symbol Device:C
- added J22: PWR_SEL, Connector_PinHeader_2.54mm:PinHeader_1x03_P2.54mm_Vertical, symbol Connector:Conn_01x03_Pin
- added J36: IR, Connector_JST:JST_XH_B3B-XH-A_1x03_P2.50mm_Vertical, symbol Connector:Conn_01x03_Pin
- D2: value 1n5819 -> 1n5817; footprint Diode_THT:D_DO-41_SOD81_P7.62mm_Horizontal -> Diode_THT:D_DO-41_SOD81_P3.81mm_Vertical_CathodeUp
- J34: value SDA -> I2C/ALPS
- R38: value 10K -> 100
Connections:
- net 3.3V_PICO: now also J30.3 (Pin_3), J22.1 (Pin_1), J36.3 (Pin_3); no longer J30.2 (Pin_2), J34.4 (Pin_4)
- net 5V_board1: no longer C13.1, C21.1
- net ADC_L: now also C36.1
- net ADC_R: now also C35.2
- net AGND_L: no longer R36.2
- net AGND_PICO: now also A2.31 (GPIO26_ADC0), R36.2, R37.2, C35.1, C36.2
- net AGND_R: no longer R37.2
- net GNDD: now also J30.2 (Pin_2), J34.3 (Pin_3), C34.2, J36.2 (Pin_2); no longer J30.3 (Pin_3), J34.1 (Pin_1)
- net SCL: now also J34.1 (Pin_1); no longer J34.2 (Pin_2)
- net SDA: now also J34.2 (Pin_2); no longer J34.3 (Pin_3)
- net TFT_BLK: now also A2.10 (GPIO7), J29.2 (Pin_2); no longer A2.6 (GPIO4), J29.6 (Pin_6)
- net TFT_DC: now also A2.6 (GPIO4), J29.6 (Pin_6); no longer A2.9 (GPIO6), J29.3 (Pin_3)
- net TFT_RST: now also A2.9 (GPIO6), J29.3 (Pin_3); no longer A2.10 (GPIO7), J29.2 (Pin_2)
- net at R38.1, U6.2 (Vs): now also C34.1
- net MUTE_CTRL: now reaches A2.26 (GPIO20)
- net MUTE_CTRL: now also J36.1 (Pin_1)
- net 5v_local: now reaches A2.39 (VSYS), D2.1 (K)
- net 5v_local: now also C13.1, C21.1, J22.3 (Pin_3)
- new net PWR_SEL: J22.2 (Pin_2), J34.4 (Pin_4)
Other:
- moved on the sheet: D2

Commit message: updates
Parts:
- removed J14: Conn_02x04_Counter_Clockwise, Connector_PinHeader_2.54mm:PinHeader_2x04_P2.54mm_Vertical, symbol Connector_Generic:Conn_02x04_Counter_Clockwise
- removed J29: TFT, Connector_PinHeader_2.54mm:PinHeader_1x08_P2.54mm_Horizontal, symbol Connector:Conn_01x08_Pin
- removed J30: IR, Connector_JST:JST_XH_B3B-XH-A_1x03_P2.50mm_Vertical, symbol Connector:Conn_01x03_Pin
- added C37: 100nF, Capacitor_THT:C_Disc_D5.0mm_W2.5mm_P5.00mm, symbol Device:C
- added D6: WHITE LED, LED_THT:LED_D3.0mm_Horizontal_O1.27mm_Z2.0mm, symbol Device:LED
- added D7: LED, LED_THT:LED_D3.0mm_Horizontal_O1.27mm_Z2.0mm, symbol Device:LED
- added J29: IR, Connector_PinHeader_2.54mm:PinHeader_1x03_P2.54mm_Vertical, symbol Connector:Conn_01x03_Pin
- added J30: TFT, Connector_PinHeader_2.54mm:PinHeader_1x09_P2.54mm_Horizontal, symbol Connector:Conn_01x09_Pin
- added J42: PWR_BTN, Connector_PinHeader_2.54mm:PinHeader_1x02_P2.54mm_Vertical, symbol Connector:Conn_01x02_Pin
- added J43: PWR_BTN_LED, Connector_PinHeader_2.54mm:PinHeader_1x02_P2.54mm_Vertical, symbol Connector:Conn_01x02_Pin
- added J44: ALPS, Connector_PinHeader_2.54mm:PinHeader_1x04_P2.54mm_Vertical, symbol Connector:Conn_01x04_Pin
- added J45: PWR_RELAY, Connector_PinHeader_2.54mm:PinHeader_1x03_P2.54mm_Vertical, symbol Connector:Conn_01x03_Pin
- added Q13: BC547, Package_TO_SOT_THT:TO-92_Inline_Wide, symbol Transistor_BJT:BC547
- added R45, R50: 1k, Resistor_THT:R_Axial_DIN0207_L6.3mm_D2.5mm_P7.62mm_Horizontal, symbol Device:R
- added R46, R47: 100, Resistor_THT:R_Axial_DIN0207_L6.3mm_D2.5mm_P2.54mm_Vertical, symbol Device:R
- added R48, R49: 22, Resistor_THT:R_Axial_DIN0207_L6.3mm_D2.5mm_P2.54mm_Vertical, symbol Device:R
- added SW5: SW_PWR, Button_Switch_THT:SW_SPST_Omron_B3F-50xx, symbol Switch:SW_Push
- J33: value IR -> IR_SENSOR
- J34: value I2C/ALPS -> I2C; footprint Connector_JST:JST_XH_B4B-XH-A_1x04_P2.50mm_Vertical -> Connector_PinHeader_2.54mm:PinHeader_1x04_P2.54mm_Vertical
- J36: value IR -> MUTE; footprint Connector_JST:JST_XH_B3B-XH-A_1x03_P2.50mm_Vertical -> Connector_PinHeader_2.54mm:PinHeader_1x03_P2.54mm_Vertical
- SW1: value SW_Push -> SW_UP
- SW2: value SW_Push -> SW_DN
- SW3: value SW_Push -> SW_LT
- SW4: value SW_Push -> SW_RT
Connections:
- net EXT_2 is gone; now on net MUTE_CTRL: A2.15 (GPIO11)
- net 3.3V_PICO: now also J34.4 (Pin_4), J29.3 (Pin_3)
- net 5v_local: now also J30.9 (Pin_9), J44.1 (Pin_1), J45.1 (Pin_1), R46.2, R47.2
- net BTN_DN: now also A2.17 (GPIO13), J35.2 (Pin_2); no longer A2.19 (GPIO14), J35.3 (Pin_3)
- net BTN_LT: now also A2.16 (GPIO12), J35.3 (Pin_3); no longer A2.20 (GPIO15), J35.1 (Pin_1)
- net BTN_RT: now also A2.5 (GPIO3); no longer A2.2 (GPIO1)
- net BTN_UP: now also A2.4 (GPIO2), J38.2 (Pin_2); no longer A2.1 (GPIO0), J38.3 (Pin_3)
- net GNDD: now also J34.1 (Pin_1), J35.1 (Pin_1), J38.3 (Pin_3), C37.2, J29.2 (Pin_2), J30.1 (Pin_1), J30.6 (Pin_6), J42.1 (Pin_1), J43.1 (Pin_1), J44.2 (Pin_2), J45.2 (Pin_2), Q13.3 (E), SW5.2; no longer J34.3 (Pin_3), J35.2 (Pin_2), J38.2 (Pin_2)
- net IR: now also A2.11 (GPIO8), J29.1 (Pin_1); no longer A2.24 (GPIO18)
- net MUTE_CTRL: no longer A2.26 (GPIO20)
- net PWR_SEL: no longer J34.4 (Pin_4)
- net SCL: now also A2.20 (GPIO15), J34.3 (Pin_3); no longer A2.22 (GPIO17), J34.1 (Pin_1)
- net SDA: now also A2.19 (GPIO14); no longer A2.21 (GPIO16)
- net TFT_BLK: now also A2.27 (GPIO21), J30.2 (Pin_2); no longer A2.10 (GPIO7)
- net TFT_CS: now also A2.22 (GPIO17), J30.7 (Pin_7); no longer A2.7 (GPIO5)
- net TFT_DC: now also A2.21 (GPIO16), J30.8 (Pin_8); no longer A2.6 (GPIO4)
- net TFT_RST: now also A2.26 (GPIO20), J30.3 (Pin_3); no longer A2.9 (GPIO6)
- net TFT_SCL: now also J30.5 (Pin_5), R48.1; no longer A2.4 (GPIO2)
- net TFT_SDA: now also J30.4 (Pin_4), R49.1; no longer A2.5 (GPIO3)
- net UART_RX: now also A2.2 (GPIO1); no longer A2.17 (GPIO13)
- net UART_TX: now also A2.1 (GPIO0); no longer A2.16 (GPIO12)
- net at A2.25 (GPIO19): now also R49.2
- net EXT_1 renamed PWR_BTN
- net PWR_BTN: now also J42.2 (Pin_2), R45.1
- net PWR_CTRL renamed PWR_BTN_LED
- net PWR_BTN_LED: now also J43.2 (Pin_2)
- new net: D6.1 (K), D7.1 (K), Q13.1 (C)
- new net: D7.2 (A), R46.1
- new net: D6.2 (A), R47.1
- new net: Q13.2 (B), R50.2
- new net: C37.1, R45.2, SW5.1
- new net: A2.24 (GPIO18), R48.2
- new net ALPS_L: A2.10 (GPIO7), J44.3 (Pin_3)
- new net ALPS_R: A2.9 (GPIO6), J44.4 (Pin_4)
- new net LED_CTRL: R50.1
- new net RLCTRL: A2.7 (GPIO5), J45.3 (Pin_3)
- no-connect marks 0 -> 6
Other:
- note added: "Push button 5v or 3v led direct gpio drive"
- moved on the sheet: C27, C31, C32, C33, C34, C35, C36, J22, J33, J35, J38, J40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
