File: amp_v3/ldr_volume/ldrctrl_v1b.kicad_pcb (KiCad board)
At the start: 2 copper layers, 92.7 x 62.9 mm, 56 parts, among them J18 UART, J19 MUTE, J20 CTRL, J21 CTRL, J22 PWR_IN, J23 I2C_L, J24 I2C_R, Q1 BC557, Q10 2N7000, Q2 BC557, Q3 BC547, Q4 BC547, Q5 BC557, Q6 BC557, Q7 BC547, Q8 BC547, Q9 2N7000, U7 TL431LP

Commit message: updates
Parts:
- removed J20, J21: CTRL, Connector_JST:JST_XH_B6B-XH-A_1x06_P2.50mm_Vertical
- added J16: MUTE_OUT, Connector_JST:JST_XH_B2B-XH-A_1x02_P2.50mm_Vertical, F.Cu at (291.7, 174.7)
- added J17: MUTE, Connector_JST:JST_XH_B2B-XH-A_1x02_P2.50mm_Vertical, F.Cu at (285.0, 152.9)
- added J25: LDR_R, Connector_JST:JST_XH_B5B-XH-A_1x05_P2.50mm_Vertical, F.Cu at (210.7, 123.0)
- added J37: LDR_L, Connector_JST:JST_XH_B5B-XH-A_1x05_P2.50mm_Vertical, F.Cu at (210.7, 97.0)
- added Q11: BC547, Package_TO_SOT_THT:TO-92_Inline_Wide, F.Cu at (287.6, 174.7)
- added R26: 100, Resistor_THT:R_Axial_DIN0207_L6.3mm_D2.5mm_P7.62mm_Horizontal, F.Cu at (293.2, 158.2)
- added R27: 1K, Resistor_THT:R_Axial_DIN0207_L6.3mm_D2.5mm_P7.62mm_Horizontal, F.Cu at (285.0, 170.1)
- added R53: 4.7K, Resistor_THT:R_Axial_DIN0207_L6.3mm_D2.5mm_P2.54mm_Vertical, F.Cu at (279.2, 111.2)
- added U5: 4N25, Package_DIP:DIP-6_W7.62mm, F.Cu at (289.2, 158.2)
- added U8: DS18B20, Connector_JST:JST_XH_B3B-XH-A_1x03_P2.50mm_Vertical, F.Cu at (285.8, 119.3)
- C34, C35: footprint Capacitor_THT:C_Disc_D5.0mm_W2.5mm_P5.00mm -> Capacitor_THT:C_Rect_L7.2mm_W2.5mm_P5.00mm_FKS2_FKP2_MKS2_MKP2
- moved R32 269.1 mm to (269.0, 121.4), turned to -90 degrees
- moved J19 268.2 mm to (279.7, 116.8)
- moved J18 266.4 mm to (283.7, 126.5)
- moved C35 265.7 mm to (277.7, 103.6)
- moved J22 264.9 mm to (285.8, 86.8)
- moved R30 264.6 mm to (267.5, 112.5)
- moved D2 264.4 mm to (281.2, 79.2)
- moved R31 264.4 mm to (267.5, 115.5)
- moved R52 263.9 mm to (270.3, 102.8)
- moved TH1 263.9 mm to (284.0, 101.1)
- moved A1 263.9 mm to (255.7, 80.8)
- moved C16 263.9 mm to (237.4, 100.9)
- moved C17 263.9 mm to (237.2, 127.0)
- moved C18 263.9 mm to (237.4, 88.2)
- moved C19 263.9 mm to (237.4, 114.2)
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Connections:
- A1 pad 27: /LDR Driver/MUTE_CTRL -> /LDR Driver/DQ_IN
- A1 pad 31: /LDR Driver/ADC_TL431REF -> /LDR Driver/ADC_NTC
- A1 pad 32: /LDR Driver/ADC_NTC -> /LDR Driver/AGND_PICO
Routing:
- net /LDR Driver/3.3V_PICO: track 28.3 -> 50.5 mm
- net /LDR Driver/DQ_IN: track 0.00 -> 17.2 mm
- net /LDR Driver/ADC_TL431REF: track 40.6 -> 25.6 mm
- net Net-(Q11-B): track 0.00 -> 9.59 mm
- net /LDR Driver/AMP_MUTE_PIN: track 0.00 -> 9.06 mm
- net /LDR Driver/MUTE_CTRL: track 10.2 -> 18.1 mm
- net /LDR Driver/5v_local: track 132.2 -> 138.8 mm
- net Net-(R26-Pad1): track 0.00 -> 3.94 mm
- net /LDR Driver/SHUNT_R: track 14.2 -> 12.7 mm
- net /LDR Driver/COIL_R: track 38.7 -> 37.3 mm
- net /LDR Driver/UART_TX: track 10.6 -> 9.33 mm
- net /LDR Driver/UART_RX: track 6.38 -> 5.19 mm
- net /LDR Driver/SERIAL_R: track 11.7 -> 10.6 mm
- net /LDR Driver/ADC_NTC: track 13.1 -> 14.1 mm
- net /LDR Driver/SERIAL_L: track 11.3 -> 10.7 mm
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- added copper zone on B.Cu, net /LDR Driver/AMP_GND_PIN
Other:
- board size 92.7 x 62.9 mm -> 95.2 x 114.2 mm
