File: amp_v3/ldr_volume/ldr_volume.kicad_pcb (KiCad board)
At the start: 2 copper layers, 424.2 x 159 mm, 176 parts, among them J1 A_IN, J10 CTRL, J12 EXT, J13 NTC, J14 Conn_01x05_Pin, J15 PWR_IN, J16 CTRL, J17 CTRL, J18 PWR3, J19 PWR_IN, J2 A_OUT, J20 I2C_L, J21 I2C_R, J22 PWR_SEL, J23 MUTE, J24 UART, J25 PWR4, J26 Conn_01x03_Pin, J27 5V_IN, J28 5V_IN, J29 IR, J3 5v_in, J30 TFT, J31 S_AIN_L, J32 S_AIN_R, J33 IR_SENSOR, J34 I2C, J35 BTN_VOL, J36 MUTE, J37 MUTE, J38 BTN_MENU, J39 UART, J4 ADS1115, J40 BTN_EXT1, J41 BTN_EXT2, J42 PWR_BTN, J43 PWR_BTN_LED, J44 PWR_RLY, J45 MUTE_OUT, J46 ALPS, J5 I2C_R, J6 PWR1, J7 PWR2, J8 PWR3, J9 PWR4, K1 G5V-2, Q1 BC547, Q10 BC557, Q11 2N7000, Q12 2N7000, Q13 BC547, Q14 BC547, Q2 BC557, Q3 BC547, Q4 BC557, Q5 BC547, Q6 BC557, Q7 BC547, Q8 BC557, Q9 BC547, SW1 SW_UP, SW2 SW_DN, SW3 SW_LT, SW4 SW_RT, SW5 SW_PWR, U1 MCP1700x-330xxTO, U2 NSL-32-SR3-Rseries, U3 NSL-32-SR3-Rshunt, U4 4N25, U5 NSL-32-SR3, U6 TSOP312xx, U7 IRM-10-5

Commit message: updates
Parts:
- removed J12: EXT, Connector_PinHeader_2.54mm:PinHeader_1x04_P2.54mm_Vertical
- removed J37: MUTE, Connector_JST:JST_XH_B3B-XH-A_1x03_P2.50mm_Vertical
- removed R11: 1M, Resistor_THT:R_Axial_DIN0207_L6.3mm_D2.5mm_P7.62mm_Horizontal
- added J47: MUTE, Connector_JST:JST_XH_B2B-XH-A_1x02_P2.50mm_Vertical, F.Cu at (147.0, -137.8)
- added R52: 10K, Resistor_THT:R_Axial_DIN0207_L6.3mm_D2.5mm_P2.54mm_Vertical, F.Cu at (144.7, -130.2)
- D3: footprint Diode_THT:D_DO-41_SOD81_P10.16mm_Horizontal -> Diode_THT:D_DO-41_SOD81_P3.81mm_Vertical_CathodeUp
- R15: value 200 -> 150
- moved J1 25.5 mm to (46.9, -137.3)
- moved U3 20.2 mm to (48.1, -120.1)
- moved D3 8.13 mm to (146.0, -154.3)
- moved K1 7.41 mm to (40.9, -122.7)
- moved D1 7.13 mm to (40.8, -119.4)
- moved J19 6.96 mm to (145.5, -145.5), turned to 0 degrees
- moved J2 6.87 mm to (27.2, -134.8), turned to 90 degrees
- moved U2 5.75 mm to (29.8, -120.1)
- moved J4 5.34 mm to (36.7, -155.1)
- moved R28 5.33 mm to (52.0, -147.7)
- moved J5 5.28 mm to (55.8, -159.9)
- moved C10 4.84 mm to (59.6, -151.8)
- moved J39 4.59 mm to (147.0, -125.1)
- moved NT2 4.54 mm to (51.2, -132.8)
- moved C19 4.32 mm to (46.7, -151.8), turned to 0 degrees
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Connections:
- net /board#1/5V_IRM renamed /5V power/5V_IRM
- net /board#1/5V_analog renamed /5V power/5V_analog
- net /board#1/5V_board1 renamed /5V power/5V_board1
- net /board#1/GND_IRM renamed /5V power/GND_IRM
- net /board#2/5v_ads renamed /LDR Board/5v_ads
- net /board#2/A0 renamed /LDR Board/A0
- net /board#2/A1 renamed /LDR Board/A1
- net /board#2/A3 renamed /LDR Board/A3
- net /board#2/ADS_VDD renamed /LDR Board/ADS_VDD
- net /board#2/AUDIO_IN renamed /LDR Board/AUDIO_IN
- net /board#2/AUDIO_OUT renamed /LDR Board/AUDIO_OUT
- net /board#2/MIDDLE_JUNCTION renamed /LDR Board/MIDDLE_JUNCTION
- net /board#2/SCL renamed /LDR Board/SCL
- net /board#2/SDA renamed /LDR Board/SDA
- net /board#2/TOP_JUNCTION renamed /LDR Board/TOP_JUNCTION
- net /board#3/3.3V_PICO renamed /LDR Driver/3.3V_PICO
- net /board#3/5V_board1 renamed /LDR Driver/5V_board1
- net /board#3/5v_local renamed /LDR Driver/5v_local
- net /board#3/AMP_GND_PIN renamed /LDR Driver/AMP_GND_PIN
- net /board#3/AMP_MUTE_PIN renamed /LDR Driver/AMP_MUTE_PIN
- net /board#3/COIL_CTRL_L renamed /LDR Driver/COIL_CTRL_L
- net /board#3/COIL_CTRL_R renamed /LDR Driver/COIL_CTRL_R
- net /board#3/COIL_L renamed /LDR Driver/COIL_L
- net /board#3/COIL_R renamed /LDR Driver/COIL_R
- net /board#3/PWM_SER_L renamed /LDR Driver/PWM_SER_L
- net /board#3/PWM_SER_R renamed /LDR Driver/PWM_SER_R
- net /board#3/PWM_SHUNT_L renamed /LDR Driver/PWM_SHUNT_L
- net /board#3/PWM_SHUNT_R renamed /LDR Driver/PWM_SHUNT_R
- net /board#3/SCL_L renamed /LDR Driver/SCL_L
- net /board#3/SCL_R renamed /LDR Driver/SCL_R
- net /board#3/SDA_L renamed /LDR Driver/SDA_L
- net /board#3/SDA_R renamed /LDR Driver/SDA_R
- net /board#3/SERIAL_L renamed /LDR Driver/SERIAL_L
- net /board#3/SERIAL_R renamed /LDR Driver/SERIAL_R
- net /board#3/SHUNT_L renamed /LDR Driver/SHUNT_L
- net /board#3/SHUNT_R renamed /LDR Driver/SHUNT_R
- net /board#5/3.3V_PICO renamed /Main Board/3.3V_PICO
- net /board#5/5V_board1 renamed /Main Board/5V_board1
- net /board#5/5v_local renamed /Main Board/5v_local
- net /board#5/ADC_L renamed /Main Board/ADC_L
- net /board#5/ADC_R renamed /Main Board/ADC_R
- net /board#5/AGND_L renamed /Main Board/AGND_L
- net /board#5/AGND_PICO renamed /Main Board/AGND_PICO
- net /board#5/AGND_R renamed /Main Board/AGND_R
- net /board#5/ALPS_L renamed /Main Board/ALPS_L
- net /board#5/ALPS_R renamed /Main Board/ALPS_R
- net /board#5/AUDIO_L renamed /Main Board/AUDIO_L
- net /board#5/AUDIO_R renamed /Main Board/AUDIO_R
- net /board#5/BTN_DN renamed /Main Board/BTN_DN
- net /board#5/BTN_LT renamed /Main Board/BTN_LT
- net /board#5/BTN_RT renamed /Main Board/BTN_RT
- net /board#5/BTN_UP renamed /Main Board/BTN_UP
- net /board#5/IR renamed /Main Board/IR
- net /board#5/LED_CTRL renamed /Main Board/LED_CTRL
- net /board#5/MUTE_CTRL renamed /Main Board/MUTE_CTRL
- net /board#5/PWR_BTN renamed /Main Board/PWR_BTN
- net /board#5/PWR_BTN_LED renamed /Main Board/PWR_BTN_LED
- net /board#5/PWR_SEL renamed /Main Board/PWR_SEL
- net /board#5/RLCTRL renamed /Main Board/RLCTRL
- net /board#5/SCL renamed /Main Board/SCL
- net /board#5/SDA renamed /Main Board/SDA
- net /board#5/TFT_BLK renamed /Main Board/TFT_BLK
- net /board#5/TFT_CS renamed /Main Board/TFT_CS
- net /board#5/TFT_DC renamed /Main Board/TFT_DC
- net /board#5/TFT_RST renamed /Main Board/TFT_RST
- net /board#5/TFT_SCL renamed /Main Board/TFT_SCL
- net /board#5/TFT_SDA renamed /Main Board/TFT_SDA
- net /board#5/UART_RX renamed /Main Board/UART_RX
- net /board#5/UART_TX renamed /Main Board/UART_TX
- A1 pad 21: /board#3/UART_RX -> /LDR Driver/UART_TX
- A1 pad 22: /board#3/UART_TX -> /LDR Driver/UART_RX
- D1 pad 1: /board#2/5v_local -> /LDR Board/5v_local
- D1 pad 2: /board#2/COIL_NEG -> /LDR Board/COIL_NEG
- J10 pad 1: /board#2/SHUNT_POS -> /LDR Board/SERIAL_POS
- J10 pad 2: GNDD -> /LDR Board/COIL_NEG
- J10 pad 3: /board#2/SERIAL_POS -> GNDD
- J10 pad 4: /board#2/COIL_NEG -> /LDR Board/5v_local
- J10 pad 6: /board#2/5v_local -> /LDR Board/SHUNT_POS
- J23 pad 2: /board#3/MUTE_CTRL -> /LDR Driver/MUTE_CTRL
- J39 pad 2: /board#3/UART_TX -> /LDR Driver/UART_TX
- J39 pad 3: /board#3/UART_RX -> /LDR Driver/UART_RX
- K1 pad 1: /board#2/5v_local -> /LDR Board/5v_local
- K1 pad 16: /board#2/COIL_NEG -> /LDR Board/COIL_NEG
- R15 pad 2: /board#3/MUTE_CTRL -> /LDR Driver/MUTE_CTRL
- U2 pad 1: /board#2/SERIAL_POS -> /LDR Board/SERIAL_POS
- U2 pad 3: Net-(K1-Pad13) -> Net-(K1-Pad4)
- U2 pad 4: Net-(K1-Pad4) -> Net-(K1-Pad13)
- U3 pad 1: /board#2/SHUNT_POS -> /LDR Board/SHUNT_POS
- U3 pad 3: AUDIO_GND -> Net-(K1-Pad13)
- U3 pad 4: Net-(K1-Pad13) -> AUDIO_GND
Routing:
- net /LDR Board/AUDIO_IN: track 26.5 -> 6.83 mm
- net /LDR Driver/MUTE_CTRL: track 0.00 -> 17.4 mm
- net /board#3/MUTE_CTRL: track 13.1 -> 0.00 mm
- net /LDR Driver/3.3V_PICO: track 41.5 -> 28.8 mm
- net /board#2/5v_local: track 11.9 -> 0.00 mm
- net /board#2/COIL_NEG: track 11.5 -> 0.00 mm
- net /LDR Driver/UART_RX: track 0.00 -> 9.55 mm
- net /LDR Driver/UART_TX: track 0.00 -> 9.38 mm
- net /LDR Board/COIL_NEG: track 0.00 -> 9.14 mm
- net /board#3/EXT1: track 7.84 -> 0.00 mm
- net /LDR Board/5v_local: track 0.00 -> 7.77 mm
- net /board#3/EXT2: track 7.21 -> 0.00 mm
- net /LDR Board/MIDDLE_JUNCTION: track 10.7 -> 3.97 mm
- net /board#3/EXT3: track 6.57 -> 0.00 mm
- net Net-(Q5-C): track 9.72 -> 16.2 mm
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Other:
- outline, holes or cut-outs redrawn

Commit message: updates
Routing:
- net /Main Board/5v_local: track 118.0 -> 118.6 mm
Changed lines of the file:
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@@
 	(footprint "Connector_JST:JST_XH_B2B-XH-A_1x02_P2.50mm_Vertical"
 		(layer "F.Cu")
-		(at 76.748028 -74.3744 90)
+		(at 76.748028 -74.3344 90)
 		(descr "JST XH series connector, B2B-XH-A (http://www.jst-mfg.com/product/pdf/eng/eXH.pdf)")
 		(tags "connector JST XH vertical")
@@
 	)
 	(segment
-		(start 72.938028 -79.4144)
-		(end 78.018028 -79.4144)
-		(width 1)
-		(layer "B.Cu")
-		(net "/Main Board/5v_local")
-	)
-	(segment
-		(start 72.498028 -78.9744)
-		(end 72.938028 -79.4144)
-		(width 1)
-		(layer "B.Cu")
-		(net "/Main Board/5v_local")
-	)
-	(segment
 		(start 58.303028 -75.6044)
 		(end 48.203028 -65.5044)
@@
 	)
 	(segment
+		(start 71.668028 -78.7794)
+		(end 71.863028 -78.9744)
+		(width 1)
+		(layer "B.Cu")
+		(net "/Main Board/5v_local")
+	)
+	(segment
 		(start 33.568028 -63.834248)
 		(end 33.568028 -57.8244)
@@
 	)
 	(segment
+		(start 71.863028 -78.9744)
+		(end 78.458028 -78.9744)
+		(width 1)
+		(layer "B.Cu")
+		(net "/Main Board/5v_local")
+	)
+	(segment
 		(start 59.603028 -75.6044)
 		(end 58.303028 -75.6044)
@@
 	)
 	(segment
-		(start 78.018028 -79.4144)
-		(end 84.368028 -73.0644)
-		(width 1)
-		(layer "B.Cu")
-		(net "/Main Board/5v_local")
-	)
-	(segment
 		(start 84.368028 -34.3294)
 		(end 77.383028 -27.3444)
@@
 	)
 	(segment
+		(start 78.458028 -78.9744)
+		(end 84.368028 -73.0644)
+		(width 1)
+		(layer "B.Cu")
+		(net "/Main Board/5v_local")
+	)
+	(segment
 		(start 137.346728 -152.9108)
 		(end 134.791328 -150.3554)
@@
 	)
 	(segment
-		(start 76.748028 -76.8744)
-		(end 73.573028 -76.8744)
+		(start 76.748028 -76.8344)
+		(end 74.168028 -76.8344)
+		(width 1)
+		(layer "B.Cu")
+		(net "/Main Board/5V_board1")
+	)
+	(segment
+		(start 74.168028 -76.8344)
+		(end 72.303028 -74.9694)
 		(width 1)
 		(layer "B.Cu")
@@
 	)
 	(segment
-		(start 73.573028 -76.8744)
+		(start 72.303028 -74.9694)
 		(end 71.668028 -74.9694)
 		(width 1)
@@
 	)
 	(segment
+		(start 177.078028 -134.6394)
+		(end 177.078028 -137.9614)
+		(width 1)
+		(layer "B.Cu")
+		(net "/LDR Driver/MUTE_CTRL")
+	)
+	(segment
+		(start 177.078028 -137.9614)
+		(end 174.792028 -140.2474)
+		(width 1)
+		(layer "B.Cu")
+		(net "/LDR Driver/MUTE_CTRL")
+	)
+	(segment
+		(start 144.693028 -130.2144)
+		(end 144.693028 -133.0284)
+		(width 1)
+		(layer "B.Cu")
+		(net "/LDR Driver/MUTE_CTRL")
+	)
+	(segment
+		(start 139.768828 -130.0508)
+		(end 144.529428 -130.0508)
+		(width 1)
+		(layer "B.Cu")
+		(net "/LDR Driver/MUTE_CTRL")
+	)
+	(segment
+		(start 144.693028 -133.0284)
+		(end 146.979028 -135.3144)
+		(width 1)
+		(layer "B.Cu")
+		(net "/LDR Driver/MUTE_CTRL")
+	)
+	(segment
 		(start 40.453028 -75.6044)
 		(end 38.053028 -78.0044)
@@
 	)
 	(segment
-		(start 177.078028 -134.6394)
-		(end 177.078028 -137.9614)
-		(width 1)
-		(layer "B.Cu")
-		(net "/LDR Driver/MUTE_CTRL")
-	)
-	(segment
-		(start 177.078028 -137.9614)
-		(end 174.792028 -140.2474)
-		(width 1)
-		(layer "B.Cu")
-		(net "/LDR Driver/MUTE_CTRL")
-	)
-	(segment
-		(start 144.693028 -130.2144)
-		(end 144.693028 -133.0284)
-		(width 1)
-		(layer "B.Cu")
-		(net "/LDR Driver/MUTE_CTRL")
-	)
-	(segment
-		(start 139.768828 -130.0508)
-		(end 144.529428 -130.0508)
-		(width 1)
-		(layer "B.Cu")
-		(net "/LDR Driver/MUTE_CTRL")
-	)
-	(segment
-		(start 144.693028 -133.0284)
-		(end 146.979028 -135.3144)
-		(width 1)
-		(layer "B.Cu")
-		(net "/LDR Driver/MUTE_CTRL")
-	)
-	(segment

Commit message: updates
Parts:
- removed the C24 at (-77.9, -51.8)
- removed the C26 at (-61.5, -44.5)
- removed the J13 at (-59.6, -50.9)
- removed the J14 at (-163.3, -20.4)
- removed the J22 at (-146.8, -36.9)
- removed the NT4 at (-52.9, -45.5)
- removed the Q10 at (-90.3, -50.8)
- removed the Q9 at (-81.3, -50.8)
- removed the R30 at (-94.4, -50.8)
- removed the R31 at (-85.8, -49.5)
- removed the R32 at (-78.0, -54.8)
- removed the R33 at (-61.5, -56.3)
- removed the U5 at (-97.6, -31.1)
- added R1: 1M, Resistor_THT:R_Axial_DIN0207_L6.3mm_D2.5mm_P2.54mm_Vertical, F.Cu at (45.6, -137.6)
- C16: renamed from C1; value 10nF -> 1uF
- C17: renamed from C11; value 10nF -> 1uF
- C18: renamed from C2; value 10nF -> 1uF
- C19: renamed from C12; value 10nF -> 1uF
- R16: renamed from R5; value 100K -> 1M
- R17: renamed from R13; value 100K -> 1M
- R26: renamed from R15; value 150 -> 100
- R8: renamed from R3; value 100K -> 1M
- R9: value 100K -> 1M
- moved C29 317.8 mm to (108.5, -34.3)
- moved J41 317.8 mm to (107.3, -43.1)
- moved R45 317.8 mm to (108.5, -37.5)
- moved U6 317.8 mm to (113.6, -30.5)
- moved D4 121.8 mm to (-86.4, -11.1)
- moved Q12 121.8 mm to (-84.5, 14.6)
- moved R44 121.8 mm to (-86.4, 6.31)
- moved R48 121.8 mm to (-56.6, -15.9)
- moved SW5 121.8 mm to (-80.5, -7.96)
- moved C28 121.8 mm to (-63.6, -12.1)
- moved D5 121.8 mm to (-63.6, -7.29)
- moved R42 121.8 mm to (-65.5, 16.5)
- moved R43 121.8 mm to (-56.4, 8.39)
- moved J13 4.32 mm to (45.6, -133.2), turned to 0 degrees
- moved U4 0.76 mm to (48.1, -119.3)
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- renumbered C3 to C1, C8 to C10, C9 to C11, C10 to C12, C19 to C13, C16 to C14, C18 to C15, C4 to C2, C14 to C20, C17 to C21, C32 to C22, C33 to C23, C13 to C24, C21 to C25, C27 to C26, C31 to C27, C37 to C28, C34 to C29, C5 to C3, C28 to C30, C29 to C31, C35 to C32, C36 to C33, C22 to C4, C23 to C5, C25 to C6, C15 to C7, C6 to C8, C7 to C9, D3 to D2, D2 to D3, D7 to D4, D6 to D5, J6 to J1, J3 to J10, J10 to J11, J5 to J12, J1 to J13, J2 to J14, J4 to J15, J45 to J16, J23 to J17, J39 to J18, J47 to J19, J7 to J2, J16 to J20, J17 to J21, J19 to J22, J20 to J23, J21 to J24, J30 to J26, J42 to J27, J43 to J28, J15 to J29, J8 to J3, J34 to J30, J35 to J31, J38 to J32, J46 to J33, J44 to J34, J40 to J35, J41 to J36, J29 to J38, J36 to J39, J9 to J4, J24 to J40, J33 to J41, J31 to J42, J32 to J43, J18 to J5, J25 to J6, J26 to J7, J27 to J8, J28 to J9, NT7 to NT3, NT8 to NT4, Q2 to Q1, Q12 to Q10, Q14 to Q11, Q13 to Q12, Q6 to Q2, Q1 to Q3, Q5 to Q4, Q4 to Q5, Q8 to Q6, Q3 to Q7, Q7 to Q8, Q11 to Q9, R4 to R10, R10 to R11, R55 to R12, R54 to R13, R2 to R14, R8 to R15, R6 to R18, R14 to R19, R27 to R2, R56 to R20, R53 to R21, R16 to R22, R17 to R23, R18 to R24, R19 to R25, R20 to R27, R22 to R28, R23 to R29, R28 to R3, R25 to R30, R26 to R31, R52 to R32, R43 to R33, R44 to R34, R39 to R35, R40 to R36, R41 to R37, R42 to R38, R48 to R39, R12 to R4, R49 to R40, R51 to R41, R46 to R42, R47 to R43, R45 to R44, R38 to R45, R21 to R46, R35 to R47, R50 to R48, R36 to R49, R24 to R5, R37 to R50, R1 to R6, SW3 to SW1, SW4 to SW2, SW1 to SW3, SW2 to SW4, U7 to U1, U1 to U3, U3 to U4, U4 to U5
Routing:
- net Net-(Q10-E): track 17.5 -> 0.00 mm
- net Net-(Q2-B): track 16.2 -> 0.00 mm
- net /LDR Driver/SHUNT_R: track 0.00 -> 16.2 mm
- net Net-(Q10-B): track 11.0 -> 0.00 mm
- net Net-(Q9-B): track 6.06 -> 0.00 mm
- net /LDR Board/AUDIO_IN: track 6.83 -> 10.1 mm
- net Net-(K1-Pad13): track 17.5 -> 17.0 mm
Other:
- board size 424.2 x 159 mm -> 316.9 x 199.6 mm

Commit message: updates v1b
Parts:
- added C34: 100nF, Capacitor_THT:C_Disc_D5.0mm_W2.5mm_P5.00mm, F.Cu at (219.8, -158.7)
- added C35: 100nF, Capacitor_THT:C_Disc_D5.0mm_W2.5mm_P5.00mm, F.Cu at (211.0, -153.6)
- added R51: 2.2K, Resistor_THT:R_Axial_DIN0207_L6.3mm_D2.5mm_P7.62mm_Horizontal, F.Cu at (212.0, -163.7)
- added R52: 100K, Resistor_THT:R_Axial_DIN0207_L6.3mm_D2.5mm_P7.62mm_Horizontal, F.Cu at (207.9, -153.6)
- added TH1: B3950, Connector_JST:JST_XH_B2B-XH-A_1x02_P2.50mm_Vertical, F.Cu at (216.6, -154.1)
- added U7: TL431LP, Package_TO_SOT_THT:TO-92_Inline_Wide, F.Cu at (214.8, -162.5)
- C15, C16, C17, C18, C19: footprint Capacitor_THT:C_Disc_D5.0mm_W2.5mm_P5.00mm -> Capacitor_THT:C_Rect_L7.2mm_W4.5mm_P5.00mm_FKS2_FKP2_MKS2_MKP2
- R12, R13: footprint Resistor_THT:R_Axial_DIN0309_L9.0mm_D3.2mm_P2.54mm_Vertical -> Resistor_THT:R_Axial_DIN0207_L6.3mm_D2.5mm_P7.62mm_Horizontal
- R16, R17, R8, R9: value 1M -> 100K; footprint Resistor_THT:R_Axial_DIN0207_L6.3mm_D2.5mm_P2.54mm_Vertical -> Resistor_THT:R_Axial_DIN0207_L6.3mm_D2.5mm_P7.62mm_Horizontal
- R32, R6, R7: footprint Resistor_THT:R_Axial_DIN0207_L6.3mm_D2.5mm_P2.54mm_Vertical -> Resistor_THT:R_Axial_DIN0207_L6.3mm_D2.5mm_P7.62mm_Horizontal
- moved R27 94.8 mm to (130.2, -62.3)
- moved J16 94.8 mm to (134.8, -68.9)
- moved J17 94.8 mm to (112.9, -62.3)
- moved Q11 94.8 mm to (134.8, -64.8)
- moved R26 94.8 mm to (118.3, -70.4)
- moved U5 94.8 mm to (118.3, -66.5)
- moved Q9 80.6 mm to (182.2, -168.9)
- moved Q10 77.7 mm to (181.5, -131.0)
- moved J22 74.9 mm to (216.6, -168.9), turned to 90 degrees
- moved C21 74.5 mm to (208.3, -171.4)
- moved R22 74.4 mm to (190.7, -171.4), turned to -90 degrees
- moved R10 73.2 mm to (172.6, -152.4), turned to 90 degrees
- moved R11 72.6 mm to (172.1, -126.2)
- moved R24 68.9 mm to (194.0, -171.4), turned to -90 degrees
- moved R6 67.9 mm to (147.2, -160.1), turned to 90 degrees
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Connections:
- A1 pad 12: /LDR Driver/PWM_SHUNT_R -> /LDR Driver/PWM_SER_R
- A1 pad 19: /LDR Driver/PWM_SER_R -> /LDR Driver/PWM_SHUNT_R
- A1 pad 2: /LDR Driver/PWM_SER_L -> /LDR Driver/COIL_CTRL_L
- A1 pad 33: GNDD -> /LDR Driver/AGND_PICO
- A1 pad 5: /LDR Driver/COIL_CTRL_L -> /LDR Driver/PWM_SHUNT_L
- J20 pad 1: /LDR Driver/COIL_R -> GNDD
- J20 pad 2: /LDR Driver/SERIAL_R -> GNDD
- J20 pad 3: GNDD -> /LDR Driver/SHUNT_R
- J20 pad 4: /LDR Driver/SHUNT_R -> /LDR Driver/COIL_R
- J20 pad 5: GNDD -> /LDR Driver/SERIAL_R
- J21 pad 1: /LDR Driver/COIL_L -> GNDD
- J21 pad 2: /LDR Driver/SERIAL_L -> GNDD
- J21 pad 3: GNDD -> /LDR Driver/SHUNT_L
- J21 pad 4: /LDR Driver/SHUNT_L -> /LDR Driver/COIL_L
- J21 pad 5: GNDD -> /LDR Driver/SERIAL_L
- J23 pad 2: /LDR Driver/SCL_L -> /LDR Driver/SDA_L
- J23 pad 3: /LDR Driver/SDA_L -> /LDR Driver/SCL_L
Routing:
- net /LDR Driver/ADC_TL431REF: track 0.00 -> 40.6 mm
- net /LDR Driver/COIL_L: track 4.65 -> 40.5 mm
- net /LDR Driver/COIL_R: track 5.37 -> 38.7 mm
- net /LDR Driver/ADC_NTC: track 0.00 -> 13.1 mm
- net Net-(Q2-B): track 0.00 -> 12.9 mm
- net /LDR Driver/PWM_SER_L: track 4.54 -> 14.3 mm
- net /LDR Driver/PWM_SER_R: track 4.94 -> 14.4 mm
- net /LDR Driver/PWM_SHUNT_R: track 16.2 -> 7.47 mm
- net /LDR Driver/SDA_L: track 12.4 -> 19.8 mm
- net /LDR Driver/SHUNT_L: track 6.10 -> 13.5 mm
- net /LDR Driver/SCL_L: track 18.8 -> 11.8 mm
- net Net-(Q10-G): track 13.2 -> 6.36 mm
- net /LDR Driver/SERIAL_R: track 5.40 -> 11.7 mm
- net /LDR Driver/SERIAL_L: track 6.45 -> 11.3 mm
- net /LDR Driver/ADC_VREF: track 0.00 -> 3.62 mm
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- added copper zone on B.Cu, net /LDR Driver/AGND_PICO
Other:
- board size 316.9 x 199.6 mm -> 332.1 x 201.9 mm

Commit message: updates
Parts:
- C13, C14: footprint Capacitor_THT:C_Disc_D5.0mm_W2.5mm_P5.00mm -> Capacitor_THT:C_Rect_L4.6mm_W3.0mm_P2.50mm_MKS02_FKP02
- C15: footprint Capacitor_THT:C_Rect_L7.2mm_W4.5mm_P5.00mm_FKS2_FKP2_MKS2_MKP2 -> Capacitor_THT:C_Rect_L4.6mm_W3.0mm_P2.50mm_MKS02_FKP02
- moved C34 11.4 mm to (208.4, -158.7), turned to 0 degrees
- moved R52 7.08 mm to (201.1, -151.8)
- moved D2 3.84 mm to (212.0, -175.4)
- moved R32 3.81 mm to (208.7, -137.1)
- moved C35 3.62 mm to (208.4, -151.0)
- moved U7 2.18 mm to (216.6, -163.7), turned to -90 degrees
- moved TH1 1.84 mm to (214.8, -153.6)
- moved J19 1.55 mm to (214.8, -141.9)
- moved J22 1.06 mm to (216.6, -167.8)
- turned C13 to -90 degrees
Connections:
- A1 pad 31: /LDR Driver/ADC_TL431REF -> /LDR Driver/ADC_NTC
- A1 pad 32: /LDR Driver/ADC_NTC -> /LDR Driver/AGND_PICO
Routing:
- net /LDR Driver/ADC_TL431REF: track 40.6 -> 23.6 mm
- net /LDR Driver/MUTE_CTRL: track 16.8 -> 18.8 mm
- net /LDR Driver/ADC_NTC: track 13.1 -> 14.1 mm
- net /LDR Driver/5V_board1: track 6.04 -> 5.44 mm

Commit message: updates
Parts:
- removed J20, J21: CTRL, Connector_JST:JST_XH_B6B-XH-A_1x06_P2.50mm_Vertical
- added J25: LDR_R, Connector_JST:JST_XH_B5B-XH-A_1x05_P2.50mm_Vertical, F.Cu at (141.5, -131.6)
- added J37: LDR_L, Connector_JST:JST_XH_B5B-XH-A_1x05_P2.50mm_Vertical, F.Cu at (140.9, -157.7)
- added R53: 4.7K, Resistor_THT:R_Axial_DIN0207_L6.3mm_D2.5mm_P2.54mm_Vertical, F.Cu at (210.0, -143.4)
- added U8: DS18B20, Connector_JST:JST_XH_B3B-XH-A_1x03_P2.50mm_Vertical, F.Cu at (216.6, -135.3)
- moved R32 9.67 mm to (199.8, -133.3), turned to -90 degrees
- moved J19 5.90 mm to (210.5, -137.8)
- moved J18 2.67 mm to (214.5, -128.2)
- moved C11 1.52 mm to (61.1, -141.1)
- moved C12 1.52 mm to (61.1, -151.8)
- moved C13 1.52 mm to (48.2, -151.8)
- moved C14 1.52 mm to (41.4, -151.8)
- moved C15 1.52 mm to (37.8, -151.8)
- moved C7 1.52 mm to (59.0, -121.3)
- moved C8 1.52 mm to (59.1, -126.4)
- moved C9 1.52 mm to (59.1, -129.5)
- moved D1 1.52 mm to (42.3, -119.4)
- moved J10 1.52 mm to (55.7, -115.0)
- moved J11 1.52 mm to (34.7, -115.0)
- moved J12 1.52 mm to (57.4, -159.9)
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Connections:
- A1 pad 27: /LDR Driver/MUTE_CTRL -> /LDR Driver/DQ_IN
Routing:
- net /LDR Driver/3.3V_PICO: track 28.3 -> 50.7 mm
- net /LDR Driver/DQ_IN: track 0.00 -> 17.2 mm
- net /LDR Driver/5v_local: track 132.6 -> 137.2 mm
- net /LDR Driver/SHUNT_R: track 14.2 -> 12.7 mm
- net /LDR Driver/COIL_R: track 38.7 -> 37.3 mm
- net /LDR Driver/UART_TX: track 10.6 -> 9.33 mm
- net /LDR Driver/UART_RX: track 6.38 -> 5.19 mm
- net /LDR Driver/SERIAL_R: track 11.7 -> 10.6 mm
- net /LDR Driver/MUTE_CTRL: track 18.8 -> 18.1 mm
Other:
- outline, holes or cut-outs redrawn

Commit message: v1b
Parts:
- removed J11: CTRL, Connector_JST:JST_XH_B6B-XH-A_1x06_P2.50mm_Vertical
- added J44: LDR_L, Connector_JST:JST_XH_B5B-XH-A_1x05_P2.50mm_Vertical, F.Cu at (33.7, -114.3)
- C13, C14, C15: footprint Capacitor_THT:C_Rect_L4.6mm_W3.0mm_P2.50mm_MKS02_FKP02 -> Capacitor_THT:C_Rect_L7.2mm_W2.5mm_P5.00mm_FKS2_FKP2_MKS2_MKP2
- C34, C35: footprint Capacitor_THT:C_Disc_D5.0mm_W2.5mm_P5.00mm -> Capacitor_THT:C_Rect_L7.2mm_W2.5mm_P5.00mm_FKS2_FKP2_MKS2_MKP2
- D1: footprint Diode_THT:D_DO-35_SOD27_P7.62mm_Horizontal -> Diode_THT:D_DO-35_SOD27_P2.54mm_Vertical_CathodeUp
- NT1: value GNDD_TO_GNDA -> ATOGNDA
- moved J13 22.5 mm to (24.8, -135.9), turned to -90 degrees
- moved U4 20.5 mm to (29.1, -118.8)
- moved R1 17.8 mm to (29.4, -136.6), turned to -90 degrees
- moved J14 7.75 mm to (36.5, -134.8), turned to 180 degrees
- moved K1 6.40 mm to (48.8, -122.0)
- moved U2 5.50 mm to (36.7, -118.8)
- moved J12 2.13 mm to (55.8, -161.3)
- moved C13 1.96 mm to (50.1, -152.4)
- moved J10 1.53 mm to (57.1, -114.3)
- moved D1 1.53 mm to (43.7, -118.8)
- moved J15 1.27 mm to (38.3, -156.4)
- moved R30 0.76 mm to (198.3, -142.2)
- moved C12 0.64 mm to (61.1, -152.4)
- moved C14 0.64 mm to (41.4, -152.4)
- moved C15 0.64 mm to (37.8, -152.4)
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Connections:
- C1 pad 2: GNDD -> /5V power/gnd_analog
- C2 pad 2: GNDD -> /5V power/gnd_analog
- C3 pad 2: GNDD -> /5V power/gnd_analog
- C7 pad 2: GNDD -> /LDR Board/gnd_analog
- C8 pad 2: GNDD -> /LDR Board/gnd_analog
- C9 pad 2: GNDD -> /LDR Board/gnd_analog
- J10 pad 1: GNDD -> /LDR Board/gnd_analog
- J3 pad 1: GNDD -> /5V power/gnd_analog
- J4 pad 1: GNDD -> /5V power/gnd_analog
- L2 pad 4: GNDD -> /5V power/gnd_analog
- NT1 pad 1: GNDD -> /LDR Board/gnd_analog
- U2 pad 3: Net-(K1-Pad4) -> Net-(K1-Pad13)
- U2 pad 4: Net-(K1-Pad13) -> Net-(K1-Pad4)
- U4 pad 3: Net-(K1-Pad13) -> AUDIO_GND
- U4 pad 4: AUDIO_GND -> Net-(K1-Pad13)
Routing:
- net /LDR Board/AUDIO_IN: track 10.1 -> 25.7 mm
- net /LDR Board/MIDDLE_JUNCTION: track 3.97 -> 9.01 mm
- net Net-(K1-Pad4): track 17.0 -> 12.9 mm
- net Net-(K1-Pad13): track 16.8 -> 12.9 mm
- net /LDR Board/5v_local: track 7.51 -> 10.9 mm
- net /LDR Driver/ADC_TL431REF: track 23.6 -> 25.6 mm
- net /LDR Driver/5v_local: track 137.2 -> 138.8 mm
- net /LDR Board/SHUNT_POS: track 6.07 -> 7.62 mm
- net /LDR Board/AUDIO_OUT: track 6.27 -> 4.75 mm
- net /LDR Board/COIL_NEG: track 8.67 -> 7.75 mm
- net /LDR Board/SDA: track 5.30 -> 6.09 mm
- net /LDR Board/SCL: track 5.32 -> 6.11 mm
- net /LDR Driver/SERIAL_L: track 11.3 -> 10.7 mm
- net /LDR Board/TOP_JUNCTION: track 6.94 -> 7.58 mm
- net /LDR Board/A1: track 7.36 -> 8.00 mm
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- added copper zone on B.Cu, net /LDR Board/gnd_analog
Other:
- outline, holes or cut-outs redrawn
