File: amp_v3/ldr_volume/ldr_volume.kicad_pcb (KiCad board)
At the start: 2 copper layers, 332.1 x 201.9 mm, 171 parts, among them J1 PWR1, J10 5v_in, J12 I2C_R, J13 A_IN, J14 A_OUT, J15 ADS1115, J16 MUTE_OUT, J17 MUTE, J18 UART, J19 MUTE, J2 PWR2, J22 PWR_IN, J23 I2C_L, J24 I2C_R, J25 LDR_R, J26 TFT, J27 PWR_BTN, J28 PWR_BTN_LED, J29 PWR_IN, J3 PWR3, J30 I2C, J31 BTN_VOL, J32 BTN_MENU, J33 ALPS, J34 PWR_RLY, J35 BTN_EXT1, J36 BTN_EXT2, J37 LDR_L, J38 IR, J39 MUTE, J4 PWR4, J40 UART, J41 IR_SENSOR, J42 S_AIN_L, J43 S_AIN_R, J44 LDR_L, J5 PWR3, J6 PWR4, J7 Conn_01x03_Pin, J8 5V_IN, J9 5V_IN, K1 G5V-2, Q1 BC557, Q10 2N7000, Q11 BC547, Q12 BC547, Q2 BC557, Q3 BC547, Q4 BC547, Q5 BC557, Q6 BC557, Q7 BC547, Q8 BC547, Q9 2N7000, SW1 SW_LT, SW2 SW_RT, SW3 SW_UP, SW4 SW_DN, SW5 SW_PWR, U1 IRM-10-5, U2 NSL-32-SR3-Rseries, U3 MCP1700x-330xxTO, U4 NSL-32-SR3-Rshunt, U5 4N25, U6 TSOP312xx, U7 TL431LP, U8 DS18B20

Commit message: updates
Parts:
- J27: value PWR_BTN -> PWR_CTRL
- J38: value IR -> MUTE
- J39: value MUTE -> IR
Connections:
- A2 pad 14: /Main Board/PWR_BTN -> /Main Board/PWR_CTRL
- J27 pad 2: /Main Board/PWR_BTN -> /Main Board/PWR_CTRL
Routing:
- net /Main Board/PWR_CTRL: track 0.00 -> 4.45 mm
- net /Main Board/PWR_BTN: track 4.45 -> 0.00 mm
Changed lines of the file:
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@@
 		(tags "Through hole pin header THT 1x03 2.54mm single row")
 		(property "Reference" "J39"
-			(at 0 -2.38 90)
+			(at 0 6.985 90)
 			(layer "F.SilkS")
 			(effects
@@
 			)
 		)
-		(property "Value" "MUTE"
-			(at 0 7.46 90)
+		(property "Value" "IR"
+			(at -1.905 2.54 180)
 			(layer "F.Fab")
 			(effects
@@
 		)
 		(fp_text user "${REFERENCE}"
-			(at 0 2.54 0)
+			(at 0 6.985 90)
 			(layer "F.Fab")
 			(effects
@@
 		(tags "Resistor Axial_DIN0207 series Axial Vertical pin pitch 2.54mm 0.25W = 1/4W length 6.3mm diameter 2.5mm")
 		(property "Reference" "R41"
-			(at 1.27 -2.37 0)
+			(at 3.175 1.27 0)
 			(layer "F.SilkS")
 			(effects
@@
 		)
 		(property "Value" "10K"
-			(at 1.27 2.37 0)
+			(at -2.54 0 0)
 			(layer "F.Fab")
 			(effects
@@
 		)
 		(fp_text user "${REFERENCE}"
-			(at 1.27 -2.37 0)
+			(at 3.175 1.27 0)
 			(layer "F.Fab")
 			(effects
@@
 			)
 		)
-		(property "Value" "IR"
-			(at 0 7.46 90)
+		(property "Value" "MUTE"
+			(at -1.905 2.54 180)
 			(layer "F.Fab")
 			(effects
@@
 			)
 		)
-		(property "Value" "PWR_BTN"
-			(at 0 4.92 90)
+		(property "Value" "PWR_CTRL"
+			(at 1.905 1.27 180)
 			(layer "F.Fab")
 			(effects
@@
 		)
 		(fp_text user "${REFERENCE}"
-			(at 0 1.27 0)
+			(at 0 4.445 90)
 			(layer "F.Fab")
 			(effects
@@
 			(layers "*.Cu" "*.Mask")
 			(remove_unused_layers no)
-			(net "/Main Board/PWR_BTN")
+			(net "/Main Board/PWR_CTRL")
 			(pinfunction "Pin_2_2")
 			(pintype "passive")
@@
 		(tags "Through hole pin header THT 1x05 2.54mm single row")
 		(property "Reference" "J33"
-			(at 0 -2.38 90)
+			(at -1.27 -3.175 180)
 			(layer "F.SilkS")
 			(effects
@@
 		)
 		(property "Value" "ALPS"
-			(at 0 12.54 90)
+			(at 0.635 -3.175 180)
 			(layer "F.Fab")
 			(effects
@@
 		)
 		(fp_text user "${REFERENCE}"
-			(at 0 5.08 0)
+			(at -1.27 -3.175 0)
 			(layer "F.Fab")
 			(effects
@@
 		(tags "Through hole pin header THT 1x04 2.54mm single row")
 		(property "Reference" "J34"
-			(at -1.905 0.635 180)
+			(at 1.27 -2.54 180)
 			(layer "F.SilkS")
 			(effects
@@
 		)
 		(property "Value" "PWR_RLY"
-			(at 0 10 90)
+			(at 2.54 -1.27 180)
 			(layer "F.Fab")
 			(effects
@@
 		)
 		(fp_text user "${REFERENCE}"
-			(at 0 3.81 0)
+			(at 1.27 -2.54 0)
 			(layer "F.Fab")
 			(effects
@@
 			(layers "*.Cu" "*.Mask")
 			(remove_unused_layers no)
-			(net "/Main Board/PWR_BTN")
+			(net "/Main Board/PWR_CTRL")
 			(pinfunction "GPIO10_14")
 			(pintype "bidirectional")
@@
 		)
 		(property "Value" "PWR_BTN_LED"
-			(at 0 4.92 90)
+			(at 1.905 3.81 0)
 			(layer "F.Fab")
 			(effects
@@
 	)
 	(segment
-		(start 38.728028 -118.0744)
-		(end 36.748028 -120.0544)
+		(start 190.24518 -142.1524)
+		(end 188.93858 -140.8458)
 		(width 1)
 		(layer "B.Cu")
-		(net "/LDR Board/SERIAL_POS")
+		(net "/LDR Driver/SDA_R")
 	)
 	(segment
-		(start 38.728028 -114.3394)
-		(end 38.728028 -118.0744)
+		(start 188.93858 -140.8458)
+		(end 186.504828 -140.8458)
 		(width 1)
 		(layer "B.Cu")
-		(net "/LDR Board/SERIAL_POS")
+		(net "/LDR Driver/SDA_R")
 	)
 	(segment
-		(start 41.188028 -114.4194)
-		(end 41.108028 -114.3394)
+		(start 186.504828 -140.8458)
+		(end 183.378476 -140.8458)
 		(width 1)
 		(layer "B.Cu")
-		(net "/LDR Board/COIL_NEG")
+		(net "/LDR Driver/SDA_R")
 	)
 	(segment
-		(start 41.188028 -118.7844)
-		(end 41.188028 -121.9869)
+		(start 190.667028 -142.1524)
+		(end 190.24518 -142.1524)
 		(width 1)
 		(layer "B.Cu")
-		(net "/LDR Board/COIL_NEG")
+		(net "/LDR Driver/SDA_R")
 	)
 	(segment
-		(start 41.188028 -118.7844)
-		(end 41.188028 -114.4194)
+		(start 183.378476 -140.8458)
+		(end 181.857876 -142.3664)
 		(width 1)
 		(layer "B.Cu")
-		(net "/LDR Board/COIL_NEG")
+		(net "/LDR Driver/SDA_R")
 	)
 	(segment
-		(start 41.188028 -121.9869)
-		(end 41.140528 -122.0344)
+		(start 181.857876 -142.3664)
+		(end 180.888028 -142.3664)
 		(width 1)
 		(layer "B.Cu")
-		(net "/LDR Board/COIL_NEG")
+		(net "/LDR Driver/SDA_R")
 	)
 	(segment
@@
 	)
 	(segment
-		(start 33.728028 -115.4544)
-		(end 29.128028 -120.0544)
-		(width 1)
-		(layer "B.Cu")
-		(net "/LDR Board/SHUNT_POS")
-	)
-	(segment
-		(start 33.728028 -114.3394)
-		(end 33.728028 -115.4544)
-		(width 1)
-		(layer "B.Cu")
-		(net "/LDR Board/SHUNT_POS")
-	)
-	(segment
-		(start 190.24518 -142.1524)
-		(end 188.93858 -140.8458)
-		(width 1)
-		(layer "B.Cu")
-		(net "/LDR Driver/SDA_R")
-	)
-	(segment
-		(start 188.93858 -140.8458)
-		(end 186.504828 -140.8458)
-		(width 1)
-		(layer "B.Cu")
-		(net "/LDR Driver/SDA_R")
-	)
-	(segment
-		(start 186.504828 -140.8458)
-		(end 183.378476 -140.8458)
+		(start 41.188028 -114.4194)
+		(end 41.108028 -114.3394)
 		(width 1)
 		(layer "B.Cu")
-		(net "/LDR Driver/SDA_R")
+		(net "/LDR Board/COIL_NEG")
 	)
 	(segment
-		(start 190.667028 -142.1524)
-		(end 190.24518 -142.1524)
+		(start 41.188028 -118.7844)
+		(end 41.188028 -121.9869)
 		(width 1)
 		(layer "B.Cu")
-		(net "/LDR Driver/SDA_R")
+		(net "/LDR Board/COIL_NEG")
 	)
 	(segment
-		(start 183.378476 -140.8458)
-		(end 181.857876 -142.3664)
+		(start 41.188028 -118.7844)
+		(end 41.188028 -114.4194)
 		(width 1)
 		(layer "B.Cu")
-		(net "/LDR Driver/SDA_R")
+		(net "/LDR Board/COIL_NEG")
 	)
 	(segment
-		(start 181.857876 -142.3664)
-		(end 180.888028 -142.3664)
+		(start 41.188028 -121.9869)
+		(end 41.140528 -122.0344)
 		(width 1)
 		(layer "B.Cu")
-		(net "/LDR Driver/SDA_R")
+		(net "/LDR Board/COIL_NEG")
 	)
 	(segment
@@
 	)
 	(segment
-		(start 45.633028 -45.1244)
-		(end 41.188028 -45.1244)
-		(width 1)
-		(layer "B.Cu")
-		(net "/Main Board/PWR_BTN")
-	)
-	(segment
 		(start 172.633028 -165.1394)
 		(end 169.498028 -165.1394)
@@
 	)
 	(segment
+		(start 33.728028 -115.4544)
+		(end 29.128028 -120.0544)
+		(width 1)
+		(layer "B.Cu")
+		(net "/LDR Board/SHUNT_POS")
+	)
+	(segment
+		(start 33.728028 -114.3394)
+		(end 33.728028 -115.4544)
+		(width 1)
+		(layer "B.Cu")
+		(net "/LDR Board/SHUNT_POS")
+	)
+	(segment
 		(start 180.57958 -161.1658)
 		(end 177.763028 -158.349248)
@@
 	)
 	(segment
+		(start 38.728028 -118.0744)
+		(end 36.748028 -120.0544)
+		(width 1)
+		(layer "B.Cu")
+		(net "/LDR Board/SERIAL_POS")
+	)
+	(segment
+		(start 38.728028 -114.3394)
+		(end 38.728028 -118.0744)
+		(width 1)
+		(layer "B.Cu")
+		(net "/LDR Board/SERIAL_POS")
+	)
+	(segment
 		(start 39.283028 -62.9044)
 		(end 38.648028 -62.2694)
@@
 		(net "/Main Board/TFT_BLK")
 	)
+	(segment
+		(start 45.633028 -45.1244)
+		(end 41.188028 -45.1244)
+		(width 1)
+		(layer "B.Cu")
+		(net "/Main Board/PWR_CTRL")
+	)
 	(zone
