File: amp_v3/ldr_volume/_restore_backup_2026-08-31T21-18-52-249/board#5.kicad_sch (KiCad schematic)
At the start: 62 parts, among them J14 Conn_01x05_Pin, J15 PWR_IN, J22 PWR_SEL, J24 UART, J29 IR, J30 TFT, J31 S_AIN_L, J32 S_AIN_R, J33 IR_SENSOR, J34 I2C, J35 BTN_VOL, J36 MUTE, J38 BTN_MENU, J40 BTN_EXT1, J41 BTN_EXT2, J42 PWR_BTN, J43 PWR_BTN_LED, J44 PWR_RLY, J46 ALPS, Q13 BC547, SW1 SW_UP, SW2 SW_DN, SW3 SW_LT, SW4 SW_RT, SW5 SW_PWR, U6 TSOP312xx

Commit message: update
Parts:
- removed C34, C37: 100nF, Capacitor_THT:C_Disc_D5.0mm_W2.5mm_P5.00mm, symbol Device:C
- removed C35, C36: 10nF, Capacitor_THT:C_Disc_D5.0mm_W2.5mm_P5.00mm, symbol Device:C
- removed D6: WHITE LED, LED_THT:LED_D3.0mm_Horizontal_O1.27mm_Z2.0mm, symbol Device:LED
- removed D7: LED, LED_THT:LED_D3.0mm_Horizontal_O1.27mm_Z2.0mm, symbol Device:LED
- removed J14: Conn_01x05_Pin, Connector_PinHeader_2.54mm:PinHeader_1x05_P2.54mm_Horizontal, symbol Connector:Conn_01x05_Pin
- removed J22: PWR_SEL, Connector_PinHeader_2.54mm:PinHeader_1x03_P2.54mm_Vertical, symbol Connector:Conn_01x03_Pin
- removed J29: IR, Connector_PinHeader_2.54mm:PinHeader_1x03_P2.54mm_Vertical, symbol Connector:Conn_01x03_Pin
- removed J30: TFT, Connector_PinHeader_2.54mm:PinHeader_1x09_P2.54mm_Horizontal, symbol Connector:Conn_01x09_Pin
- removed J36: MUTE, Connector_PinHeader_2.54mm:PinHeader_1x03_P2.54mm_Vertical, symbol Connector:Conn_01x03_Pin
- removed J42: PWR_BTN, Connector_PinHeader_2.54mm:PinHeader_1x02_P2.54mm_Vertical, symbol Connector:Conn_01x02_Pin
- removed J43: PWR_BTN_LED, Connector_PinHeader_2.54mm:PinHeader_1x02_P2.54mm_Vertical, symbol Connector:Conn_01x02_Pin
- removed J44: PWR_RLY, Connector_PinHeader_2.54mm:PinHeader_1x04_P2.54mm_Vertical, symbol Connector:Conn_01x04_Pin
- removed J46: ALPS, Connector_PinHeader_2.54mm:PinHeader_1x05_P2.54mm_Vertical, symbol Connector:Conn_01x05_Pin
- removed Q13: BC547, Package_TO_SOT_THT:TO-92_Inline_Wide, symbol Transistor_BJT:BC547
- removed R45, R50: 1k, Resistor_THT:R_Axial_DIN0207_L6.3mm_D2.5mm_P7.62mm_Horizontal, symbol Device:R
- removed R46, R47: 100, Resistor_THT:R_Axial_DIN0207_L6.3mm_D2.5mm_P2.54mm_Vertical, symbol Device:R
- removed R48, R49: 22, Resistor_THT:R_Axial_DIN0207_L6.3mm_D2.5mm_P2.54mm_Vertical, symbol Device:R
- removed R51: 10K, Resistor_THT:R_Axial_DIN0207_L6.3mm_D2.5mm_P2.54mm_Vertical, symbol Device:R
- removed SW5: SW_PWR, Button_Switch_THT:SW_SPST_Omron_B3F-50xx, symbol Switch:SW_Push
- added C30: 4.7uF, Capacitor_THT:CP_Radial_D5.0mm_P2.50mm, symbol Device:C_Polarized
- added J14: Conn_02x04_Counter_Clockwise, Connector_PinHeader_2.54mm:PinHeader_2x04_P2.54mm_Vertical, symbol Connector_Generic:Conn_02x04_Counter_Clockwise
- added J29: TFT, Connector_PinHeader_2.54mm:PinHeader_1x08_P2.54mm_Horizontal, symbol Connector:Conn_01x08_Pin
- added J30: IR, Connector_JST:JST_XH_B3B-XH-A_1x03_P2.50mm_Vertical, symbol Connector:Conn_01x03_Pin
- C28, C29: value 1uF -> 2.2uF; footprint Capacitor_THT:C_Rect_L7.2mm_W5.5mm_P5.00mm_FKS2_FKP2_MKS2_MKP2 -> Capacitor_THT:C_Rect_L7.2mm_W2.5mm_P5.00mm_FKS2_FKP2_MKS2_MKP2
- D2: footprint Diode_THT:D_DO-41_SOD81_P3.81mm_Vertical_CathodeUp -> Diode_THT:D_DO-41_SOD81_P7.62mm_Horizontal
- J31, J32: footprint Connector_PinHeader_2.54mm:PinHeader_1x02_P2.54mm_Vertical -> Connector_JST:JST_XH_B2B-XH-A_1x02_P2.50mm_Vertical
- J33: value IR_SENSOR -> IR
- J34: value I2C -> SDA; footprint Connector_PinHeader_2.54mm:PinHeader_1x04_P2.54mm_Vertical -> Connector_JST:JST_XH_B4B-XH-A_1x04_P2.50mm_Vertical
- R38: value 100 -> 10K
- SW1: value SW_UP -> SW_Push
- SW2: value SW_DN -> SW_Push
- SW3: value SW_LT -> SW_Push
- SW4: value SW_RT -> SW_Push
Connections:
- net ALPS_L is gone; now on net TFT_RST: A2.10 (GPIO7)
- net ALPS_R is gone; now on net TFT_DC: A2.9 (GPIO6)
- net RLCTRL is gone; now on net TFT_CS: A2.7 (GPIO5)
- net 3.3V_PICO: now also J14.1 (Pin_1), J14.2 (Pin_2), J29.1 (Pin_1), J30.2 (Pin_2)
- net 5V_board1: now also C13.1, C21.1
- net AGND_L: now also R36.2
- net AGND_PICO: no longer A2.31 (GPIO26_ADC0), R36.2, R37.2
- net AGND_R: now also R37.2
- net BTN_DN: now also A2.19 (GPIO14), J35.3 (Pin_3); no longer A2.17 (GPIO13), J35.2 (Pin_2)
- net BTN_LT: now also A2.20 (GPIO15), J35.1 (Pin_1); no longer A2.16 (GPIO12), J35.3 (Pin_3)
- net BTN_RT: now also A2.2 (GPIO1); no longer A2.5 (GPIO3)
- net BTN_UP: now also A2.1 (GPIO0), J38.3 (Pin_3); no longer A2.4 (GPIO2), J38.2 (Pin_2)
- net GNDD: now also J35.2 (Pin_2), J38.2 (Pin_2), C30.2, J14.3 (Pin_3), J14.4 (Pin_4), J14.8 (Pin_8), J29.4 (Pin_4), J30.3 (Pin_3); no longer J35.1 (Pin_1), J38.3 (Pin_3)
- net IR: now also A2.24 (GPIO18), J30.1 (Pin_1); no longer A2.15 (GPIO11)
- net SCL: now also A2.22 (GPIO17), J34.2 (Pin_2); no longer A2.20 (GPIO15), J34.3 (Pin_3)
- net SDA: now also A2.21 (GPIO16), J34.3 (Pin_3); no longer A2.19 (GPIO14), J34.2 (Pin_2)
- net TFT_BLK: now also A2.6 (GPIO4), J29.6 (Pin_6); no longer A2.27 (GPIO21)
- net TFT_CS: now also J29.5 (Pin_5); no longer A2.22 (GPIO17)
- net TFT_DC: now also J29.3 (Pin_3); no longer A2.21 (GPIO16)
- net TFT_RST: now also J29.2 (Pin_2); no longer A2.26 (GPIO20)
- net TFT_SCL: now also A2.4 (GPIO2), J29.8 (Pin_8)
- net TFT_SDA: now also A2.5 (GPIO3), J29.7 (Pin_7)
- net UART_RX: now also A2.17 (GPIO13); no longer A2.2 (GPIO1)
- net UART_TX: now also A2.16 (GPIO12); no longer A2.1 (GPIO0)
- net at R38.1, U6.2 (Vs): now also C30.1
- net 5v_local: no longer names the net of A2.39 (VSYS), D2.1 (K)
- net 5v_local: no longer C13.1, C21.1
- net MUTE_CTRL: no longer names the net of A2.11 (GPIO8)
- net PWR_BTN renamed EXT_1
- net EXT_1: now also J14.7 (Pin_7)
- net PWR_BTN_LED renamed PWR_CTRL
- net PWR_CTRL: now also J14.6 (Pin_6)
- new net EXT_2: A2.15 (GPIO11), J14.5 (Pin_5)
- no-connect marks 7 -> 0
Other:
- note removed: "Push button 5v or 3v led direct gpio drive"
- moved on the sheet: C27, C31, C32, C33, D2, J33, J35, J38, J40, J41, R38, R41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
