File: amp_v3/jfet_buffer_splitter/jfet_buffer.kicad_sch (KiCad schematic)
At the start: 25 parts, among them J3 AUDIO_IN, J4 AUDIO_IN, J5 AUDIO_OUT, J9 PWR_IN, Q1 2N5457, Q2 BC549C

Commit message: updates
Parts:
- removed C7: 470uF, Capacitor_THT:CP_Radial_D8.0mm_P3.50mm, symbol Device:C_Polarized
- removed C8: 470uF (low ESR), Capacitor_THT:CP_Radial_D8.0mm_P3.50mm, symbol Device:C_Polarized
- removed C9: 100nF, Capacitor_THT:C_Rect_L7.0mm_W2.5mm_P5.00mm, symbol Device:C
- removed D1: 1N4747, Diode_THT:D_A-405_P5.08mm_Vertical_AnodeUp, symbol Device:D_Zener_Filled
- removed D2: 1n4148, Diode_THT:D_A-405_P5.08mm_Vertical_AnodeUp, symbol Device:D_Filled
- removed D3, D4: 1N4007, Diode_THT:D_A-405_P5.08mm_Vertical_AnodeUp, symbol Device:D_Filled
- removed J4: AUDIO_IN, Connector_JST:JST_XH_B2B-XH-A_1x02_P2.50mm_Vertical, symbol Connector:Conn_01x02_Pin
- removed J9: PWR_IN, Connector_JST:JST_XH_B2B-XH-A_1x02_P2.50mm_Vertical, symbol Connector:Conn_01x02_Pin
- removed Q2: BC549C, Package_TO_SOT_THT:TO-92_Inline_Wide, symbol Transistor_BJT:BC547
- added C1: 100uF, Capacitor_THT:CP_Radial_D5.0mm_P2.50mm, symbol Device:C_Polarized
- added J1: PWR, Connector_JST:JST_XH_B2B-XH-A_1x02_P2.50mm_Vertical, symbol Connector:Conn_01x02_Pin
- added J2, J4, J6, J7: Conn_01x01_Pin, Connector_PinHeader_1.00mm:PinHeader_1x01_P1.00mm_Vertical, symbol Connector:Conn_01x01_Pin
- added J8: OUT2, Connector_JST:JST_XH_B2B-XH-A_1x02_P2.50mm_Vertical, symbol Connector:Conn_01x02_Pin
- added Q2: 2N5457, Package_TO_SOT_THT:TO-92L_Inline_Wide, symbol power_ctrl-rescue:Q_NJFET_DSG
- added R7: 3.9K, Resistor_THT:R_Axial_DIN0207_L6.3mm_D2.5mm_P7.62mm_Horizontal, symbol power_ctrl-rescue:R
- C5: footprint Capacitor_THT:C_Rect_L7.0mm_W2.5mm_P5.00mm -> Capacitor_THT:C_Rect_L7.2mm_W2.5mm_P5.00mm_FKS2_FKP2_MKS2_MKP2
- J3: value AUDIO_IN -> INPUT
- J5: value AUDIO_OUT -> OUT1
- NT1: footprint nettie 1.0:NetTie-2_SMD_Pad1.0o -> NetTie:NetTie-2_SMD_Pad2.0mm
- R4: footprint Resistor_THT:R_Axial_DIN0309_L9.0mm_D3.2mm_P2.54mm_Vertical -> Resistor_THT:R_Axial_DIN0207_L6.3mm_D2.5mm_P7.62mm_Horizontal
- R6: value 240 -> 100; footprint Resistor_THT:R_Axial_DIN0309_L9.0mm_D3.2mm_P2.54mm_Vertical -> Resistor_THT:R_Axial_DIN0207_L6.3mm_D2.5mm_P7.62mm_Horizontal
Connections:
- net 22V_REG is gone; now on net VBIAS_OUT: R6.2
- net GND: now also C1.2, J1.1 (Pin_1), J8.1 (Pin_1), R7.2
- net at R6.1: now also Q2.3 (G); no longer C5.1
- net 20V_JFET renamed +20V
- net +20V: now also C5.1, C1.1, J1.2 (Pin_2), J2.1 (Pin_1), J4.1 (Pin_1), J6.1 (Pin_1), J7.1 (Pin_1), Q2.1 (D)
- net OUT renamed OUT1
- new net OUT2: J8.2 (Pin_2), Q2.2 (S), R7.1
Other:
- note removed: "Rbias = 560 for 24V input Rbias = 240 - 270 for 22V input"
- moved on the sheet: J3, J5, NT1
