File: amp_v3/opa_buffer_splitter/_restore_backup_2026-10-07T19-32-36-209/buffer.kicad_sch (KiCad schematic)
At the start: 19 parts, among them J6 OP_PWR, J7 AUDIO_IN, J8 AOUT_MASTER, J9 AOUT_VIS, U2 OPA1656

Commit message: updates
Parts:
- removed C10, C16: 4.7uF, Capacitor_THT:CP_Radial_D5.0mm_P2.50mm, symbol Device:C_Polarized
- removed C11, C12, C13, C9: 100nF, Capacitor_THT:C_Disc_D4.3mm_W1.9mm_P5.00mm, symbol Device:C
- removed C14, C15: 10uF esr, Capacitor_THT:CP_Radial_D5.0mm_P2.50mm, symbol Device:C_Polarized
- removed C8: 1uF PP, capacitor JFC:JFC, symbol Device:C
- removed J6: OP_PWR, Connector_JST:JST_XH_B3B-XH-A_1x03_P2.50mm_Vertical, symbol Connector:Conn_01x03_Pin
- removed J7: AUDIO_IN, Connector_JST:JST_XH_B2B-XH-A_1x02_P2.50mm_Vertical, symbol Connector:Conn_01x02_Pin
- removed J8: AOUT_MASTER, Connector_JST:JST_XH_B2B-XH-A_1x02_P2.50mm_Vertical, symbol Connector:Conn_01x02_Pin
- removed J9: AOUT_VIS, Connector_JST:JST_XH_B2B-XH-A_1x02_P2.50mm_Vertical, symbol Connector:Conn_01x02_Pin
- removed R1: 100K, Resistor_THT:R_Axial_DIN0207_L6.3mm_D2.5mm_P2.54mm_Vertical, symbol Device:R
- removed R2, R3: 10R, Resistor_THT:R_Axial_DIN0207_L6.3mm_D2.5mm_P10.16mm_Horizontal, symbol Device:R
- removed R4, R5: 47R, Resistor_THT:R_Axial_DIN0207_L6.3mm_D2.5mm_P2.54mm_Vertical, symbol Device:R
- removed U2: OPA1656, Package_DIP:SMDIP-8_W7.62mm, symbol Amplifier_Operational:OPA1656ID
- added C17, C19, C20, C23: 100nF, Capacitor_THT:C_Disc_D4.3mm_W1.9mm_P5.00mm, symbol Device:C
- added C18, C24: 4.7uF, Capacitor_THT:CP_Radial_D5.0mm_P2.50mm, symbol Device:C_Polarized
- added C21, C22: 10uF esr, Capacitor_THT:CP_Radial_D5.0mm_P2.50mm, symbol Device:C_Polarized
- added J10: OP_PWR, Connector_JST:JST_XH_B3B-XH-A_1x03_P2.50mm_Vertical, symbol Connector:Conn_01x03_Pin
- added J11: AUDIO_IN, Connector_JST:JST_XH_B2B-XH-A_1x02_P2.50mm_Vertical, symbol Connector:Conn_01x02_Pin
- added J12: AUDIO_OUT, Connector_JST:JST_XH_B2B-XH-A_1x02_P2.50mm_Vertical, symbol Connector:Conn_01x02_Pin
- added R6: 1M, Resistor_THT:R_Axial_DIN0207_L6.3mm_D2.5mm_P10.16mm_Horizontal, symbol Device:R
- added R7, R8: 10R, Resistor_THT:R_Axial_DIN0207_L6.3mm_D2.5mm_P10.16mm_Horizontal, symbol Device:R
- added R9: 47R, Resistor_THT:R_Axial_DIN0207_L6.3mm_D2.5mm_P10.16mm_Horizontal, symbol Device:R
- added U3: OPA1656, Package_DIP:SMDIP-8_W7.62mm, symbol Amplifier_Operational:OPA1656ID
Connections:
- net +12VA: now also C17.2, C18.1, J10.1 (Pin_1), R7.2
- net -12VA: now also C23.1, C24.2, J10.3 (Pin_3), R8.2
- net AUDIO_GND: now also C17.1, C18.2, C19.1, C20.2, C21.2, C22.1, C23.2, C24.1, J10.2 (Pin_2), J11.2 (Pin_2), J12.2 (Pin_2), R6.1, U3.5 (+)
- new net: R9.1, U3.1, U3.2 (-)
- new net: C20.1, C22.2, R8.1, U3.4 (V-)
- new net: U3.6 (-), U3.7
- new net: C19.2, C21.1, R7.1, U3.8 (V+)
- new net AUDIO_IN_VACTROL: J11.1 (Pin_1), R6.2, U3.3 (+)
- new net AUDIO_OUT_AMP: J12.1 (Pin_1), R9.2
