File: amp_v3/opa_buffer_splitter/_restore_backup_2026-10-07T19-32-36-209/opa_buffer_splitter.kicad_pcb (KiCad board)
At the start: 2 copper layers, 94.6 x 109.2 mm, 55 parts, among them J1 UHP_PWR, J10 OP_PWR, J11 AUDIO_IN, J12 AUDIO_OUT, J2 OP_PWR_OUT, J3 OP_PWR_OUT, J4 OP_PWR_OUT, J5 OP_PWR_OUT, J6 OP_PWR, J7 AUDIO_IN, J8 AOUT_MASTER, J9 AOUT_VIS, U1 DPB09B-12, U2 OPA1656, U3 OPA1656

Commit message: updates
Parts:
- C5: moved to F.Cu
- C8: value 1uF PP -> 2.2uF (Film or PP); footprint capacitor JFC:JFC -> Capacitor_THT:C_Rect_L7.2mm_W7.2mm_P5.00mm_FKS2_FKP2_MKS2_MKP2
- R1, R4, R5, R6, R9: footprint Resistor_THT:R_Axial_DIN0207_L6.3mm_D2.5mm_P2.54mm_Vertical -> Resistor_THT:R_Axial_DIN0207_L6.3mm_D2.5mm_P10.16mm_Horizontal
- moved C18 125.3 mm to (163.5, 91.9), turned to 0 degrees
- moved C24 123.1 mm to (163.5, 111.5), turned to 0 degrees
- moved C23 119.6 mm to (156.4, 132.0), turned to 0 degrees
- moved C17 119.6 mm to (156.4, 121.6), turned to 0 degrees
- moved C21 117.8 mm to (163.5, 98.4), turned to 0 degrees
- moved C22 117.8 mm to (163.5, 105.0), turned to 0 degrees
- moved U3 113.0 mm to (172.7, 124.4), turned to 0 degrees
- moved C19 103.7 mm to (156.4, 125.1), turned to 0 degrees
- moved R8 95.4 mm to (143.1, 112.4), turned to 0 degrees
- moved R7 93.9 mm to (143.1, 108.4), turned to 0 degrees
- moved C20 93.0 mm to (156.4, 128.5), turned to 0 degrees
- moved J10 85.3 mm to (116.8, 114.9), turned to 90 degrees
- moved R9 83.4 mm to (143.1, 116.5)
- moved R6 77.0 mm to (143.1, 104.3)
- moved J11 74.2 mm to (135.5, 93.2), turned to 0 degrees
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Connections:
- R9 pad 1: Net-(U3B--) -> Net-(U3A--)
- U3 pad 3: /Buffer/AUDIO_GND -> /Buffer/AUDIO_IN_VACTROL
- U3 pad 5: /Buffer/AUDIO_IN_VACTROL -> /Buffer/AUDIO_GND
Routing:
- net Net-(U2C-V-): track 28.4 -> 0.00 mm
- net Net-(U3C-V-): track 22.6 -> 0.00 mm
- net /Splitter/AUDIO_IN: track 29.6 -> 8.67 mm
- net /Buffer/AUDIO_IN_VACTROL: track 16.1 -> 0.00 mm
- net /Splitter/+12VA: track 15.2 -> 0.00 mm
- net /Splitter/-12VA: track 15.1 -> 0.00 mm
- net /Buffer/+12VA: track 15.0 -> 0.00 mm
- net /Buffer/-12VA: track 15.0 -> 0.00 mm
- net Net-(U2C-V+): track 14.3 -> 0.00 mm
- net Net-(U3C-V+): track 13.9 -> 0.00 mm
- net /Splitter/RCA_IN: track 11.6 -> 0.00 mm
- net Net-(U2A--): track 7.82 -> 0.00 mm
- net /Splitter/AUDIO_OUT_MASTER: track 7.49 -> 0.00 mm
- net Net-(U2B--): track 7.10 -> 0.00 mm
- net Net-(U3B--): track 6.88 -> 0.00 mm
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- removed copper zone on B.Cu, net /Buffer/AUDIO_GND
- removed copper zone on B.Cu, net /Splitter/AUDIO_GND
Other:
- board size 94.6 x 109.2 mm -> 93.3 x 24.1 mm
