File: amp_v3/opa_buffer_splitter/_restore_backup_2026-10-08T20-21-59-931/opa_buffer_splitter.kicad_pcb (KiCad board)
At the start: 2 copper layers, 98.4 x 110.5 mm, 55 parts, among them J1 UHP_PWR, J10 OP_PWR, J11 AUDIO_IN, J12 AUDIO_OUT, J2 PWR_OUT_VA, J3 PWR_OUT_VA, J4 PWR_OUT_VA, J5 PWR_OUT_VA, J6 OP_PWR, J7 AUDIO_IN, J8 AOUT_MASTER, J9 AOUT_VIS, U1 DPB09B-12, U2 OPA1656, U3 OPA1656

Commit message: updates
Parts:
- J2, J3, J4, J5: value PWR_OUT_VA -> OP_PWR_OUT
- U1: footprint MeanWell-DCDC:DPB09B-12 -> Package_SIP:SIP-8_19x3mm_P2.54mm
- moved J5 24.8 mm to (87.0, 44.4)
- moved J2 17.1 mm to (108.0, 44.5)
- moved J4 10.8 mm to (94.0, 44.5)
- moved C3 3.81 mm to (81.9, 47.6)
- moved C4 3.81 mm to (81.9, 38.7)
- moved L2 3.22 mm to (66.7, 35.0)
- moved L1 3.18 mm to (66.7, 46.3)
- moved C1 3.17 mm to (77.5, 46.3)
- moved C2 3.17 mm to (77.5, 37.4)
- moved J3 3.17 mm to (101.0, 44.5)
- moved J9 2.52 mm to (57.1, 79.4), turned to 90 degrees
- moved R5 2.01 mm to (63.5, 79.2)
- moved J8 0.59 mm to (57.8, 95.9), turned to -90 degrees
Connections:
- J2 pad 3: /PSU/AUDIO_GND -> /PSU/-12VA
- J2 pad 4: /PSU/-12VA -> /PSU/AUDIO_GND
- J3 pad 3: /PSU/AUDIO_GND -> /PSU/-12VA
- J3 pad 4: /PSU/-12VA -> /PSU/AUDIO_GND
- J4 pad 3: /PSU/AUDIO_GND -> /PSU/-12VA
- J4 pad 4: /PSU/-12VA -> /PSU/AUDIO_GND
- J5 pad 3: /PSU/AUDIO_GND -> /PSU/-12VA
- J5 pad 4: /PSU/-12VA -> /PSU/AUDIO_GND
Routing:
- net /PSU/-12V_DC: track 16.7 -> 8.99 mm
- net Net-(U2B--): track 9.48 -> 7.10 mm
- net /PSU/-12VA: track 38.7 -> 40.1 mm
- net /Splitter/AUDIO_OUT_MASTER: track 6.57 -> 7.49 mm
- net /PSU/+12V_DC: track 14.8 -> 14.0 mm
- net /PSU/+12VA: track 38.8 -> 38.1 mm
- net /Splitter/AUDIO_OUT_VACTROL: track 5.65 -> 6.24 mm
Other:
- board size 98.4 x 110.5 mm -> 94.6 x 109.2 mm
