File: amp_v3/cap_bank/cap_bank.kicad_pcb (KiCad board)
At the start: 2 copper layers, 118.2 x 88.5 mm, 7 parts, among them J1 Conn_01x02_Pin, J2 Conn_01x02_Pin

Commit message: updates
Parts:
- added C6: C, Library:JFC, F.Cu at (174.3, 83.0)
- moved J1 40.2 mm to (189.4, 51.2)
- moved C5 18.5 mm to (174.3, 72.0)
- moved C4 16.0 mm to (174.3, 61.0)
- moved J2 13.1 mm to (180.6, 51.2), turned to 0 degrees
- moved C3 6.17 mm to (174.3, 42.5)
- moved C2 3.75 mm to (174.3, 31.6)
- moved C1 1.59 mm to (174.3, 20.6)
Connections:
- J2 pad 1: GNDA -> /OUT
- J2 pad 2: /OUT -> GNDA
Routing:
- net /OUT: track 13.5 -> 0.00 mm
- net /IN: track 13.4 -> 0.00 mm
- net GNDA: track 11.0 -> 0.00 mm
Other:
- board size 118.2 x 88.5 mm -> 31.2 x 88.4 mm

Commit message: updates
Parts:
- added C7: 1uF PP, Library:JFC, F.Cu at (33.3, 79.8)
- added C8: 1uF PP, Library:JFC, B.Cu at (33.3, 76.8)
- C1, C3, C5: value C -> 1uF PP
- C2, C4, C6: value C -> 1uF PP; moved to B.Cu
- moved C1 142.3 mm to (33.3, 39.8)
- moved C6 142.0 mm to (33.3, 66.0)
- moved C2 141.4 mm to (33.3, 42.8)
- moved J1 141.3 mm to (48.4, 59.1)
- moved C3 141.2 mm to (33.3, 50.5)
- moved C4 141.2 mm to (33.3, 53.5)
- moved J2 141.1 mm to (39.7, 59.1)
- moved C5 141.0 mm to (33.3, 68.9)
Other:
- board size 31.2 x 88.4 mm -> 32.8 x 63.4 mm

Commit message: updates
Other:
- board size 32.8 x 63.4 mm -> 33.3 x 58.7 mm
Changed lines of the file:
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@@
 	)
 	(gr_rect
-		(start 28.9 28.15)
-		(end 61.7 91.55)
+		(start 28.663 30.286)
+		(end 61.954 88.96)
 		(stroke
 			(width 0.2)
@@
 	)
 	(gr_circle
-		(center 32.5 31.75)
-		(end 34.1 31.75)
+		(center 32.473 34.274)
+		(end 34.073 34.274)
 		(stroke
 			(width 0.2)
@@
 	)
 	(gr_circle
-		(center 32.5 87.95)
-		(end 34.1 87.95)
+		(center 32.5 85.15)
+		(end 34.1 85.15)
 		(stroke
 			(width 0.2)
@@
 	)
 	(gr_circle
-		(center 58.1 31.75)
-		(end 59.7 31.75)
+		(center 58.073 34.274)
+		(end 59.673 34.274)
 		(stroke
 			(width 0.2)
@@
 	)
 	(gr_circle
-		(center 58.1 87.95)
-		(end 59.7 87.95)
+		(center 58.1 85.15)
+		(end 59.7 85.15)
 		(stroke
 			(width 0.2)
@@
 			(clearance 0.8)
 		)
-		(min_thickness 0.25)
+		(min_thickness 0.8)
 		(fill yes
-			(thermal_gap 0.5)
-			(thermal_bridge_width 0.5)
+			(thermal_gap 0.8)
+			(thermal_bridge_width 0.8)
 			(smoothing fillet)
-			(radius 1)
-			(island_removal_mode 1)
+			(radius 0.5)
+			(island_removal_mode 0)
 		)
 		(polygon
@@
 			(clearance 0.8)
 		)
-		(min_thickness 0.25)
+		(min_thickness 0.8)
 		(fill yes
-			(thermal_gap 0.5)
-			(thermal_bridge_width 0.5)
+			(thermal_gap 0.8)
+			(thermal_bridge_width 0.8)
 			(smoothing fillet)
-			(radius 1)
-			(island_removal_mode 1)
+			(radius 0.5)
+			(island_removal_mode 0)
 		)
 		(polygon
@@
 			(clearance 0.8)
 		)
-		(min_thickness 0.25)
+		(min_thickness 0.8)
 		(fill yes
-			(thermal_gap 0.5)
-			(thermal_bridge_width 0.5)
+			(thermal_gap 0.8)
+			(thermal_bridge_width 0.8)
 			(smoothing fillet)
-			(radius 1)
-			(island_removal_mode 1)
+			(radius 0.5)
+			(island_removal_mode 0)
 		)
 		(polygon
@@
 			(clearance 0.8)
 		)
-		(min_thickness 0.25)
+		(min_thickness 0.8)
 		(fill yes
-			(thermal_gap 0.5)
-			(thermal_bridge_width 0.5)
+			(thermal_gap 0.8)
+			(thermal_bridge_width 0.8)
 			(smoothing fillet)
-			(radius 1)
-			(island_removal_mode 1)
+			(radius 0.5)
+			(island_removal_mode 0)
 		)
 		(polygon
@@
 		(hatch none 0.5)
 		(connect_pads yes
-			(clearance 1)
+			(clearance 0.8)
 		)
-		(min_thickness 1)
+		(min_thickness 0.8)
 		(fill yes
-			(thermal_gap 1.5)
-			(thermal_bridge_width 1.5)
+			(thermal_gap 0.8)
+			(thermal_bridge_width 0.8)
 			(smoothing fillet)
-			(radius 1)
+			(radius 0.5)
 			(island_removal_mode 0)
 		)
 		(polygon
 			(pts
-				(xy 29.9 29.15) (xy 60.7 29.15) (xy 60.7 90.55) (xy 29.9 90.55)
+				(xy 29.9 31.556) (xy 60.7 31.556) (xy 60.7 87.69) (xy 29.9 87.69)
 			)
 		)

Commit message: updates
Parts:
- added C9: 10uF PP, Library:10uF - D18 - W46, F.Cu at (95.5, 111.2)
- added C9: 10uF PP, Library:10uF - D18 - W46, F.Cu at (95.5, 69.3)
- added C9: 10uF PP, Library:10uF - D18 - W46, F.Cu at (95.5, 90.2)
- added C9: 10uF PP, Library:10uF - D18 - W46, F.Cu at (95.5, 48.3)
- added J3: CAP_IN, Connector_JST:JST_XH_B2B-XH-A_1x02_P2.50mm_Vertical, F.Cu at (131.8, 80.7)
- added J3: CAP_IN, Connector_JST:JST_XH_B2B-XH-A_1x02_P2.50mm_Vertical, F.Cu at (131.8, 101.6)
- added J3: CAP_IN, Connector_JST:JST_XH_B2B-XH-A_1x02_P2.50mm_Vertical, F.Cu at (131.8, 59.7)
- added J3: CAP_IN, Connector_JST:JST_XH_B2B-XH-A_1x02_P2.50mm_Vertical, F.Cu at (131.8, 122.6)
- added J4: CAP_OUT, Connector_JST:JST_XH_B2B-XH-A_1x02_P2.50mm_Vertical, F.Cu at (78.9, 122.6)
- added J4: CAP_OUT, Connector_JST:JST_XH_B2B-XH-A_1x02_P2.50mm_Vertical, F.Cu at (78.9, 59.8)
- added J4: CAP_OUT, Connector_JST:JST_XH_B2B-XH-A_1x02_P2.50mm_Vertical, F.Cu at (78.9, 101.7)
- added J4: CAP_OUT, Connector_JST:JST_XH_B2B-XH-A_1x02_P2.50mm_Vertical, F.Cu at (78.9, 80.7)
Routing:
- net /OUT: track 0.00 -> 17.6 mm
- net /IN: track 0.00 -> 16.6 mm
Other:
- board size 33.3 x 58.7 mm -> 108.1 x 96.8 mm

Commit message: updates v1b
Parts:
- removed the C9 at (95.5, 111.2)
- removed the C9 at (95.5, 69.3)
- removed the C9 at (95.5, 90.2)
- removed the J3 at (131.8, 80.7)
- removed the J3 at (131.8, 101.6)
- removed the J3 at (131.8, 122.6)
- removed the J4 at (78.9, 122.6)
- removed the J4 at (78.9, 101.7)
- removed the J4 at (78.9, 80.7)
- added C10: 1uF PP, Library:JFC, F.Cu at (99.4, 75.6)
- added C11: 1uF PP, Library:JFC, F.Cu at (99.4, 86.7)
- added J5: CAP_IN, Connector_JST:JST_XH_B2B-XH-A_1x02_P2.50mm_Vertical, F.Cu at (127.8, 81.3)
- added J6: CAP_OUT, Connector_JST:JST_XH_B2B-XH-A_1x02_P2.50mm_Vertical, F.Cu at (94.9, 80.7)
- moved J3 12.7 mm to (132.9, 47.1), turned to -90 degrees
- moved J4 0.64 mm to (78.3, 59.7)
Routing:
- net /IN: track 16.6 -> 17.3 mm
Other:
- board size 108.1 x 96.8 mm -> 108.1 x 62.5 mm
