File: amp_v3/cap_bank/cap_bank.kicad_sch (KiCad schematic)
At the start: 7 parts, among them J1 Conn_01x02_Pin, J2 Conn_01x02_Pin

Commit message: updates
Parts:
- added C6: C, Library:JFC, symbol Device:C
Connections:
- net GNDA: now also J2.2 (Pin_2); no longer J2.1 (Pin_1)
- net IN: now also C6.2
- net OUT: now also J2.1 (Pin_1), C6.1; no longer J2.2 (Pin_2)
Other:
- moved on the sheet: J2
Changed lines of the file:
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@@
+	)
+	(junction
+		(at 101.6 72.39)
+		(diameter 0)
+		(color 0 0 0 0)
 	)
 	(junction
@@
 	)
 	(junction
+		(at 113.03 64.77)
+		(diameter 0)
+		(color 0 0 0 0)
+	)
+	(junction
 		(at 78.74 64.77)
 		(diameter 0)
@@
 	(wire
 		(pts
-			(xy 101.6 64.77) (xy 105.41 64.77)
-		)
-		(stroke
-			(width 0)
-			(type default)
-		)
-	)
-	(wire
-		(pts
-			(xy 105.41 59.69) (xy 105.41 64.77)
+			(xy 101.6 64.77) (xy 113.03 64.77)
+		)
+		(stroke
+			(width 0)
+			(type default)
+		)
+	)
+	(wire
+		(pts
+			(xy 115.57 59.69) (xy 115.57 64.77)
 		)
 		(stroke
@@
 	(wire
 		(pts
+			(xy 101.6 72.39) (xy 113.03 72.39)
+		)
+		(stroke
+			(width 0)
+			(type default)
+		)
+	)
+	(wire
+		(pts
 			(xy 90.17 64.77) (xy 101.6 64.77)
+		)
+		(stroke
+			(width 0)
+			(type default)
+		)
+	)
+	(wire
+		(pts
+			(xy 113.03 64.77) (xy 115.57 64.77)
 		)
 		(stroke
@@
 	)
 	(label "OUT"
-		(at 105.41 59.69 0)
+		(at 115.57 59.69 0)
 		(effects
 			(font
@@
 	(symbol
 		(lib_id "Connector:Conn_01x02_Pin")
-		(at 83.82 39.37 270)
+		(at 81.28 39.37 90)
+		(mirror x)
 		(unit 1)
 		(body_style 1)
@@
 		(in_pos_files yes)
 		(dnp no)
-		(fields_autoplaced yes)
 		(property "Reference" "J2"
-			(at 85.09 38.7349 90)
+			(at 80.01 38.7349 90)
 			(show_name no)
 			(do_not_autoplace no)
@@
 		)
 		(property "Value" "Conn_01x02_Pin"
-			(at 85.09 41.2749 90)
+			(at 80.01 41.2749 90)
 			(show_name no)
 			(do_not_autoplace no)
@@
 		)
 		(property "Footprint" "Connector_JST:JST_XH_B2B-XH-A_1x02_P2.50mm_Vertical"
-			(at 83.82 39.37 0)
+			(at 81.28 39.37 0)
 			(hide yes)
 			(show_name no)
@@
 		)
 		(property "Datasheet" ""
-			(at 83.82 39.37 0)
+			(at 81.28 39.37 0)
 			(hide yes)
 			(show_name no)
@@
 		)
 		(property "Description" "Generic connector, single row, 01x02, script generated"
-			(at 83.82 39.37 0)
+			(at 81.28 39.37 0)
 			(hide yes)
 			(show_name no)
@@
 					(unit 1)
 				)
+			)
+		)
+	)
+	(symbol
+		(lib_id "Device:C")
+		(at 113.03 68.58 0)
+		(unit 1)
+		(body_style 1)
+		(exclude_from_sim no)
+		(in_bom yes)
+		(on_board yes)
+		(in_pos_files yes)
+		(dnp no)
+		(fields_autoplaced yes)
+		(property "Reference" "C6"
+			(at 116.84 67.3099 0)
+			(show_name no)
+			(do_not_autoplace no)
+			(effects
+				(font
+					(size 1.27 1.27)
+				)
+				(justify left)
+			)
+		)
+		(property "Value" "C"
+			(at 116.84 69.8499 0)
+			(show_name no)
+			(do_not_autoplace no)
+			(effects
+				(font
+					(size 1.27 1.27)
+				)
+				(justify left)
+			)
+		)
+		(property "Footprint" "Library:JFC"
+			(at 113.9952 72.39 0)
+			(hide yes)
+			(show_name no)
+			(do_not_autoplace no)
+			(effects
+				(font
+					(size 1.27 1.27)
+				)
+			)
+		)
+		(property "Datasheet" ""
+			(at 113.03 68.58 0)
+			(hide yes)
+			(show_name no)
+			(do_not_autoplace no)
+			(effects
+				(font
+					(size 1.27 1.27)
+				)
+			)
+		)
+		(property "Description" "Unpolarized capacitor"
+			(at 113.03 68.58 0)
+			(hide yes)
+			(show_name no)
+			(do_not_autoplace no)
+			(effects
+				(font
+					(size 1.27 1.27)
+				)
+			)
+		)
+		(pin "1"
+		)
+		(pin "2"
+		)
+		(instances
+			(project "cap_bank"
+				(path "/f17f0f6a-aa79-4f33-8502-21ae7788042f"
+					(reference "C6")
+					(unit 1)
+				)

Commit message: updates
Parts:
- added C7, C8: 1uF PP, Library:JFC, symbol Device:C
- C1, C2, C3, C4, C5, C6: value C -> 1uF PP
Connections:
- net IN: now also C7.2, C8.2
- net OUT: now also C7.1, C8.1

Commit message: updates
Parts:
- added C9: 10uF PP, Library:10uF - D18 - W46, symbol Device:C
- added J3: CAP_IN, Connector_JST:JST_XH_B2B-XH-A_1x02_P2.50mm_Vertical, symbol Connector:Conn_01x02_Pin
- added J4: CAP_OUT, Connector_JST:JST_XH_B2B-XH-A_1x02_P2.50mm_Vertical, symbol Connector:Conn_01x02_Pin
Connections:
- net GNDA: now also J3.1 (Pin_1), J4.1 (Pin_1)
- net IN: now also C9.1, J3.2 (Pin_2)
- net OUT: now also C9.2, J4.2 (Pin_2)

Commit message: updates v1b
Parts:
- added C10, C11: 1uF PP, Library:JFC, symbol Device:C
- added J5: CAP_IN, Connector_JST:JST_XH_B2B-XH-A_1x02_P2.50mm_Vertical, symbol Connector:Conn_01x02_Pin
- added J6: CAP_OUT, Connector_JST:JST_XH_B2B-XH-A_1x02_P2.50mm_Vertical, symbol Connector:Conn_01x02_Pin
Connections:
- net GNDA: now also J5.1 (Pin_1), J6.1 (Pin_1)
- net IN: now also C10.2, C11.2, J5.2 (Pin_2)
- net OUT: now also C10.1, C11.1, J6.2 (Pin_2)
