File: amp_v3/ground_loop_breaker/ground_loop_breaker.kicad_sch (KiCad schematic)
At the start: 6 parts, among them J1 Conn_01x02_Socket, J2 Conn_01x03_Socket

Commit message: updates
Parts:
- J1: footprint Connector_AMASS:AMASS_XT30U-F_1x02_P5.0mm_Vertical -> TerminalBlock_Phoenix:TerminalBlock_Phoenix_PT-1,5-2-5.0-H_1x02_P5.00mm_Horizontal
- J2: footprint Connector_TE-Connectivity:TE_826576-3_1x03_P3.96mm_Vertical -> TerminalBlock_Phoenix:TerminalBlock_Phoenix_PT-1,5-3-5.0-H_1x03_P5.00mm_Horizontal
Changed lines of the file:
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@@
 			)
 		)
-		(property "Footprint" "Connector_AMASS:AMASS_XT30U-F_1x02_P5.0mm_Vertical"
+		(property "Footprint" "TerminalBlock_Phoenix:TerminalBlock_Phoenix_PT-1,5-2-5.0-H_1x02_P5.00mm_Horizontal"
 			(at 69.85 44.45 0)
 			(hide yes)
@@
 			)
 		)
-		(property "Footprint" "Connector_TE-Connectivity:TE_826576-3_1x03_P3.96mm_Vertical"
+		(property "Footprint" "TerminalBlock_Phoenix:TerminalBlock_Phoenix_PT-1,5-3-5.0-H_1x03_P5.00mm_Horizontal"
 			(at 82.55 44.45 0)
 			(hide yes)

Commit message: updates
Changed lines of the file:
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@@
 		(dnp no)
 		(property "Reference" "R1"
-			(at 81.788 57.15 90)
+			(at 82.042 59.944 90)
 			(show_name no)
 			(do_not_autoplace no)
@@
 		)
 		(property "Value" "10"
-			(at 67.31 57.15 90)
+			(at 69.596 59.436 90)
 			(show_name no)
 			(do_not_autoplace no)
