File: amp_v3/opa_buffer_dual_rail/opa_buffer_dual_rail.kicad_sch (KiCad schematic)
At the start: 16 parts, among them J10 PWR_IN, J11 AUDIO_IN, J12 AUDIO_OUT, U3 OPA1656

Commit message: updates
Parts:
- C17, C19, C20, C23: footprint Capacitor_THT:C_Disc_D4.3mm_W1.9mm_P5.00mm -> Capacitor_THT:C_Disc_D3.8mm_W2.6mm_P2.50mm
- R9: footprint Resistor_THT:R_Axial_DIN0207_L6.3mm_D2.5mm_P7.62mm_Horizontal -> Resistor_THT:R_Axial_DIN0207_L6.3mm_D2.5mm_P2.54mm_Vertical
Other:
- note added: "X7R Caps"
- note removed: "Film Caps (wima)"
Changed lines of the file:
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@@
 	(generator_version "10.0")
 	(paper "A4")
-	(text "Film Caps (wima)\n"
+	(text "X7R Caps\n"
 		(exclude_from_sim no)
-		(at 76.454 87.63 0)
+		(at 107.696 41.148 0)
 		(effects
 			(font
@@
 		)
 	)
-	(text "Film Caps (wima)\n"
+	(text "X7R Caps\n"
 		(exclude_from_sim no)
-		(at 107.696 41.148 0)
+		(at 79.756 87.376 0)
 		(effects
 			(font
@@
 			)
 		)
-		(property "Footprint" "Resistor_THT:R_Axial_DIN0207_L6.3mm_D2.5mm_P7.62mm_Horizontal"
+		(property "Footprint" "Resistor_THT:R_Axial_DIN0207_L6.3mm_D2.5mm_P2.54mm_Vertical"
 			(at 180.34 76.708 90)
 			(hide yes)
@@
 			)
 		)
-		(property "Footprint" "Capacitor_THT:C_Disc_D4.3mm_W1.9mm_P5.00mm"
+		(property "Footprint" "Capacitor_THT:C_Disc_D3.8mm_W2.6mm_P2.50mm"
 			(at 87.9348 27.94 0)
 			(hide yes)
@@
 			)
 		)
-		(property "Footprint" "Capacitor_THT:C_Disc_D4.3mm_W1.9mm_P5.00mm"
+		(property "Footprint" "Capacitor_THT:C_Disc_D3.8mm_W2.6mm_P2.50mm"
 			(at 107.6452 95.25 0)
 			(hide yes)
@@
 			)
 		)
-		(property "Footprint" "Capacitor_THT:C_Disc_D4.3mm_W1.9mm_P5.00mm"
+		(property "Footprint" "Capacitor_THT:C_Disc_D3.8mm_W2.6mm_P2.50mm"
 			(at 107.6452 72.39 0)
 			(hide yes)
@@
 			)
 		)
-		(property "Footprint" "Capacitor_THT:C_Disc_D4.3mm_W1.9mm_P5.00mm"
+		(property "Footprint" "Capacitor_THT:C_Disc_D3.8mm_W2.6mm_P2.50mm"
 			(at 87.9348 48.26 0)
 			(hide yes)
